File: kicad/Frame_PCB/V0-UmbilicalBoard.kicad_sch (KiCad schematic)
At the start: 16 parts, among them J1 Conn_02x08_Odd_Even, J10 Neopixel Strip 1, J11 Neopixel Strip 1, J12 Neopixel Out, J2 Motor, J3 Hotend Fan, J4 Part Cooling Fan, J5 Heater, J6 Thermistor, J7 X-Endstop, J8 Chamber Thermistor, J9 Neopixel (from controller)

Commit message: v0 2020
Parts:
- removed C1, C2, C3: C, Capacitor_SMD:C_0805_2012Metric_Pad1.18x1.45mm_HandSolder, symbol Device:C
- removed J10, J11: Neopixel Strip 1, Connector_JST:JST_XH_B4B-XH-A_1x04_P2.50mm_Vertical, symbol Connector_Generic:Conn_01x04
- removed J12: Neopixel Out, Connector_JST:JST_XH_B3B-XH-A_1x03_P2.50mm_Vertical, symbol Connector_Generic:Conn_01x03
- removed J8: Chamber Thermistor, Connector_JST:JST_XH_B2B-XH-A_1x02_P2.50mm_Vertical, symbol Connector_Generic:Conn_01x02
- removed J9: Neopixel (from controller), Connector_JST:JST_XH_B3B-XH-A_1x03_P2.50mm_Vertical, symbol Connector_Generic:Conn_01x03
- removed TH1: Thermistor, Resistor_SMD:R_0805_2012Metric_Pad1.20x1.40mm_HandSolder, symbol Device:Thermistor
- added H1, H2: MountingHole_Pad, MountingHole:MountingHole_3.2mm_M3_Pad, symbol Mechanical:MountingHole_Pad
Connections:
- net GND: now also H1.1, H2.1
