File: kicad/Sensor board V10/sensorboard_v10/voltage.kicad_sch (KiCad schematic)
At the start: 2 parts

Commit message: Sensor Board V10
Parts:
- added C13: 100nF, RMC_Capacitor:C_0805_2012Metric_Pad1.18x1.45mm_HandSolder_L, symbol Device:C
- added J13: Conn_01x03, Connector_JST:JST_XH_B3B-XH-A_1x03_P2.50mm_Vertical, symbol Connector_Generic:Conn_01x03
- R7: renamed from R5; footprint (none) -> RMC_Resistor:R_0805_2012Metric_Pad1.20x1.40mm_HandSolder_L
- R8: renamed from R4; footprint (none) -> RMC_Resistor:R_0805_2012Metric_Pad1.20x1.40mm_HandSolder_L
Connections:
- net +5V: now also J13.3 (Pin_3); no longer R7.1
- net GND: now also C13.1, J13.2 (Pin_2)
- net 2.5V renamed 1.65V OUTPUT
- net 1.65V OUTPUT: now also C13.2
- new net 3.3V_INPUT: J13.1 (Pin_1), R7.1

Commit message: Sensor Board V10 schematics
Connections:
- net 1.65V OUTPUT renamed 2.5V OUTPUT
- net 3.3V_INPUT renamed 5V_INPUT
Changed lines of the file:
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@@
 		)
 	)
-	(hierarchical_label "3.3V_INPUT"
+	(hierarchical_label "5V_INPUT"
 		(shape input)
 		(at 46.99 69.215 0)
@@
 		)
 	)
-	(hierarchical_label "1.65V OUTPUT"
+	(hierarchical_label "2.5V OUTPUT"
 		(shape output)
 		(at 102.235 81.28 0)
@@
 		)
 	)
-	(hierarchical_label "3.3V_INPUT"
+	(hierarchical_label "5V_INPUT"
 		(shape input)
 		(at 80.01 81.28 180)
@@
 				(path "/bee3e03c-9a5f-4c66-913e-823f7b125a2a/c95b4a2b-b42a-4024-af14-ef340befd390"
 					(reference "R20")
-					(unit 1)
-				)
-				(path "/bee3e03c-9a5f-4c66-913e-823f7b125a2a/1153a467-d12c-4cbb-8264-2e80c29423fe"
-					(reference "R22")
 					(unit 1)
 				)
@@
 					(unit 1)
 				)
-				(path "/bee3e03c-9a5f-4c66-913e-823f7b125a2a/1153a467-d12c-4cbb-8264-2e80c29423fe"
-					(reference "J19")
-					(unit 1)
-				)
 				(path "/bee3e03c-9a5f-4c66-913e-823f7b125a2a/ee05c668-fdc5-4e58-a917-4d64b0e277cb"
 					(reference "J12")
@@
 					(unit 1)
 				)
-				(path "/bee3e03c-9a5f-4c66-913e-823f7b125a2a/1153a467-d12c-4cbb-8264-2e80c29423fe"
-					(reference "#PWR058")
-					(unit 1)
-				)
 			)
 		)
@@
 					(unit 1)
 				)
-				(path "/bee3e03c-9a5f-4c66-913e-823f7b125a2a/1153a467-d12c-4cbb-8264-2e80c29423fe"
-					(reference "C20")
-					(unit 1)
-				)
 			)
 		)
@@
 					(unit 1)
 				)
-				(path "/bee3e03c-9a5f-4c66-913e-823f7b125a2a/1153a467-d12c-4cbb-8264-2e80c29423fe"
-					(reference "#PWR060")
-					(unit 1)
-				)
 			)
 		)
@@
 				(path "/bee3e03c-9a5f-4c66-913e-823f7b125a2a/c95b4a2b-b42a-4024-af14-ef340befd390"
 					(reference "R19")
-					(unit 1)
-				)
-				(path "/bee3e03c-9a5f-4c66-913e-823f7b125a2a/1153a467-d12c-4cbb-8264-2e80c29423fe"
-					(reference "R21")
 					(unit 1)
 				)
@@
 					(unit 1)
 				)
-				(path "/bee3e03c-9a5f-4c66-913e-823f7b125a2a/1153a467-d12c-4cbb-8264-2e80c29423fe"
-					(reference "#PWR059")
-					(unit 1)
-				)
