File: kicad/Sensor board V10/sensorboard_v10/sensorboard_v10.kicad_sch (KiCad schematic)
At the start: 76 parts, among them J1 Conn_01x03, J10 Conn_01x04, J11 Conn_01x02, J2 USB_C_Receptacle_USB2.0_14P, J20 Conn_01x02, J21 Conn_01x02, J23 Conn_01x03, J25 Conn_01x04, J26 Conn_01x03, J27 Conn_01x03, J3 Conn_01x02, J6 Conn_01x04, J7 Conn_01x04, Q1 MMBT3904, Q2 MMBT3904, SW1 SW_SPST, SW2 SW_SPST, U1 ESP32-S3-WROOM-2, U2 CH340C, U3 TJA1051T-3, U4 LM2576S-5, U5 AMS1117-3.3, U7 TXS0102DCU, U9 MT3608/SDB628

Commit message: sensor board v10
Parts:
- C32, C33: footprint RMC_Capacitor:C_0805_2012Metric_Pad1.18x1.45mm_HandSolder_L -> RMC_Capacitor:CP_EIA-3528-15_AVX-H_Pad1.50x2.35mm_HandSolder_RMC
Changed lines of the file:
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@@
 	(paper "A4")
 	(junction
-		(at 196.85 29.21)
+		(at 179.07 58.42)
 		(diameter 0)
 		(color 0 0 0 0)
 	)
 	(junction
-		(at 179.07 58.42)
+		(at 196.85 29.21)
 		(diameter 0)
 		(color 0 0 0 0)
@@
 			)
 		)
-		(property "Footprint" "RMC_Capacitor:C_0805_2012Metric_Pad1.18x1.45mm_HandSolder_L"
+		(property "Footprint" "RMC_Capacitor:CP_EIA-3528-15_AVX-H_Pad1.50x2.35mm_HandSolder_RMC"
 			(at 219.4052 66.04 0)
 			(effects
@@
 	)
 	(symbol
+		(lib_id "Device:C_Polarized")
+		(at 179.07 62.23 0)
+		(unit 1)
+		(exclude_from_sim no)
+		(in_bom yes)
+		(on_board yes)
+		(dnp no)
+		(property "Reference" "C32"
+			(at 182.88 60.0709 0)
+			(effects
+				(font
+					(size 1.27 1.27)
+				)
+				(justify left)
+			)
+		)
+		(property "Value" "22uF"
+			(at 182.88 62.6109 0)
+			(effects
+				(font
+					(size 1.27 1.27)
+				)
+				(justify left)
+			)
+		)
+		(property "Footprint" "RMC_Capacitor:CP_EIA-3528-15_AVX-H_Pad1.50x2.35mm_HandSolder_RMC"
+			(at 180.0352 66.04 0)
+			(effects
+				(font
+					(size 1.27 1.27)
+				)
+				(hide yes)
+			)
+		)
+		(property "Datasheet" "~"
+			(at 179.07 62.23 0)
+			(effects
+				(font
+					(size 1.27 1.27)
+				)
+				(hide yes)
+			)
+		)
+		(property "Description" "Polarized capacitor"
+			(at 179.07 62.23 0)
+			(effects
+				(font
+					(size 1.27 1.27)
+				)
+				(hide yes)
+			)
+		)
+		(pin "1"
+		)
+		(pin "2"
+		)
+		(instances
+			(project "sensorboard_v10"
+				(path "/bee3e03c-9a5f-4c66-913e-823f7b125a2a"
+					(reference "C32")
+					(unit 1)
+				)
+			)
+		)
+	)
+	(symbol
 		(lib_id "Device:C")
 		(at 184.15 34.29 180)
@@
 					(unit 1)
 				)
-			)
-		)
-	)
-	(symbol
-		(lib_id "Device:C_Polarized")
-		(at 179.07 62.23 0)
-		(unit 1)
-		(exclude_from_sim no)
-		(in_bom yes)
-		(on_board yes)
-		(dnp no)
-		(property "Reference" "C32"
-			(at 182.88 60.0709 0)
-			(effects
-				(font
-					(size 1.27 1.27)
-				)
-				(justify left)
-			)
-		)
-		(property "Value" "22uF"
-			(at 182.88 62.6109 0)
-			(effects
-				(font
-					(size 1.27 1.27)
-				)
-				(justify left)
-			)
-		)
-		(property "Footprint" "RMC_Capacitor:C_0805_2012Metric_Pad1.18x1.45mm_HandSolder_L"
-			(at 180.0352 66.04 0)
-			(effects
-				(font
-					(size 1.27 1.27)
-				)
-				(hide yes)
-			)
-		)
-		(property "Datasheet" "~"
-			(at 179.07 62.23 0)
-			(effects
-				(font
-					(size 1.27 1.27)
-				)
-				(hide yes)
-			)
-		)
-		(property "Description" "Polarized capacitor"
-			(at 179.07 62.23 0)
-			(effects
-				(font
-					(size 1.27 1.27)
-				)
-				(hide yes)
-			)
-		)
-		(pin "1"
-		)
-		(pin "2"
-		)
-		(instances
-			(project "sensorboard_v10"
-				(path "/bee3e03c-9a5f-4c66-913e-823f7b125a2a"
-					(reference "C32")
-					(unit 1)
-				)
