File: kicad/BDU/BDU_v1/BDU_v1.kicad_pcb (KiCad board)
At the start: 2 copper layers, 2 parts, among them U1 LTV-847S, U2 TRA3-1212

Commit message: BDU
Parts:
- added C1: 2.2uF, RMC_Capacitor:C_0805_2012Metric_Pad1.18x1.45mm_HandSolder_L, F.Cu at (169.7, 94.2)
- added C2: 1uF, RMC_Capacitor:C_0805_2012Metric_Pad1.18x1.45mm_HandSolder_L, F.Cu at (169.9, 104.5)
- added D1: LED, RMC_LED:LED_0805_2012Metric_Pad1.45x1.40mm_HandSolder, F.Cu at (195.3, 90.0)
- added D2: LED, RMC_LED:LED_0805_2012Metric_Pad1.45x1.40mm_HandSolder, F.Cu at (190.2, 90.0)
- added D3: LED, RMC_LED:LED_0805_2012Metric_Pad1.45x1.40mm_HandSolder, F.Cu at (185.1, 90.0)
- added D4: LED, RMC_LED:LED_0805_2012Metric_Pad1.45x1.40mm_HandSolder, F.Cu at (180.2, 90.0)
- added F10: Fuse, Fuse:Fuseholder_Littelfuse_Nano2_157x, F.Cu at (127.0, 111.3)
- added F2: Fuse, Fuse:Fuseholder_Littelfuse_Nano2_157x, F.Cu at (144.4, 110.6)
- added H1: MountingHole_Pad, MountingHole:MountingHole_4.3mm_M4_DIN965_Pad, F.Cu at (85.0, 75.0)
- added H2: MountingHole_Pad, MountingHole:MountingHole_4.3mm_M4_DIN965_Pad, F.Cu at (158.2, 75.0)
- added H3: MountingHole_Pad, MountingHole:MountingHole_4.3mm_M4_DIN965_Pad, F.Cu at (215.0, 75.0)
- added H4: MountingHole_Pad, MountingHole:MountingHole_4.3mm_M4_DIN965_Pad, F.Cu at (85.0, 125.0)
- added H5: MountingHole_Pad, MountingHole:MountingHole_4.3mm_M4_DIN965_Pad, F.Cu at (158.2, 125.0)
- added H6: MountingHole_Pad, MountingHole:MountingHole_4.3mm_M4_DIN965_Pad, F.Cu at (215.0, 125.0)
- added J1: Relay connector, Connector_Molex:Molex_Micro-Fit_3.0_43650-0410_1x04-1MP_P3.00mm_Horizontal_PnP, F.Cu at (175.0, 124.4)
- added J10: Voltmeter-, Connector_Molex:Molex_Micro-Fit_3.0_43650-0210_1x02-1MP_P3.00mm_Horizontal_PnP, F.Cu at (85.5, 100.0)
- added J11: IMD-, Connector_Molex:Molex_Micro-Fit_3.0_43650-0210_1x02-1MP_P3.00mm_Horizontal_PnP, F.Cu at (100.0, 75.0)
- added J12: AIR-, Connector_Molex:Molex_Micro-Fit_3.0_43650-0210_1x02-1MP_P3.00mm_Horizontal_PnP, F.Cu at (85.5, 111.1)
- added J13: AIR+, Connector_Molex:Molex_Micro-Fit_3.0_43650-0210_1x02-1MP_P3.00mm_Horizontal_PnP, F.Cu at (142.9, 124.2)
- added J14: AIR+, Connector_Molex:Molex_Micro-Fit_3.0_43650-0210_1x02-1MP_P3.00mm_Horizontal_PnP, F.Cu at (214.9, 90.5)
- added J15: AMS, Connector_Molex:Molex_Micro-Fit_3.0_43650-0410_1x04-1MP_P3.00mm_Horizontal_PnP, F.Cu at (196.4, 75.9)
- added J16: DCDC, Connector_Molex:Molex_Micro-Fit_3.0_43650-0210_1x02-1MP_P3.00mm_Horizontal_PnP, F.Cu at (181.4, 75.7)
- added J2: Relay connector, Connector_Molex:Molex_Micro-Fit_3.0_43650-0410_1x04-1MP_P3.00mm_Horizontal_PnP, F.Cu at (196.2, 124.4)
- added J3: Relay connector, Connector_Molex:Molex_Micro-Fit_3.0_43650-0410_1x04-1MP_P3.00mm_Horizontal_PnP, F.Cu at (214.4, 109.3)
- added J4: Conn_01x02, Connector_Molex:Molex_Micro-Fit_3.0_43650-0210_1x02-1MP_P3.00mm_Horizontal_PnP, F.Cu at (170.0, 75.8)
- added J5: IMD+, Connector_Molex:Molex_Micro-Fit_3.0_43650-0210_1x02-1MP_P3.00mm_Horizontal_PnP, F.Cu at (115.0, 75.0)
- added J6: Voltmeter+, Connector_Molex:Molex_Micro-Fit_3.0_43650-0210_1x02-1MP_P3.00mm_Horizontal_PnP, F.Cu at (127.3, 75.0)
- added J7: TSAL_green+, Connector_Molex:Molex_Micro-Fit_3.0_43650-0210_1x02-1MP_P3.00mm_Horizontal_PnP, F.Cu at (139.7, 75.2)
- added J8: AIR+, Connector_Molex:Molex_Micro-Fit_3.0_43650-0210_1x02-1MP_P3.00mm_Horizontal_PnP, F.Cu at (130.8, 124.2)
- added J9: TSAL_green-, Connector_Molex:Molex_Micro-Fit_3.0_43650-0210_1x02-1MP_P3.00mm_Horizontal_PnP, F.Cu at (85.5, 88.0)
- added R1: 3K9, Resistor_THT:R_Axial_DIN0207_L6.3mm_D2.5mm_P15.24mm_Horizontal, F.Cu at (144.7, 103.1)
- added R10: 1k, RMC_Resistor:R_0805_2012Metric_Pad1.20x1.40mm_HandSolder_L, F.Cu at (194.2, 93.9)
- added R11: 1k, RMC_Resistor:R_0805_2012Metric_Pad1.20x1.40mm_HandSolder_L, F.Cu at (189.1, 94.0)
- added R12: 1k, RMC_Resistor:R_0805_2012Metric_Pad1.20x1.40mm_HandSolder_L, F.Cu at (184.0, 94.0)
- added R13: 1k, RMC_Resistor:R_0805_2012Metric_Pad1.20x1.40mm_HandSolder_L, F.Cu at (179.0, 94.0)
- added R2: 1k, RMC_Resistor:R_0805_2012Metric_Pad1.20x1.40mm_HandSolder_L, F.Cu at (178.8, 111.8)
- added R3: 1k, RMC_Resistor:R_0805_2012Metric_Pad1.20x1.40mm_HandSolder_L, F.Cu at (183.9, 111.6)
- added R4: 1k, RMC_Resistor:R_0805_2012Metric_Pad1.20x1.40mm_HandSolder_L, F.Cu at (188.9, 111.7)
- added R5: 1k, RMC_Resistor:R_0805_2012Metric_Pad1.20x1.40mm_HandSolder_L, F.Cu at (194.1, 111.8)
- added R6: 4k7, RMC_Resistor:R_0805_2012Metric_Pad1.20x1.40mm_HandSolder_L, F.Cu at (181.4, 94.0)
- added R7: 4k7, RMC_Resistor:R_0805_2012Metric_Pad1.20x1.40mm_HandSolder_L, F.Cu at (186.4, 93.9)
- added R8: 4k7, RMC_Resistor:R_0805_2012Metric_Pad1.20x1.40mm_HandSolder_L, F.Cu at (191.5, 94.0)
- added R9: 4k7, RMC_Resistor:R_0805_2012Metric_Pad1.20x1.40mm_HandSolder_L, F.Cu at (196.7, 94.1)
- moved U1 107.1 mm to (187.7, 102.9), turned to 90 degrees
- moved U2 76.2 mm to (166.3, 93.0)
Connections:
- U1 pad 11: unconnected-(U1-Pad11) -> /pre_out
- U1 pad 13: unconnected-(U1-Pad13) -> /low_out
- U1 pad 15: unconnected-(U1-Pad15) -> /high_out
- U1 pad 8: GND -> PRE-
- U1 pad 9: unconnected-(U1-Pad9) -> /sdc_out
Routing:
- net /low_out: track 0.00 -> 5.55 mm
- net /pre_out: track 0.00 -> 5.40 mm
- net /high_out: track 0.00 -> 5.39 mm
- net Net-(R2-Pad2): track 0.00 -> 3.00 mm
- net TS+: track 0.00 -> 3.00 mm
- net Net-(R5-Pad2): track 0.00 -> 2.99 mm
- net Net-(R4-Pad2): track 0.00 -> 2.92 mm
- net Net-(D4-A): track 0.00 -> 2.87 mm
- net Net-(D3-A): track 0.00 -> 2.87 mm
- net Net-(D2-A): track 0.00 -> 2.87 mm
- net Net-(R3-Pad2): track 0.00 -> 2.79 mm
- net Net-(D1-A): track 0.00 -> 2.77 mm
Other:
- board outline added: 140 x 60 mm

Commit message: BDU
Parts:
- H1, H2, H3, H4, H5, H6: value MountingHole_Pad -> MountingHole; footprint MountingHole:MountingHole_4.3mm_M4_DIN965_Pad -> MountingHole:MountingHole_4.3mm_M4
- J14: value AIR+ -> SDC+
- moved C2 4.65 mm to (169.9, 109.2)
- moved U2 4.65 mm to (166.3, 97.6)
- moved C1 4.65 mm to (169.7, 98.8)
Connections:
- J14 pad 1: SDC+ -> GND
- J15 pad 1: AIR_H- -> GND
- J15 pad 2: AIR_L- -> AIR_H-
- J15 pad 3: PRE- -> AIR_L-
- J15 pad 4: GND -> PRE-
- U1 pad 2: GND -> GNDA
- U1 pad 4: GND -> GNDA
- U1 pad 6: GND -> GNDA
Routing:
- net +12V: track 0.00 -> 20.9 mm
- added copper zone on B.Cu, net GND
- added copper zone on F.Cu, net GND
- added copper zone on B.Cu, net GNDA
- added copper zone on F.Cu, net GNDA
Other:
- outline, holes or cut-outs redrawn

Commit message: BDU
Parts:
- removed J14: SDC+, Connector_Molex:Molex_Micro-Fit_3.0_43650-0210_1x02-1MP_P3.00mm_Horizontal_PnP
- removed J15: AMS, Connector_Molex:Molex_Micro-Fit_3.0_43650-0410_1x04-1MP_P3.00mm_Horizontal_PnP
- added J17: AMS, Connector_Molex:Molex_Micro-Fit_3.0_43650-0410_1x04-1MP_P3.00mm_Horizontal_PnP, F.Cu at (214.8, 90.8)
- moved J3 2.30 mm to (214.4, 111.6)
- moved R4 1.81 mm to (190.2, 110.5), turned to 180 degrees
- moved R2 1.77 mm to (180.0, 110.5), turned to 180 degrees
- moved R5 1.74 mm to (195.2, 110.5), turned to 180 degrees
- moved R3 1.56 mm to (185.0, 110.5), turned to 180 degrees
Routing:
- net SDC+: track 0.00 -> 67.8 mm, vias 0 -> 3
- net +12VA: track 0.00 -> 64.2 mm, vias 0 -> 4
- net AIR_H-: track 0.00 -> 58.9 mm, vias 0 -> 2
- net PRE-: track 0.00 -> 39.5 mm
- net AIR_L-: track 0.00 -> 36.5 mm, vias 0 -> 2
- net +12V: track 20.9 -> 45.5 mm, vias 0 -> 5
- net /pre_aux: track 0.00 -> 21.1 mm
- net /pre_out: track 5.40 -> 24.4 mm
- net /high_aux: track 0.00 -> 18.0 mm
- net /low_aux: track 0.00 -> 12.9 mm
- net /sdc_out: track 0.00 -> 5.50 mm
Other:
- outline, holes or cut-outs redrawn

Commit message: BDU_LVS done
Routing:
- net PRE-: track 39.5 -> 34.2 mm
- net SDC+: track 67.8 -> 66.4 mm, vias 3 -> 0
- net /pre_out: track 24.4 -> 24.0 mm, vias 0 -> 2
Changed lines of the file:
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@@
 			(psa4output no)
 			(plot_black_and_white yes)
+			(plotinvisibletext no)
 			(sketchpadsonfab no)
 			(plotpadnumbers no)
@@
 	)
 	(segment
-		(start 182.9 80.805)
-		(end 182.9 84.15)
-		(width 0.5)
+		(start 191.51 98.135)
+		(end 191.51 95.195)
+		(width 1.2)
 		(layer "F.Cu")
 		(net 7)
 	)
 	(segment
-		(start 191.51 98.135)
-		(end 191.51 95.195)
+		(start 191.51 95.195)
+		(end 191.4675 95.1525)
 		(width 1.2)
 		(layer "F.Cu")
 		(net 7)
 	)
+	(via
+		(at 189.0675 95.1525)
+		(size 1)
+		(drill 0.5)
+		(layers "F.Cu" "B.Cu")
+		(net 7)
+	)
+	(via
+		(at 182.9 80.805)
+		(size 1)
+		(drill 0.5)
+		(layers "F.Cu" "B.Cu")
+		(net 7)
+	)
 	(segment
-		(start 183.5 84.75)
-		(end 187 84.75)
-		(width 0.5)
-		(layer "F.Cu")
+		(start 189.0675 95.1525)
+		(end 187.7 93.785)
+		(width 1.2)
+		(layer "B.Cu")
 		(net 7)
 	)
 	(segment
-		(start 187 84.75)
-		(end 187.75 85.5)
-		(width 0.5)
-		(layer "F.Cu")
+		(start 182.9 82.7)
+		(end 182.9 80.805)
+		(width 1.2)
+		(layer "B.Cu")
 		(net 7)
 	)
 	(segment
-		(start 187.75 85.5)
-		(end 187.75 93.835)
-		(width 0.5)
-		(layer "F.Cu")
+		(start 186.6 83.5)
+		(end 187.7 84.6)
+		(width 1.2)
+		(layer "B.Cu")
 		(net 7)
 	)
 	(segment
-		(start 187.75 93.835)
-		(end 189.0675 95.1525)
-		(width 0.5)
-		(layer "F.Cu")
+		(start 187.7 84.6)
+		(end 187.7 93.785)
+		(width 1.2)
+		(layer "B.Cu")
 		(net 7)
 	)
 	(segment
-		(start 191.51 95.195)
-		(end 191.4675 95.1525)
+		(start 183.7 83.5)
+		(end 182.9 82.7)
 		(width 1.2)
-		(layer "F.Cu")
+		(layer "B.Cu")
 		(net 7)
 	)
 	(segment
-		(start 182.9 84.15)
-		(end 183.5 84.75)
-		(width 0.5)
-		(layer "F.Cu")
+		(start 186.6 83.5)
+		(end 183.7 83.5)
+		(width 1.2)
+		(layer "B.Cu")
 		(net 7)
 	)
 	(segment
-		(start 201.65 107.1)
-		(end 209.28 107.1)
+		(start 209.28 107.1)
+		(end 209.28 104.38)
+		(width 1.2)
+		(layer "F.Cu")
+		(net 8)
+	)
+	(segment
+		(start 205.5 102.8)
+		(end 205.5 93.5)
 		(width 1.2)
 		(layer "F.Cu")
@@
 	(segment
 		(start 205.5 93.5)
-		(end 205.5 104)
+		(end 206.75 92.25)
 		(width 1.2)
 		(layer "F.Cu")
@@
 	)
 	(segment
-		(start 206.75 92.25)
-		(end 205.5 93.5)
+		(start 208.6 103.4)
+		(end 206.1 103.4)
 		(width 1.2)
 		(layer "F.Cu")
@@
 	)
 	(segment
-		(start 204.75 104.75)
-		(end 197.75 104.75)
+		(start 206.1 103.4)
+		(end 205.5 102.8)
 		(width 1.2)
 		(layer "F.Cu")
@@
 	)
 	(segment
-		(start 197.75 104.75)
-		(end 196.59 105.91)
+		(start 196.59 107.665)
+		(end 206.735 107.665)
 		(width 1.2)
 		(layer "F.Cu")
@@
 	)
 	(segment
-		(start 201.085 107.665)
-		(end 201.65 107.1)
+		(start 209.28 104.38)
+		(end 209.3 104.36)
 		(width 1.2)
 		(layer "F.Cu")
@@
 	)
 	(segment
-		(start 196.59 105.91)
-		(end 196.59 107.665)
+		(start 206.735 107.665)
+		(end 207.3 107.1)
 		(width 1.2)
 		(layer "F.Cu")
@@
 	)
 	(segment
-		(start 205.5 104)
-		(end 204.75 104.75)
+		(start 207.3 107.1)
+		(end 209.28 107.1)
 		(width 1.2)
 		(layer "F.Cu")
@@
 	)
 	(segment
-		(start 196.59 107.665)
-		(end 201.085 107.665)
+		(start 206.75 92.25)
+		(end 209.63 92.25)
 		(width 1.2)
 		(layer "F.Cu")
@@
 	)
 	(segment
-		(start 209.63 92.25)
-		(end 206.75 92.25)
+		(start 209.3 104.1)
+		(end 208.6 103.4)
+		(width 1.2)
+		(layer "F.Cu")
+		(net 8)
+	)
+	(segment
+		(start 209.3 104.36)
+		(end 209.3 104.1)
 		(width 1.2)
 		(layer "F.Cu")
@@
 	)
 	(segment
-		(start 176.5 119.28)
-		(end 176.5 120.75)
+		(start 211.75 112.57)
+		(end 209.28 110.1)
 		(width 1.2)
 		(layer "F.Cu")
@@
 	)
 	(segment
-		(start 177.75 122)
-		(end 196.75 122)
+		(start 199.25 121.75)
+		(end 207 121.75)
 		(width 1.2)
 		(layer "F.Cu")
@@
 	)
 	(segment
-		(start 196.75 122)
-		(end 197.7 121.05)
+		(start 207 121.75)
+		(end 211.75 117)
 		(width 1.2)
 		(layer "F.Cu")
@@
 	)
 	(segment
-		(start 197.7 121.05)
-		(end 197.7 119.28)
+		(start 197.7 120.2)
+		(end 199.25 121.75)
 		(width 1.2)
 		(layer "F.Cu")
@@
 		(net 24)
 	)
-	(via
-		(at 209.28 110.1)
-		(size 1)
-		(drill 0.5)
-		(layers "F.Cu" "B.Cu")
-		(net 24)
-	)
-	(via
-		(at 209.63 95.25)
-		(size 1)
-		(drill 0.5)
-		(layers "F.Cu" "B.Cu")
-		(net 24)
-	)
-	(via
-		(at 197.7 119.28)
-		(size 1)
-		(drill 0.5)
-		(layers "F.Cu" "B.Cu")
-		(net 24)
-	)
-	(segment
-		(start 211.75 112.57)
-		(end 209.28 110.1)
-		(width 1.2)
-		(layer "B.Cu")
-		(net 24)
-	)
-	(segment
-		(start 199.25 121.75)
-		(end 207 121.75)
-		(width 1.2)
-		(layer "B.Cu")
-		(net 24)
-	)
-	(segment
-		(start 207 121.75)
-		(end 211.75 117)
-		(width 1.2)
-		(layer "B.Cu")
-		(net 24)
-	)
 	(segment
-		(start 197.7 120.2)
-		(end 199.25 121.75)
+		(start 212 97.62)
+		(end 209.63 95.25)
 		(width 1.2)
-		(layer "B.Cu")
+		(layer "F.Cu")
 		(net 24)
 	)
 	(segment
-		(start 212 97.62)
-		(end 209.63 95.25)
+		(start 177.75 122)
+		(end 195.9 122)
 		(width 1.2)
-		(layer "B.Cu")
+		(layer "F.Cu")
 		(net 24)
 	)
@@
 		(end 197.7 120.2)
 		(width 1.2)
-		(layer "B.Cu")
+		(layer "F.Cu")
 		(net 24)
 	)
@@
 		(end 211.75 112.57)
 		(width 1.2)
-		(layer "B.Cu")
+		(layer "F.Cu")
 		(net 24)
 	)
@@
 		(end 212 107.38)
 		(width 1.2)
-		(layer "B.Cu")
+		(layer "F.Cu")
 		(net 24)
 	)
@@
 		(end 212 97.62)
 		(width 1.2)
-		(layer "B.Cu")
+		(layer "F.Cu")
+		(net 24)
+	)
+	(segment
+		(start 176.5 119.28)
+		(end 176.5 120.75)
+		(width 1.2)
+		(layer "F.Cu")
+		(net 24)
+	)
+	(segment
+		(start 195.9 122)
+		(end 197.7 120.2)
+		(width 1.2)
+		(layer "F.Cu")
 		(net 24)
 	)
@@
 		(polygon
 			(pts
-				(xy 157.5 102.5) (xy 225.25 102.9) (xy 225.25 66.75) (xy 157.5 66.5)
+				(xy 157.5 101.557261) (xy 225.25 101.957261) (xy 225.25 66.75) (xy 157.5 66.5)
 			)
 		)
@@
 		(polygon
 			(pts
-				(xy 157.436279 138.868809) (xy 225.186279 139.268809) (xy 225.186279 103.118809) (xy 157.436279 102.868809)
+				(xy 157.436279 138.868809) (xy 225.186279 139.268809) (xy 225.186279 104.069363) (xy 157.436279 103.819363)
 			)
 		)

Commit message: SSRU new layout
Parts:
- removed C1: 2.2uF, RMC_Capacitor:C_0805_2012Metric_Pad1.18x1.45mm_HandSolder_L
- removed C2: 1uF, RMC_Capacitor:C_0805_2012Metric_Pad1.18x1.45mm_HandSolder_L
- removed D1, D2, D3, D4: LED, RMC_LED:LED_0805_2012Metric_Pad1.45x1.40mm_HandSolder
- removed F10, F2: Fuse, Fuse:Fuseholder_Littelfuse_Nano2_157x
- removed J1, J2, J3: Relay connector, Connector_Molex:Molex_Micro-Fit_3.0_43650-0410_1x04-1MP_P3.00mm_Horizontal_PnP
- removed J10: Voltmeter-, Connector_Molex:Molex_Micro-Fit_3.0_43650-0210_1x02-1MP_P3.00mm_Horizontal_PnP
- removed J11: IMD-, Connector_Molex:Molex_Micro-Fit_3.0_43650-0210_1x02-1MP_P3.00mm_Horizontal_PnP
- removed J12: AIR-, Connector_Molex:Molex_Micro-Fit_3.0_43650-0210_1x02-1MP_P3.00mm_Horizontal_PnP
- removed J13, J8: AIR+, Connector_Molex:Molex_Micro-Fit_3.0_43650-0210_1x02-1MP_P3.00mm_Horizontal_PnP
- removed J16: DCDC, Connector_Molex:Molex_Micro-Fit_3.0_43650-0210_1x02-1MP_P3.00mm_Horizontal_PnP
- removed J17: AMS, Connector_Molex:Molex_Micro-Fit_3.0_43650-0410_1x04-1MP_P3.00mm_Horizontal_PnP
- removed J4: Conn_01x02, Connector_Molex:Molex_Micro-Fit_3.0_43650-0210_1x02-1MP_P3.00mm_Horizontal_PnP
- removed J5: IMD+, Connector_Molex:Molex_Micro-Fit_3.0_43650-0210_1x02-1MP_P3.00mm_Horizontal_PnP
- removed J6: Voltmeter+, Connector_Molex:Molex_Micro-Fit_3.0_43650-0210_1x02-1MP_P3.00mm_Horizontal_PnP
- removed J7: TSAL_green+, Connector_Molex:Molex_Micro-Fit_3.0_43650-0210_1x02-1MP_P3.00mm_Horizontal_PnP
- removed J9: TSAL_green-, Connector_Molex:Molex_Micro-Fit_3.0_43650-0210_1x02-1MP_P3.00mm_Horizontal_PnP
- removed R1: 3K9, Resistor_THT:R_Axial_DIN0207_L6.3mm_D2.5mm_P15.24mm_Horizontal
- removed R10, R11, R12, R13, R2, R3, R4, R5: 1k, RMC_Resistor:R_0805_2012Metric_Pad1.20x1.40mm_HandSolder_L
- removed R6, R7, R8, R9: 4k7, RMC_Resistor:R_0805_2012Metric_Pad1.20x1.40mm_HandSolder_L
- removed U1: LTV-847S, Package_DIP:SMDIP-16_W9.53mm
- removed U2: TRA3-1212, Converter_DCDC:Converter_DCDC_TRACO_TRA3-xxxx_THT
Routing:
- net SDC+: track 66.4 -> 0.00 mm
- net +12VA: track 64.2 -> 0.00 mm, vias 4 -> 0
- net AIR_H-: track 58.9 -> 0.00 mm, vias 2 -> 0
- net +12V: track 45.5 -> 0.00 mm, vias 5 -> 0
- net AIR_L-: track 36.5 -> 0.00 mm, vias 2 -> 0
- net PRE-: track 34.2 -> 0.00 mm
- net /pre_out: track 24.0 -> 0.00 mm, vias 2 -> 0
- net /pre_aux: track 21.1 -> 0.00 mm
- net /high_aux: track 18.0 -> 0.00 mm
- net /low_aux: track 12.9 -> 0.00 mm
- net /low_out: track 5.55 -> 0.00 mm
- net /sdc_out: track 5.50 -> 0.00 mm
- net /high_out: track 5.39 -> 0.00 mm
- net TS+: track 3.00 -> 0.00 mm
- net Net-(R4-Pad2): track 2.92 -> 0.00 mm
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- removed copper zone on B.Cu, net GND
- removed copper zone on F.Cu, net GND
- removed copper zone on B.Cu, net GNDA
- removed copper zone on F.Cu, net GNDA
Other:
- outline, holes or cut-outs redrawn
