File: kicad/SSRU_v3/SSRU_v3/SSRU_v3.kicad_sch (KiCad schematic)
At the start: 85 parts, among them J10 Conn_01x04, J11 Conn_01x02, J20 Conn_01x02, J21 Conn_01x02, J22 Conn_01x04, J24 Conn_01x04, J26 Conn_01x03, J27 Conn_01x03, J3 Conn_01x02, SW1 SW_Push, U1 MCP2515-xSO, U10 TJA1051T, U11 Ai-Thinker-Ra-02, U2 ATmega328P-A, U3 TJA1051T-3, U4 LM2576S-5, U5 AMS1117-3.3, U7 MCP2515-xSO, U7 TJA1051T, U9 MT3608/SDB628, Y1 16MHz, Y3 16MHz, Y4 16MHz

Commit message: Add files via upload
Parts:
- added C45: 22uF, RMC_Capacitor:C_0805_2012Metric_Pad1.18x1.45mm_HandSolder_L, symbol Device:C
- added C46: 0.1uF, RMC_Capacitor:C_0805_2012Metric_Pad1.18x1.45mm_HandSolder_L, symbol Device:C
- renumbered U7 to U12
Connections:
- net +3.3V: now also C45.2, C46.1
- net GND: now also C45.1, C46.2
Other:
- moved on the sheet: C1, C2, C3, C4, J20, U2
