File: kicad/SSRU_v3.1/current to voltage.kicad_sch (KiCad schematic)
At the start: 12 parts, among them J4 Conn_01x02, J5 Conn_01x02, U14 LM2904

Commit message: ssru3.1 pcb edgec ut
Parts:
- removed J4, J5: Conn_01x02, Connector_JST:JST_XH_B2B-XH-A_1x02_P2.50mm_Vertical, symbol Connector_Generic:Conn_01x02
Connections:
- net BRAKE_TEMP1 renamed BRAKE_TEMP_IN1
- net BRAKE_TEMP2 renamed BRAKE_TEMP_IN2

Commit message: SSRU v3.1 updates
Parts:
- removed R30: 5k, RMC_Resistor:R_0805_2012Metric_Pad1.20x1.40mm_HandSolder_L, symbol Device:R
- removed R31: 1k, RMC_Resistor:R_0805_2012Metric_Pad1.20x1.40mm_HandSolder_L, symbol Device:R
- added R32: 1k, RMC_Resistor:R_0805_2012Metric_Pad1.20x1.40mm_HandSolder_L, symbol Device:R
- added R33: 22k, RMC_Resistor:R_0805_2012Metric_Pad1.20x1.40mm_HandSolder_L, symbol Device:R
Connections:
- net BRAKE_TEMP_OUT2: now also R33.2
- net GND: now also R32.1
- net at U14.2 (-): now also R32.2, R33.1
Other:
- moved on the sheet: R25

Commit message: sorry I loved you
Connections:
- net BRAKE_TEMP_IN1: now also R25.2, U14.3 (+); no longer R24.2, U14.5 (+)
- net BRAKE_TEMP_IN2: now also R24.2, U14.5 (+); no longer R25.2, U14.3 (+)
- net BRAKE_TEMP_OUT1: now also C25.1, R33.2, U14.1; no longer C22.1, R28.2, U14.7
- net BRAKE_TEMP_OUT2: now also C22.1, R28.2, U14.7; no longer C25.1, R33.2, U14.1
Other:
- moved on the sheet: C22, C25, R24, R25, R28, R29, R32, R33, U14A, U14B
