File: kicad/SSRU_v3.1/SSRU_v3.1.kicad_sch (KiCad schematic)
At the start: 83 parts, among them J1 AVR-ISP-6, J2 Conn_01x24, J3 Conn_02x03_Odd_Even, J31 Conn_01x04, J6 Conn_02x03_Odd_Even, SW1 SW_Push, U1 MCP2515-xSO, U10 TJA1051T, U11 TCA9517D, U12 TJA1051T, U13 CH340N, U2 ATmega328P-A, U4 LM2576S-5, U5 AMS1117-3.3, U7 MCP2515-xSO, U8 74LVC1G17, U9 MT3608/SDB628, Y1 16MHz, Y3 16MHz, Y4 16MHz

Commit message: ssru3.1 pcb edgec ut
Parts:
- removed C9: 22uF, RMC_Capacitor:C_0805_2012Metric_Pad1.18x1.45mm_HandSolder_L, symbol Device:C_Polarized
- removed H3, H4: MountingHole, MountingHole:MountingHole_3.2mm_M3, symbol Mechanical:MountingHole
- removed J1: AVR-ISP-6, Connector_PinHeader_2.54mm:PinHeader_2x03_P2.54mm_Vertical, symbol Connector:AVR-ISP-6
- removed J6: Conn_02x03_Odd_Even, symbol Connector_Generic:Conn_02x03_Odd_Even
- added C20: 22uF, RMC_Capacitor:C_0805_2012Metric_Pad1.18x1.45mm_HandSolder_L, symbol Device:C_Polarized
- added J1, J5: Conn_01x03, Connector_PinHeader_2.54mm:PinHeader_1x03_P2.54mm_Vertical, symbol Connector_Generic:Conn_01x03
- added J4: AVR-ISP-6, Connector_PinHeader_2.54mm:PinHeader_2x03_P2.54mm_Vertical, symbol Connector:AVR-ISP-6
- added R1, R2, R3, R6, R7, R8: 1M, RMC_Resistor:R_0805_2012Metric_Pad1.20x1.40mm_HandSolder_L, symbol Device:R
- C32, C33: footprint RMC_Capacitor:CP_EIA-3528-15_AVX-H_Pad1.50x2.35mm_HandSolder_RMC -> RMC_Capacitor:C_0805_2012Metric_Pad1.18x1.45mm_HandSolder_L
- J2: footprint (none) -> RMC_Connnector:HD241_24pin
- J3: footprint (none) -> Connector_PinHeader_2.54mm:PinHeader_2x03_P2.54mm_Vertical
- L2: footprint Inductor_SMD:L_Wuerth_HCI-5040 -> RMC_Inductor:L_10.4x10.4_H4.8_handsolder
Connections:
- net +12V: no longer J2.2 (Pin_2)
- net +24V: now also J2.14 (Pin_14)
- net +5V: now also J2.9 (Pin_9), J4.2 (VCC); no longer J2.10 (Pin_10), J2.14 (Pin_14)
- net CAN1+: now also J2.4 (Pin_4), J2.6 (Pin_6); no longer J2.5 (Pin_5), J2.7 (Pin_7)
- net CAN1-: now also J2.3 (Pin_3), J2.5 (Pin_5); no longer J2.4 (Pin_4), J2.6 (Pin_6)
- net CAN2+: now also J2.8 (Pin_8); no longer J2.9 (Pin_9)
- net CAN2-: now also J2.7 (Pin_7); no longer J2.8 (Pin_8)
- net DS18B20: now also J2.13 (Pin_13); no longer J2.16 (Pin_16)
- net ENCODER_A: now also J3.5 (Pin_5), R8.2
- net ENCODER_B: now also J3.6 (Pin_6), R7.2
- net FLOW_IN: now also J3.2 (Pin_2), J5.2 (Pin_2), R3.2; no longer J3.3 (Pin_3), U8.2
- net FLOW_OUT: now also J5.1 (Pin_1)
- net GND: now also J2.2 (Pin_2), C20.2, J1.3 (Pin_3), J4.6 (GND), R1.1, R2.1, R3.1, R6.1, R7.1, R8.1; no longer J2.15 (Pin_15), J2.3 (Pin_3)
- net MISO: now also J4.1 (MISO)
- net MOSI: now also J4.4 (MOSI)
- net POT1_IN: now also J2.10 (Pin_10), R1.2; no longer J2.11 (Pin_11)
- net POT2_IN: now also J2.11 (Pin_11), R2.2; no longer J2.13 (Pin_13)
- net PUMP_NTC_50k: now also R6.2
- net PUMP_PWM: now also J1.1 (Pin_1); no longer J3.5 (Pin_5)
- net RST: now also J4.5 (~{RST})
- net SCK: now also J4.3 (SCK)
- net j1: now also J3.3 (Pin_3); no longer J3.2 (Pin_2)
- net j3: now also J1.2 (Pin_2); no longer J3.6 (Pin_6)
- net at C10.2, F1.2, U5.2 (VO): now also C20.1
- new net: J5.3 (Pin_3), U8.2
- new net BRAKE_TEMP1: J2.15 (Pin_15)
- new net BRAKE_TEMP2: J2.16 (Pin_16)
Other:
- sheet current to voltage ports: added BRAKE_TEMP_IN1, BRAKE_TEMP_IN2; removed none
- moved on the sheet: C19, C30, J3, U8

Commit message: SSRU v3.1 updates
Parts:
- added C9: 10uF, RMC_Capacitor:C_0805_2012Metric_Pad1.18x1.45mm_HandSolder_L, symbol Device:C
- J5: footprint Connector_PinHeader_2.54mm:PinHeader_1x03_P2.54mm_Vertical -> Jumper:SolderJumper-3_P1.3mm_Open_Pad1.0x1.5mm
- L2: footprint RMC_Inductor:L_10.4x10.4_H4.8_handsolder -> Inductor_SMD:L_Sunlord_SWPA5040S
- U11: footprint Package_SO:SOIC-8_3.9x4.9mm_P1.27mm -> RMC_SO:SOIC-8_3.9x4.9mm_P1.27mm_RMC_Handsolder
- U13: footprint Package_SO:SOP-8_3.9x4.9mm_P1.27mm -> RMC_SO:SOIC-8_3.9x4.9mm_P1.27mm_RMC_Handsolder
- Y3, Y4: value 16MHz -> 20MHz
Connections:
- net +24V: now also J2.24 (Pin_24); no longer J2.14 (Pin_14)
- net +3.3V: now also J2.2 (Pin_2); no longer J2.21 (Pin_21)
- net +5V: now also J2.20 (Pin_20), C9.2; no longer J2.12 (Pin_12)
- net BRAKE_TEMP1: now also J2.22 (Pin_22); no longer J2.15 (Pin_15)
- net BRAKE_TEMP2: now also J2.23 (Pin_23); no longer J2.16 (Pin_16)
- net CAN1+: now also J2.14 (Pin_14); no longer J2.4 (Pin_4)
- net CAN1-: now also J2.13 (Pin_13); no longer J2.3 (Pin_3)
- net CAN2+: now also J2.7 (Pin_7); no longer J2.8 (Pin_8)
- net CAN2-: now also J2.15 (Pin_15); no longer J2.7 (Pin_7)
- net DS18B20: now also J2.21 (Pin_21); no longer J2.13 (Pin_13)
- net GND: now also J2.16 (Pin_16), J2.8 (Pin_8), C9.1; no longer J2.2 (Pin_2), J2.22 (Pin_22)
- net POT1_IN: now also J2.18 (Pin_18); no longer J2.10 (Pin_10)
- net POT2_IN: now also J2.19 (Pin_19); no longer J2.11 (Pin_11)
- net SCL_3V3: now also J2.3 (Pin_3); no longer J2.23 (Pin_23)
- net SDA_3V3: now also J2.4 (Pin_4); no longer J2.24 (Pin_24)
- net j1: now also J2.10 (Pin_10); no longer J2.18 (Pin_18)
- net j2: now also J2.11 (Pin_11); no longer J2.19 (Pin_19)
- net j3: now also J2.12 (Pin_12); no longer J2.20 (Pin_20)
Other:
- moved on the sheet: C10, C13, C14, C15, C16, C20, C32, C33, C34, C35, C8, D3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

Commit message: ssruv3.1
Connections:
- net +12V: now also J2.9 (Pin_9)
- net +24V: now also J2.22 (Pin_22); no longer J2.24 (Pin_24)
- net +5V: no longer J2.9 (Pin_9)
- net BRAKE_TEMP1: now also J2.23 (Pin_23); no longer J2.22 (Pin_22)
- net BRAKE_TEMP2: now also J2.24 (Pin_24); no longer J2.23 (Pin_23)
Other:
- added sheet CAN scheme (can.kicad_sch)
Changed lines of the file:
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@@
 	(global_label "BRAKE_TEMP1"
 		(shape input)
-		(at 303.53 82.55 0)
+		(at 303.53 85.09 0)
 		(fields_autoplaced yes)
 		(effects
@@
 		)
 		(property "Intersheetrefs" "${INTERSHEET_REFS}"
-			(at 319.5779 82.55 0)
+			(at 319.5779 85.09 0)
 			(effects
 				(font
@@
 	(global_label "BRAKE_TEMP2"
 		(shape input)
-		(at 303.53 85.09 0)
+		(at 303.53 87.63 0)
 		(fields_autoplaced yes)
 		(effects
@@
 		)
 		(property "Intersheetrefs" "${INTERSHEET_REFS}"
-			(at 319.5779 85.09 0)
+			(at 319.5779 87.63 0)
 			(effects
 				(font
@@
 	(symbol
 		(lib_id "power:+5V")
-		(at 303.53 49.53 270)
-		(mirror x)
-		(unit 1)
-		(exclude_from_sim no)
-		(in_bom yes)
-		(on_board yes)
-		(dnp no)
-		(fields_autoplaced yes)
-		(property "Reference" "#PWR043"
-			(at 299.72 49.53 0)
-			(effects
-				(font
-					(size 1.27 1.27)
-				)
-				(hide yes)
-			)
-		)
-		(property "Value" "+5V"
-			(at 307.34 49.5299 90)
-			(effects
-				(font
-					(size 1.27 1.27)
-				)
-				(justify left)
-			)
-		)
-		(property "Footprint" ""
-			(at 303.53 49.53 0)
-			(effects
-				(font
-					(size 1.27 1.27)
-				)
-				(hide yes)
-			)
-		)
-		(property "Datasheet" ""
-			(at 303.53 49.53 0)
-			(effects
-				(font
-					(size 1.27 1.27)
-				)
-				(hide yes)
-			)
-		)
-		(property "Description" "Power symbol creates a global label with name \"+5V\""
-			(at 303.53 49.53 0)
-			(effects
-				(font
-					(size 1.27 1.27)
-				)
-				(hide yes)
-			)
-		)
-		(pin "1"
-		)
-		(instances
-			(project "SSRU_v3.1"
-				(path "/bee3e03c-9a5f-4c66-913e-823f7b125a2a"
-					(reference "#PWR043")
-					(unit 1)
-				)
-			)
-		)
-	)
-	(symbol
-		(lib_id "power:+5V")
 		(at 350.52 68.58 270)
 		(mirror x)
@@
 	)
 	(symbol
+		(lib_id "power:+12V")
+		(at 303.53 49.53 270)
+		(mirror x)
+		(unit 1)
+		(exclude_from_sim no)
+		(in_bom yes)
+		(on_board yes)
+		(dnp no)
+		(fields_autoplaced yes)
+		(property "Reference" "#PWR029"
+			(at 299.72 49.53 0)
+			(effects
+				(font
+					(size 1.27 1.27)
+				)
+				(hide yes)
+			)
+		)
+		(property "Value" "+12V"
+			(at 307.34 49.5299 90)
+			(effects
+				(font
+					(size 1.27 1.27)
+				)
+				(justify left)
+			)
+		)
+		(property "Footprint" ""
+			(at 303.53 49.53 0)
+			(effects
+				(font
+					(size 1.27 1.27)
+				)
+				(hide yes)
+			)
+		)
+		(property "Datasheet" ""
+			(at 303.53 49.53 0)
+			(effects
+				(font
+					(size 1.27 1.27)
+				)
+				(hide yes)
+			)
+		)
+		(property "Description" "Power symbol creates a global label with name \"+12V\""
+			(at 303.53 49.53 0)
+			(effects
+				(font
+					(size 1.27 1.27)
+				)
+				(hide yes)
+			)
+		)
+		(pin "1"
+		)
+		(instances
+			(project "SSRU_v3.1"
+				(path "/bee3e03c-9a5f-4c66-913e-823f7b125a2a"
+					(reference "#PWR029")
+					(unit 1)
+				)
+			)
+		)
+	)
+	(symbol
 		(lib_id "Device:C")
 		(at 53.34 22.86 0)
@@
 	(symbol
 		(lib_id "power:+24V")
-		(at 303.53 87.63 270)
+		(at 303.53 82.55 270)
 		(mirror x)
 		(unit 1)
@@
 		(fields_autoplaced yes)
 		(property "Reference" "#PWR061"
-			(at 299.72 87.63 0)
+			(at 299.72 82.55 0)
 			(effects
 				(font
@@
 		)
 		(property "Value" "+24V"
-			(at 307.34 87.6299 90)
+			(at 307.34 82.5499 90)
 			(effects
 				(font
@@
 		)
 		(property "Footprint" ""
-			(at 303.53 87.63 0)
+			(at 303.53 82.55 0)
 			(effects
 				(font
@@
 		)
 		(property "Datasheet" ""
-			(at 303.53 87.63 0)
+			(at 303.53 82.55 0)
 			(effects
 				(font
@@
 		)
 		(property "Description" "Power symbol creates a global label with name \"+24V\""
-			(at 303.53 87.63 0)
+			(at 303.53 82.55 0)
 			(effects
 				(font
@@
 				)
 			)
+		)
+	)
+	(sheet
+		(at 354.33 152.4)
+		(size 12.7 3.81)
+		(exclude_from_sim no)
+		(in_bom yes)
+		(on_board yes)
+		(dnp no)
+		(fields_autoplaced yes)
+		(stroke
+			(width 0.1524)
+			(type solid)
+		)
+		(fill
+			(color 0 0 0 0.0000)
+		)
+		(property "Sheetname" "CAN scheme"
+			(at 354.33 151.6884 0)
+			(effects
+				(font
+					(size 1.27 1.27)
+				)
+				(justify left bottom)
+			)
+		)
+		(property "Sheetfile" "can.kicad_sch"
+			(at 354.33 156.7946 0)
+			(effects
+				(font
+					(size 1.27 1.27)
+				)
+				(justify left top)
+			)
+		)
+		(property "Field2" ""
+			(at 354.33 152.4 0)
+			(effects
+				(font
+					(size 1.27 1.27)
+				)
+			)
+		)
+		(instances
+			(project "SSRU_v3.1"
+				(path "/bee3e03c-9a5f-4c66-913e-823f7b125a2a"
+					(page "3")
+				)
+			)

Commit message: ssru
Parts:
- added U3: LM2904, symbol Amplifier_Operational:LM2904
Connections:
- net Temp_sensor is gone; now on net DS18B20: R40.2
- net POT1_IN: now also U3.3 (+); no longer U2.22 (ADC7)
- net POT2_IN: now also U3.5 (+); no longer U2.19 (ADC6)
- new net POT1_OUT: U2.22 (ADC7), U3.1, U3.2 (-)
- new net POT2_OUT: U2.19 (ADC6), U3.6 (-), U3.7
Other:
- moved on the sheet: C19, C30, C31, J5, R1, R2, R3, U8

Commit message: TS scheme update
Parts:
- added C23: 100nF, RMC_Capacitor:C_0805_2012Metric_Pad1.18x1.45mm_HandSolder_L, symbol Device:C
- U3: footprint (none) -> RMC_SO:SOIC-8_3.9x4.9mm_P1.27mm_RMC_Handsolder
Connections:
- net +3.3V: now also J2.5 (Pin_5); no longer J2.2 (Pin_2)
- net +5V: now also U3.4 (V-), C23.2
- net CAN1+: now also J2.11 (Pin_11), J2.3 (Pin_3); no longer J2.14 (Pin_14), J2.6 (Pin_6)
- net CAN1-: now also J2.10 (Pin_10), J2.2 (Pin_2); no longer J2.13 (Pin_13), J2.5 (Pin_5)
- net CAN2+: now also J2.19 (Pin_19); no longer J2.7 (Pin_7)
- net CAN2-: now also J2.18 (Pin_18); no longer J2.15 (Pin_15)
- net GND: now also U3.8 (V+), C23.1
- net POT1_IN: now also J2.4 (Pin_4); no longer J2.18 (Pin_18)
- net POT2_IN: now also J2.12 (Pin_12); no longer J2.19 (Pin_19)
- net SCL_3V3: now also J2.6 (Pin_6); no longer J2.3 (Pin_3)
- net SDA_3V3: now also J2.7 (Pin_7); no longer J2.4 (Pin_4)
- net j1: now also J2.13 (Pin_13); no longer J2.10 (Pin_10)
- net j2: now also J2.14 (Pin_14); no longer J2.11 (Pin_11)
- net j3: now also J2.15 (Pin_15); no longer J2.12 (Pin_12)
Other:
- moved on the sheet: U3C

Commit message: SSRU
Parts:
- removed H1, H2: MountingHole, MountingHole:MountingHole_3.2mm_M3, symbol Mechanical:MountingHole
- added C24, C29: 100nF, RMC_Capacitor:C_0805_2012Metric_Pad1.18x1.45mm_HandSolder_L, symbol Device:C
- added H1, H2: MountingHole_Pad, MountingHole:MountingHole_3.2mm_M3_ISO14580_Pad, symbol Mechanical:MountingHole_Pad
- added R10, R9: 1M, RMC_Resistor:R_0805_2012Metric_Pad1.20x1.40mm_HandSolder_L, symbol Device:R
Connections:
- net CS_CAN1: now also U2.14 (PB2); no longer U2.12 (PB0)
- net GND: now also C24.1, C29.1, R10.1, R9.1
- net 328_RX renamed 328+
- net 328_TX renamed 328-
- new net Earth: C24.2, C29.2, H1.1, H2.1, R10.2, R9.2

Commit message: sorry I loved you
Connections:
- net CAN1+: now also J2.19 (Pin_19); no longer J2.3 (Pin_3)
- net CAN1-: now also J2.18 (Pin_18); no longer J2.2 (Pin_2)
- net CAN2+: now also J2.3 (Pin_3); no longer J2.19 (Pin_19)
- net CAN2-: now also J2.2 (Pin_2); no longer J2.18 (Pin_18)
- net DS18B20: now also U2.12 (PB0); no longer U2.11 (PD7)
- net SCL renamed I2C+
- net SDA renamed I2C-

Commit message: gerbers
Connections:
- net ENCODER_A renamed ENCODER+
- net ENCODER_B renamed ENCODER-
Changed lines of the file:
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@@
+		)
+	)
+	(global_label "ENCODER-"
+		(shape input)
+		(at 40.64 88.9 0)
+		(fields_autoplaced yes)
+		(effects
+			(font
+				(size 1.27 1.27)
+			)
+			(justify left)
+		)
+		(property "Intersheetrefs" "${INTERSHEET_REFS}"
+			(at 53.9666 88.9 0)
+			(effects
+				(font
+					(size 1.27 1.27)
+				)
+				(justify left)
+				(hide yes)
+			)
 		)
 	)
@@
 		)
 	)
+	(global_label "ENCODER_A"
+		(shape input)
+		(at 40.64 86.36 180)
+		(fields_autoplaced yes)
+		(effects
+			(font
+				(size 1.27 1.27)
+			)
+			(justify right)
+		)
+		(property "Intersheetrefs" "${INTERSHEET_REFS}"
+			(at 26.8296 86.36 0)
+			(effects
+				(font
+					(size 1.27 1.27)
+				)
+				(justify right)
+				(hide yes)
+			)
+		)
+	)
 	(global_label "ENCODER_B"
 		(shape input)
@@
 		)
 	)
+	(global_label "ENCODER_B"
+		(shape input)
+		(at 40.64 88.9 180)
+		(fields_autoplaced yes)
+		(effects
+			(font
+				(size 1.27 1.27)
+			)
+			(justify right)
+		)
+		(property "Intersheetrefs" "${INTERSHEET_REFS}"
+			(at 26.6482 88.9 0)
+			(effects
+				(font
+					(size 1.27 1.27)
+				)
+				(justify right)
+				(hide yes)
+			)
+		)
+	)
 	(global_label "CANH_2"
 		(shape input)
@@
 			(effects
 				(font
+					(size 1.27 1.27)
+				)
+				(justify left)
+				(hide yes)
+			)
+		)
+	)
+	(global_label "ENCODER+"
+		(shape input)
+		(at 40.64 86.36 0)
+		(fields_autoplaced yes)
+		(effects
+			(font
+				(size 1.27 1.27)
+			)
+			(justify left)
+		)
+		(property "Intersheetrefs" "${INTERSHEET_REFS}"
+			(at 53.9666 86.36 0)
+			(effects
+				(font
