File: kicad/TS schematics/TSAC.kicad_sch (KiCad schematic)
At the start: 5 parts, among them J3 TE HVP800

Commit message: TS schematics
Parts:
- removed J3: TE HVP800, symbol Connector_Generic:Conn_01x02
- added J18: Amphenol PL00Y-301-10M8, symbol Connector_Generic:Conn_01x01
- added J19: TSAL voltage detection, symbol Connector_Generic:Conn_01x02
- added J20: Bender Isometer IR155-3203, symbol Connector_Generic:Conn_01x02
- added J21: KLclear BMS, symbol Connector_Generic:Conn_01x03
- added J3: Amphenol PL00x-301-10M8, symbol Connector_Generic:Conn_01x01
Connections:
- net TS+: now also J3.1 (Pin_1)
- net TS-: now also J18.1 (Pin_1), J19.1 (Pin_1), J20.1 (Pin_1), J21.1 (Pin_1)
- net at Fuse.2, Fuse1.2: now also J19.2 (Pin_2), J20.2 (Pin_2), J21.3 (Pin_3)
- net at precharge_resistor.2: now also J21.2 (Pin_2)
Other:
- note added: "Voltage detection for 2P in series at each battery pack through Micro-Fit 3.0 22p connector"
