File: kicad/TS schematics/TSAC.kicad_sch (KiCad schematic)
At the start: 9 parts, among them J18 Amphenol PL00Y-301-10M8, J19 TSAL voltage detection, J20 Bender Isometer IR155-3203, J21 KLclear BMS, J3 Amphenol PL00x-301-10M8

Commit message: haha VCU V3.2 AND NEW SCHEMATICS HAHAHA
Parts:
- removed J19: TSAL voltage detection, symbol Connector_Generic:Conn_01x02
- added J32: TSAL, symbol Connector_Generic:Conn_01x03
Connections:
- net TS-: now also J32.1 (Pin_1)
- net at Fuse.2, Fuse1.2, J20.2 (Pin_2)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: now also J32.2 (Pin_2)
- new net TSALight_Green: J32.3 (Pin_3)
Changed lines of the file:
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@@
+		)
+	)
+	(hierarchical_label "TSALight_Green"
+		(shape input)
+		(at 170.18 77.47 180)
+		(effects
+			(font
+				(size 1.27 1.27)
+			)
+			(justify right)
 		)
 	)
@@
 	)
 	(symbol
-		(lib_id "Connector_Generic:Conn_01x02")
-		(at 175.26 72.39 0)
+		(lib_id "Connector_Generic:Conn_01x03")
+		(at 175.26 74.93 0)
 		(unit 1)
 		(exclude_from_sim no)
@@
 		(dnp no)
 		(fields_autoplaced yes)
-		(property "Reference" "J19"
-			(at 177.8 72.3899 0)
-			(effects
-				(font
-					(size 1.27 1.27)
-				)
-				(justify left)
-			)
-		)
-		(property "Value" "TSAL voltage detection"
-			(at 177.8 74.9299 0)
-			(effects
-				(font
-					(size 1.27 1.27)
-				)
-				(justify left)
-			)
-		)
-		(property "Footprint" ""
-			(at 175.26 72.39 0)
-			(effects
-				(font
-					(size 1.27 1.27)
-				)
-				(hide yes)
-			)
-		)
-		(property "Datasheet" "~"
-			(at 175.26 72.39 0)
-			(effects
-				(font
-					(size 1.27 1.27)
-				)
-				(hide yes)
-			)
-		)
-		(property "Description" "Generic connector, single row, 01x02, script generated (kicad-library-utils/schlib/autogen/connector/)"
-			(at 175.26 72.39 0)
-			(effects
-				(font
-					(size 1.27 1.27)
-				)
-				(hide yes)
-			)
-		)
-		(pin "1"
+		(property "Reference" "J32"
+			(at 177.8 73.6599 0)
+			(effects
+				(font
+					(size 1.27 1.27)
+				)
+				(justify left)
+			)
+		)
+		(property "Value" "TSAL"
+			(at 177.8 76.1999 0)
+			(effects
+				(font
+					(size 1.27 1.27)
+				)
+				(justify left)
+			)
+		)
+		(property "Footprint" ""
+			(at 175.26 74.93 0)
+			(effects
+				(font
+					(size 1.27 1.27)
+				)
+				(hide yes)
+			)
+		)
+		(property "Datasheet" "~"
+			(at 175.26 74.93 0)
+			(effects
+				(font
+					(size 1.27 1.27)
+				)
+				(hide yes)
+			)
+		)
+		(property "Description" "Generic connector, single row, 01x03, script generated (kicad-library-utils/schlib/autogen/connector/)"
+			(at 175.26 74.93 0)
+			(effects
+				(font
+					(size 1.27 1.27)
+				)
+				(hide yes)
+			)
 		)
 		(pin "2"
 		)
-		(instances
-			(project ""
-				(path "/55cbadab-af07-45b3-b9ce-9748abc6dcd0/ba531de5-0225-4458-93d2-6539cce2b96a"
-					(reference "J19")
-					(unit 1)
-				)
+		(pin "1"
+		)
+		(pin "3"
+		)
+		(instances
+			(project "TS schematics"
+				(path "/55cbadab-af07-45b3-b9ce-9748abc6dcd0/ba531de5-0225-4458-93d2-6539cce2b96a"
+					(reference "J32")
+					(unit 1)
+				)
