File: kicad/TS schematics/TS schematics.kicad_sch (KiCad schematic)
At the start: 13 parts, among them J1 Conn_01x05, J2 TSAL_R, J4 TSMP, K1 DISCHARGE RELAY GIGAVAC PNC11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

Commit message: bunch of schemes
Other:
- added sheet accumulator (TSAC.kicad_sch)
- note added: "Alpha Wire Eco Wire Series 6712 0.2mm^2"
- note added: "Copper Bus Bar Custom made 20mm^2"
- note added: "Ningbo KBE FHL2G 25mm^2"
Changed lines of the file:
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@@
+		)
+	)
+	(text "Copper Bus Bar	Custom made	20mm^2"
+		(exclude_from_sim no)
+		(at 120.396 122.428 0)
+		(effects
+			(font
+				(size 1.27 1.27)
+			)
+		)
+	)
+	(text "Alpha Wire	Eco Wire Series 6712	0.2mm^2"
+		(exclude_from_sim no)
+		(at 60.706 130.048 0)
+		(effects
+			(font
+				(size 1.27 1.27)
+			)
+		)
+	)
+	(text "Ningbo	KBE FHL2G	25mm^2"
+		(exclude_from_sim no)
+		(at 147.574 115.57 0)
+		(effects
+			(font
+				(size 1.27 1.27)
+			)
 		)
 	)
@@
 				(size 5 5)
 				(thickness 0.625)
+			)
+		)
+	)
+	(text "Ningbo	KBE FHL2G	25mm^2"
+		(exclude_from_sim no)
+		(at 166.624 73.914 0)
+		(effects
+			(font
+				(size 1.27 1.27)
 			)
 		)
@@
 				)
 			)
+		)
+	)
+	(sheet
+		(at 182.88 100.33)
+		(size 13.97 6.35)
+		(exclude_from_sim no)
+		(in_bom yes)
+		(on_board yes)
+		(dnp no)
+		(fields_autoplaced yes)
+		(stroke
+			(width 0.1524)
+			(type solid)
+		)
+		(fill
+			(color 0 0 0 0.0000)
+		)
+		(property "Sheetname" "accumulator"
+			(at 182.88 99.6184 0)
+			(effects
+				(font
+					(size 1.27 1.27)
+				)
+				(justify left bottom)
+			)
+		)
+		(property "Sheetfile" "TSAC.kicad_sch"
+			(at 182.88 107.2646 0)
+			(effects
+				(font
+					(size 1.27 1.27)
+				)
+				(justify left top)
+			)
+		)
+		(instances
+			(project "TS schematics"
+				(path "/55cbadab-af07-45b3-b9ce-9748abc6dcd0"
+					(page "2")
+				)
+			)

Commit message: new schematics
Parts:
- added BT1, BT2, BT3: Battery_Cell, symbol Device:Battery_Cell
- added F2: 10A fuse, symbol Device:Fuse_Small
- added F3: 50A fuse, symbol Device:Fuse_Small
- added F4: 15A fuse, symbol Device:Fuse_Small
- added J10: DT 3 pin, symbol Connector_Generic:Conn_01x03
- added J11, J13: Conn_01x04, symbol Connector_Generic:Conn_01x04
- added J12: SDC_END DT2, symbol Connector_Generic:Conn_01x02
- added J14: 紅色儲能接綫柱100A, symbol Connector_Generic:Conn_01x01
- added J15: 黑色儲能接綫柱100A, symbol Connector_Generic:Conn_01x01
- added J5: DT 2 pin, symbol Connector_Generic:Conn_01x02
- added J6: WS16-5, symbol Connector_Generic:Conn_01x05
- added J7: Conn_01x12, symbol Connector_Generic:Conn_01x12
- added J8: DALY K40 BMS, symbol Connector_Generic:Conn_01x06
- added U1: dumb ass dcdc 15V8A 120W, Converter_DCDC:Converter_DCDC_TRACO_TDN_5-xxxxWISM_SMD, symbol Regulator_Switching:TDN_5-0910WISM
- added U2: CCCV 300W, Package_TO_SOT_THT:TO-220-5_Vertical, symbol Regulator_Switching:LM2575-12BT
Connections:
- net GND: now also BT3.2 (-), J10.3 (Pin_3), J11.4 (Pin_4), J12.2 (Pin_2), J13.1 (Pin_1), J15.1 (Pin_1), J5.2 (Pin_2), J6.5 (Pin_5), J7.3 (Pin_3), J7.4 (Pin_4), J8.4 (Pin_4), U1.6 (-VOUT), U2.3 (GND)
- net MCU+: now also U1.1 (+VIN)
- net SDC+: now also J12.1 (Pin_1), J7.7 (Pin_7)
- net TS-: now also U1.2 (-VIN)
- net at J4.1 (Pin_1), R1.1: now also J6.1 (Pin_1)
- net at J4.2 (Pin_2), R2.1: now also J6.2 (Pin_2)
- new net: BT1.2 (-), BT2.1 (+), J8.2 (Pin_2)
- new net: BT2.2 (-), BT3.1 (+), J8.3 (Pin_3)
- new net: F4.1, U2.2 (OUT)
- new net: F2.2, U1.7 (+VOUT)
- new net: BT1.1 (+), F3.1, J8.1 (Pin_1)
- new net +12V: F3.2, F4.2, J11.1 (Pin_1), J13.4 (Pin_4), J14.1 (Pin_1), J7.5 (Pin_5), J7.6 (Pin_6)
- new net +15V: F2.1, J5.1 (Pin_1), J7.1 (Pin_1), J7.2 (Pin_2), U2.1 (VIN)
- new net AMS_CANH: J7.8 (Pin_8)
- new net AMS_CANL: J7.9 (Pin_9)
- new net AMS_LIGHT: J7.10 (Pin_10)
- new net CAN_H: J10.1 (Pin_1), J8.5 (Pin_5)
- new net CAN_L: J10.2 (Pin_2), J8.6 (Pin_6)
- new net FS_CAN_H: J13.3 (Pin_3)
- new net FS_CAN_L: J13.2 (Pin_2)
- new net IMD_LIGHT: J7.11 (Pin_11)
- new net SDC_in: J11.2 (Pin_2)
- new net TSAL_G: J7.12 (Pin_12)
- new net TSAL_R: J11.3 (Pin_3)
- new net interlock: J6.3 (Pin_3), J6.4 (Pin_4)
Other:
- note added: "LVB"
- note added: "RING CRIMP"

Commit message: ts SCHEME AND SSRU
Parts:
- J11, J13: value Conn_01x04 -> DT 04
- J12: value SDC_END DT2 -> DT-02
- J7: value Conn_01x12 -> dt12
Connections:
- net +12V: no longer J7.6 (Pin_6)
- net SDC+: no longer J12.1 (Pin_1), K1.A1
- net SDC_in renamed SDC_Relay
- net SDC_Relay: now also J7.6 (Pin_6), K1.A1
- new net TSMS_SDC: J12.1 (Pin_1)

Commit message: ssru
Parts:
- removed J6: WS16-5, symbol Connector_Generic:Conn_01x05
- removed J7: dt12, symbol Connector_Generic:Conn_01x12
- added J6: amphenol, symbol Connector_Generic:Conn_01x04
- added J7: Conn_01x19, symbol Connector_Generic:Conn_01x19
Connections:
- net +12V: now also J7.5 (Pin_5)
- net +15V: now also J7.1 (Pin_1), J7.2 (Pin_2)
- net AMS_LIGHT: now also J7.10 (Pin_10)
- net GND: now also J7.16 (Pin_16), J7.3 (Pin_3), J7.4 (Pin_4)
- net IMD_LIGHT: now also J7.11 (Pin_11)
- net SDC+: now also J7.7 (Pin_7)
- net SDC_Relay: now also J7.6 (Pin_6)
- net TSAL_G: now also J7.12 (Pin_12)
- net interlock: now also J6.3 (Pin_3), J6.4 (Pin_4)
- net at J4.1 (Pin_1), R1.1: now also J6.1 (Pin_1)
- net at J4.2 (Pin_2), R2.1: now also J6.2 (Pin_2)
- new net +5V: J7.15 (Pin_15)
- new net AMS_CANH_1: J7.8 (Pin_8)
- new net AMS_CANH_2: J7.13 (Pin_13)
- new net AMS_CANL_1: J7.9 (Pin_9)
- new net AMS_CANL_2: J7.14 (Pin_14)

Commit message: TS scheme update
Parts:
- removed AC, HVbox: TE connectivity HVP800 2pcs Connector, symbol Connector_Generic:Conn_01x02
- removed J10: DT 3 pin, symbol Connector_Generic:Conn_01x03
- removed J12: DT-02, symbol Connector_Generic:Conn_01x02
- added J10, J17: Amphenol PL00Y-301-10M8, symbol Connector_Generic:Conn_01x01
- added J12, J16: Amphenol PL00X-301-10M8, symbol Connector_Generic:Conn_01x01
- added J9: Amphenol RT0W0106PN03, symbol Connector_Generic:Conn_01x06
- J11: value DT 04 -> Amphenol RT00104PN03
- J13: value DT 04 -> DT04
- J5: value DT 2 pin -> Amphenol RT00122PM03
- J6: value amphenol -> Amphenol RT00122PM03
- J7: value Conn_01x19 -> Amphenol RT001619PNH
Connections:
- net +12V: now also J7.6 (Pin_6), J9.5 (Pin_5); no longer J11.1 (Pin_1)
- net +5V: now also J7.16 (Pin_16); no longer J7.15 (Pin_15)
- net AMS_CANH_1: now also J7.13 (Pin_13); no longer J7.8 (Pin_8)
- net AMS_CANH_2: now also J7.18 (Pin_18); no longer J7.13 (Pin_13)
- net AMS_CANL_1: now also J7.14 (Pin_14); no longer J7.9 (Pin_9)
- net AMS_CANL_2: now also J7.19 (Pin_19); no longer J7.14 (Pin_14)
- net AMS_LIGHT: now also J7.15 (Pin_15); no longer J7.10 (Pin_10)
- net CAN_H: now also J11.1 (Pin_1)
- net CAN_L: now also J11.2 (Pin_2)
- net GND: now also J11.3 (Pin_3), J7.17 (Pin_17), J7.8 (Pin_8), J7.9 (Pin_9), J9.2 (Pin_2), J9.6 (Pin_6); no longer J7.16 (Pin_16)
- net IMD_LIGHT: now also J7.7 (Pin_7); no longer J7.11 (Pin_11)
- net MCU+: now also J12.1 (Pin_1), J16.1 (Pin_1)
- net SDC+: now also J7.12 (Pin_12); no longer J7.7 (Pin_7)
- net SDC_Relay: now also J7.11 (Pin_11), J9.4 (Pin_4); no longer J11.2 (Pin_2), J7.6 (Pin_6)
- net TS-: now also J10.1 (Pin_1), J17.1 (Pin_1)
- net TSAL_G: now also J7.10 (Pin_10); no longer J7.12 (Pin_12)
- net TSAL_R: now also J9.1 (Pin_1); no longer J11.3 (Pin_3)
- net TSMS_SDC: now also J9.3 (Pin_3)
Other:
- note added: "AMS DISPLAY"
- note added: "Minzan EVRP 50mm^{2}"
- note added: "PL28X-301-50"
- note added: "PL28Y-301-50"

Commit message: TS schematics
Other:
- added sheet Shutdown Circuit (sdc.kicad_sch)
Changed lines of the file:
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@@
+	)
+	(sheet
+		(at 208.28 67.945)
+		(size 32.385 12.7)
+		(exclude_from_sim no)
+		(in_bom yes)
+		(on_board yes)
+		(dnp no)
+		(fields_autoplaced yes)
+		(stroke
+			(width 0.1524)
+			(type solid)
+		)
+		(fill
+			(color 0 0 0 0.0000)
+		)
+		(property "Sheetname" "Shutdown Circuit"
+			(at 208.28 67.2334 0)
+			(effects
+				(font
+					(size 1.27 1.27)
+				)
+				(justify left bottom)
+			)
+		)
+		(property "Sheetfile" "sdc.kicad_sch"
+			(at 208.28 81.2296 0)
+			(effects
+				(font
+					(size 1.27 1.27)
+				)
+				(justify left top)
+			)
+		)
+		(instances
+			(project "TS schematics"
+				(path "/55cbadab-af07-45b3-b9ce-9748abc6dcd0"
+					(page "3")
+				)
+			)
+		)
 	)
 	(sheet

Commit message: gerbers
Parts:
- added J23: DT03, symbol Connector_Generic:Conn_01x03
Connections:
- net +5V: now also J23.3 (Pin_3)
- net GND: now also J23.1 (Pin_1)
- new net HALL CURRENT: J23.2 (Pin_2)
Changed lines of the file:
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@@
 		)
 	)
+	(global_label "HALL CURRENT"
+		(shape input)
+		(at 55.88 33.02 0)
+		(fields_autoplaced yes)
+		(effects
+			(font
+				(size 1.27 1.27)
+			)
+			(justify left)
+		)
+		(property "Intersheetrefs" "${INTERSHEET_REFS}"
+			(at 72.8957 33.02 0)
+			(effects
+				(font
+					(size 1.27 1.27)
+				)
+				(justify left)
+				(hide yes)
+			)
+		)
+	)
 	(global_label "AMS_CANL_1"
 		(shape input)
@@
 	)
 	(symbol
+		(lib_id "Connector_Generic:Conn_01x03")
+		(at 50.8 33.02 0)
+		(mirror y)
+		(unit 1)
+		(exclude_from_sim no)
+		(in_bom yes)
+		(on_board yes)
+		(dnp no)
+		(fields_autoplaced yes)
+		(property "Reference" "J23"
+			(at 50.8 24.13 0)
+			(effects
+				(font
+					(size 1.27 1.27)
+				)
+			)
+		)
+		(property "Value" "DT03"
+			(at 50.8 26.67 0)
+			(effects
+				(font
+					(size 1.27 1.27)
+				)
+			)
+		)
+		(property "Footprint" ""
+			(at 50.8 33.02 0)
+			(effects
+				(font
+					(size 1.27 1.27)
+				)
+				(hide yes)
+			)
+		)
+		(property "Datasheet" "~"
+			(at 50.8 33.02 0)
+			(effects
+				(font
+					(size 1.27 1.27)
+				)
+				(hide yes)
+			)
+		)
+		(property "Description" "Generic connector, single row, 01x03, script generated (kicad-library-utils/schlib/autogen/connector/)"
+			(at 50.8 33.02 0)
+			(effects
+				(font
+					(size 1.27 1.27)
+				)
+				(hide yes)
+			)
+		)
+		(pin "1"
+		)
+		(pin "2"
+		)
+		(pin "3"
+		)
+		(instances
+			(project ""
+				(path "/55cbadab-af07-45b3-b9ce-9748abc6dcd0"
+					(reference "J23")
+					(unit 1)
+				)
+			)
+		)
+	)
+	(symbol
 		(lib_id "Device:Fuse_Small")
 		(at 179.07 127 0)
@@
 	)
 	(symbol
+		(lib_id "power:GND")
+		(at 55.88 30.48 90)
+		(unit 1)
+		(exclude_from_sim no)
+		(in_bom yes)
+		(on_board yes)
+		(dnp no)
+		(fields_autoplaced yes)
+		(property "Reference" "#PWR033"
+			(at 62.23 30.48 0)
+			(effects
+				(font
+					(size 1.27 1.27)
+				)
+				(hide yes)
+			)
+		)
+		(property "Value" "GND"
+			(at 59.69 30.4799 90)
+			(effects
+				(font
+					(size 1.27 1.27)
+				)
+				(justify right)
+			)
+		)
+		(property "Footprint" ""
+			(at 55.88 30.48 0)
+			(effects
+				(font
+					(size 1.27 1.27)
+				)
+				(hide yes)
+			)
+		)
+		(property "Datasheet" ""
+			(at 55.88 30.48 0)
+			(effects
+				(font
+					(size 1.27 1.27)
+				)
+				(hide yes)
+			)
+		)
+		(property "Description" "Power symbol creates a global label with name \"GND\" , ground"
+			(at 55.88 30.48 0)
+			(effects
+				(font
+					(size 1.27 1.27)
+				)
+				(hide yes)
+			)
+		)
+		(pin "1"
+		)
+		(instances
+			(project ""
+				(path "/55cbadab-af07-45b3-b9ce-9748abc6dcd0"
+					(reference "#PWR033")
+					(unit 1)
+				)
+			)
+		)
+	)
+	(symbol
 		(lib_id "Connector_Generic:Conn_01x04")
 		(at 15.24 120.65 0)
@@
 					(unit 1)
 				)
+			)
+		)
+	)
+	(symbol
+		(lib_id "power:+5V")
+		(at 55.88 35.56 270)
+		(unit 1)
+		(exclude_from_sim no)
+		(in_bom yes)
+		(on_board yes)
+		(dnp no)
+		(fields_autoplaced yes)
+		(property "Reference" "#PWR032"
+			(at 52.07 35.56 0)
+			(effects
+				(font
+					(size 1.27 1.27)
+				)
+				(hide yes)
+			)
+		)
+		(property "Value" "+5V"
+			(at 59.69 35.5599 90)
+			(effects
+				(font
+					(size 1.27 1.27)
+				)
+				(justify left)
+			)
+		)
+		(property "Footprint" ""
+			(at 55.88 35.56 0)
+			(effects
+				(font
+					(size 1.27 1.27)
+				)
+				(hide yes)
+			)
+		)
+		(property "Datasheet" ""
+			(at 55.88 35.56 0)
+			(effects
+				(font
+					(size 1.27 1.27)
+				)
+				(hide yes)
+			)
+		)
+		(property "Description" "Power symbol creates a global label with name \"+5V\""
+			(at 55.88 35.56 0)
+			(effects
+				(font
+					(size 1.27 1.27)
+				)
+				(hide yes)
+			)
+		)
+		(pin "1"
+		)
+		(instances
+			(project ""
+				(path "/55cbadab-af07-45b3-b9ce-9748abc6dcd0"
+					(reference "#PWR032")
+					(unit 1)
+				)

Commit message: schematics
Parts:
- added J24: Conn_01x02, symbol Connector_Generic:Conn_01x02
Connections:
- net MCU+: now also J24.2 (Pin_2)
- net MCU-: now also J24.1 (Pin_1)
Other:
- note added: "Copper Bus Bar Custom made 60mm^2"
- note removed: "Copper Bus Bar Custom made 20mm^2"
Changed lines of the file:
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@@
 		)
 	)
-	(text "Copper Bus Bar	Custom made	20mm^2"
+	(text "Copper Bus Bar	Custom made	60mm^2"
 		(exclude_from_sim no)
 		(at 120.396 122.428 0)
@@
 	)
 	(junction
-		(at 130.81 95.25)
-		(diameter 0)
-		(color 0 0 0 0)
-	)
-	(junction
 		(at 35.56 171.45)
 		(diameter 0)
@@
 	)
 	(junction
+		(at 133.35 95.25)
+		(diameter 0)
+		(color 0 0 0 0)
+	)
+	(junction
 		(at 33.02 118.11)
 		(diameter 0)
@@
 	)
 	(junction
+		(at 133.35 100.33)
+		(diameter 0)
+		(color 0 0 0 0)
+	)
+	(junction
 		(at 87.63 100.33)
 		(diameter 0)
@@
 	)
 	(junction
-		(at 35.56 163.83)
+		(at 133.35 102.87)
 		(diameter 0)
 		(color 0 0 0 0)
 	)
 	(junction
-		(at 133.35 97.79)
+		(at 35.56 163.83)
 		(diameter 0)
 		(color 0 0 0 0)
@@
 		(color 0 0 0 0)
 	)
+	(junction
+		(at 138.43 102.87)
+		(diameter 0)
+		(color 0 0 0 0)
+	)
 	(wire
 		(pts
@@
 	(wire
 		(pts
+			(xy 133.35 100.33) (xy 133.35 95.25)
+		)
+		(stroke
+			(width 0)
+			(type default)
+		)
+	)
+	(wire
+		(pts
 			(xy 59.69 127) (xy 60.96 127)
 		)
@@
 	(wire
 		(pts
+			(xy 133.35 102.87) (xy 133.35 106.68)
+		)
+		(stroke
+			(width 0)
+			(type default)
+		)
+	)
+	(wire
+		(pts
 			(xy 50.8 156.21) (xy 50.8 154.94)
 		)
@@
 	(wire
 		(pts
-			(xy 133.35 68.58) (xy 147.32 68.58)
+			(xy 133.35 68.58) (xy 144.78 68.58)
 		)
 		(stroke
@@
 	(wire
 		(pts
+			(xy 133.35 100.33) (xy 144.78 100.33)
+		)
+		(stroke
+			(width 0)
+			(type default)
+		)
+	)
+	(wire
+		(pts
 			(xy 67.31 162.56) (xy 55.88 162.56)
 		)
@@
 	(wire
 		(pts
-			(xy 130.81 95.25) (xy 147.32 95.25)
+			(xy 114.3 124.46) (xy 95.25 124.46)
 		)
 		(stroke
@@
 	(wire
 		(pts
-			(xy 114.3 124.46) (xy 95.25 124.46)
+			(xy 53.34 171.45) (xy 53.34 160.02)
 		)
 		(stroke
@@
 	(wire
 		(pts
-			(xy 133.35 97.79) (xy 149.86 97.79)
+			(xy 116.84 124.46) (xy 116.84 106.68)
 		)
 		(stroke
@@
 	(wire
 		(pts
-			(xy 53.34 171.45) (xy 53.34 160.02)
+			(xy 138.43 90.17) (xy 138.43 102.87)
 		)
 		(stroke
@@
 	(wire
 		(pts
-			(xy 116.84 124.46) (xy 116.84 106.68)
+			(xy 144.78 68.58) (xy 144.78 100.33)
 		)
 		(stroke
@@
 	(wire
 		(pts
-			(xy 90.17 92.71) (xy 130.81 92.71)
+			(xy 90.17 92.71) (xy 133.35 92.71)
 		)
 		(stroke
@@
 	(wire
 		(pts
-			(xy 92.71 95.25) (xy 130.81 95.25)
+			(xy 92.71 95.25) (xy 133.35 95.25)
 		)
 		(stroke
@@
 	(wire
 		(pts
-			(xy 147.32 95.25) (xy 147.32 68.58)
+			(xy 59.69 127) (xy 59.69 123.19)
 		)
 		(stroke
@@
 	(wire
 		(pts
-			(xy 59.69 127) (xy 59.69 123.19)
+			(xy 35.56 171.45) (xy 53.34 171.45)
 		)
 		(stroke
@@
 	(wire
 		(pts
-			(xy 35.56 171.45) (xy 53.34 171.45)
+			(xy 138.43 102.87) (xy 152.4 102.87)
 		)
 		(stroke
@@
 	(wire
 		(pts
-			(xy 149.86 97.79) (xy 149.86 66.04)
+			(xy 152.4 66.04) (xy 152.4 102.87)
 		)
 		(stroke
@@
 	(wire
 		(pts
-			(xy 68.58 118.11) (xy 87.63 118.11)
+			(xy 138.43 102.87) (xy 133.35 102.87)
 		)
 		(stroke
@@
 	(wire
 		(pts
-			(xy 133.35 106.68) (xy 133.35 97.79)
+			(xy 68.58 118.11) (xy 87.63 118.11)
 		)
 		(stroke
@@
 	(wire
 		(pts
-			(xy 87.63 90.17) (xy 133.35 90.17)
+			(xy 87.63 90.17) (xy 138.43 90.17)
 		)
 		(stroke
@@
 	(wire
 		(pts
-			(xy 33.02 123.19) (xy 59.69 123.19)
+			(xy 133.35 92.71) (xy 133.35 95.25)
 		)
 		(stroke
@@
 	(wire
 		(pts
-			(xy 53.34 160.02) (xy 55.88 160.02)
+			(xy 33.02 123.19) (xy 59.69 123.19)
 		)
 		(stroke
@@
 	(wire
 		(pts
-			(xy 39.37 92.71) (xy 49.53 92.71)
+			(xy 53.34 160.02) (xy 55.88 160.02)
 		)
 		(stroke
@@
 	(wire
 		(pts
-			(xy 20.32 118.11) (xy 33.02 118.11)
+			(xy 39.37 92.71) (xy 49.53 92.71)
 		)
 		(stroke
@@
 	(wire
 		(pts
-			(xy 92.71 124.46) (xy 92.71 95.25)
+			(xy 20.32 118.11) (xy 33.02 118.11)
 		)
 		(stroke
@@
 	(wire
 		(pts
-			(xy 33.02 115.57) (xy 60.96 115.57)
+			(xy 92.71 124.46) (xy 92.71 95.25)
 		)
 		(stroke
@@
 	(wire
 		(pts
-			(xy 130.81 92.71) (xy 130.81 95.25)
+			(xy 33.02 115.57) (xy 60.96 115.57)
 		)
 		(stroke
@@
 	(wire
 		(pts
-			(xy 133.35 90.17) (xy 133.35 97.79)
-		)
-		(stroke
-			(width 0)
-			(type default)
-		)
-	)
-	(wire
-		(pts
-			(xy 133.35 66.04) (xy 149.86 66.04)
+			(xy 133.35 66.04) (xy 152.4 66.04)
 		)
 		(stroke
@@
 	)
 	(label "MCU+"
-		(at 149.86 97.79 0)
+		(at 152.4 97.79 0)
 		(effects
 			(font
@@
 	)
 	(label "MCU-"
-		(at 140.97 95.25 0)
+		(at 144.78 95.25 0)
 		(effects
 			(font
@@
 					(unit 1)
 				)
+			)
+		)
+	)
+	(symbol
+		(lib_id "Connector_Generic:Conn_01x02")
+		(at 128.27 100.33 0)
+		(mirror y)
+		(unit 1)
+		(exclude_from_sim no)
+		(in_bom yes)
+		(on_board yes)
+		(dnp no)
+		(fields_autoplaced yes)
+		(property "Reference" "J24"
+			(at 128.27 93.98 0)
+			(effects
+				(font
+					(size 1.27 1.27)
+				)
+			)
+		)
+		(property "Value" "Conn_01x02"
+			(at 128.27 96.52 0)
+			(effects
+				(font
+					(size 1.27 1.27)
+				)
+			)
+		)
+		(property "Footprint" ""
+			(at 128.27 100.33 0)
+			(effects
+				(font
+					(size 1.27 1.27)
+				)
+				(hide yes)
+			)
+		)
+		(property "Datasheet" "~"
+			(at 128.27 100.33 0)
+			(effects
+				(font
+					(size 1.27 1.27)
+				)
+				(hide yes)
+			)
+		)
+		(property "Description" "Generic connector, single row, 01x02, script generated (kicad-library-utils/schlib/autogen/connector/)"
+			(at 128.27 100.33 0)
+			(effects
+				(font
+					(size 1.27 1.27)
+				)
+				(hide yes)
+			)
+		)
+		(pin "1"
+		)
+		(pin "2"
+		)
+		(instances
+			(project ""
+				(path "/55cbadab-af07-45b3-b9ce-9748abc6dcd0"
+					(reference "J24")
+					(unit 1)
+				)
