File: kicad/TS schematics/MCU_scheme.kicad_sch (KiCad schematic)
At the start: 2 parts

Commit message: haha VCU V3.2 AND NEW SCHEMATICS HAHAHA
Parts:
- gave numbers to parts that had none: 2
Connections:
- net CAN_H renamed MCU_CAN_H
- net CAN_L renamed MCU_CAN_L
Other:
- moved on the sheet: J2
Changed lines of the file:
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@@
 	)
 	(junction
-		(at 53.34 77.47)
+		(at 64.77 62.23)
 		(diameter 0)
 		(color 0 0 0 0)
@@
 	(wire
 		(pts
-			(xy 53.34 77.47) (xy 40.64 77.47)
+			(xy 46.99 57.15) (xy 64.77 57.15)
 		)
 		(stroke
@@
 	(wire
 		(pts
-			(xy 40.64 72.39) (xy 53.34 72.39)
+			(xy 67.31 62.23) (xy 64.77 62.23)
 		)
 		(stroke
@@
 	(wire
 		(pts
-			(xy 55.88 77.47) (xy 53.34 77.47)
+			(xy 64.77 57.15) (xy 64.77 62.23)
 		)
 		(stroke
@@
 	(wire
 		(pts
-			(xy 53.34 72.39) (xy 53.34 77.47)
+			(xy 46.99 62.23) (xy 64.77 62.23)
 		)
 		(stroke
@@
 		)
 	)
-	(global_label "CAN_L"
-		(shape input)
-		(at 40.64 82.55 0)
-		(fields_autoplaced yes)
-		(effects
-			(font
-				(size 1.27 1.27)
-			)
-			(justify left)
-		)
-		(property "Intersheetrefs" "${INTERSHEET_REFS}"
-			(at 49.31 82.55 0)
+	(global_label "MCU_CAN_L"
+		(shape input)
+		(at 46.99 67.31 0)
+		(fields_autoplaced yes)
+		(effects
+			(font
+				(size 1.27 1.27)
+			)
+			(justify left)
+		)
+		(property "Intersheetrefs" "${INTERSHEET_REFS}"
+			(at 60.6795 67.31 0)
 			(effects
 				(font
@@
 	(global_label "FE"
 		(shape input)
-		(at 53.34 72.39 0)
-		(fields_autoplaced yes)
-		(effects
-			(font
-				(size 1.27 1.27)
-			)
-			(justify left)
-		)
-		(property "Intersheetrefs" "${INTERSHEET_REFS}"
-			(at 58.5628 72.39 0)
+		(at 64.77 57.15 0)
+		(fields_autoplaced yes)
+		(effects
+			(font
+				(size 1.27 1.27)
+			)
+			(justify left)
+		)
+		(property "Intersheetrefs" "${INTERSHEET_REFS}"
+			(at 69.9928 57.15 0)
 			(effects
 				(font
@@
 	(global_label "CAN_GND"
 		(shape input)
-		(at 55.88 77.47 0)
-		(fields_autoplaced yes)
-		(effects
-			(font
-				(size 1.27 1.27)
-			)
-			(justify left)
-		)
-		(property "Intersheetrefs" "${INTERSHEET_REFS}"
-			(at 67.3924 77.47 0)
+		(at 67.31 62.23 0)
+		(fields_autoplaced yes)
+		(effects
+			(font
+				(size 1.27 1.27)
+			)
+			(justify left)
+		)
+		(property "Intersheetrefs" "${INTERSHEET_REFS}"
+			(at 78.8224 62.23 0)
 			(effects
 				(font
@@
 		)
 	)
-	(global_label "CAN_H"
-		(shape input)
-		(at 40.64 80.01 0)
-		(fields_autoplaced yes)
-		(effects
-			(font
-				(size 1.27 1.27)
-			)
-			(justify left)
-		)
-		(property "Intersheetrefs" "${INTERSHEET_REFS}"
-			(at 49.6124 80.01 0)
+	(global_label "MCU_CAN_H"
+		(shape input)
+		(at 46.99 64.77 0)
+		(fields_autoplaced yes)
+		(effects
+			(font
+				(size 1.27 1.27)
+			)
+			(justify left)
+		)
+		(property "Intersheetrefs" "${INTERSHEET_REFS}"
+			(at 60.9819 64.77 0)
 			(effects
 				(font
@@
 	(global_label "CAN_V+"
 		(shape input)
-		(at 40.64 74.93 0)
-		(fields_autoplaced yes)
-		(effects
-			(font
-				(size 1.27 1.27)
-			)
-			(justify left)
-		)
-		(property "Intersheetrefs" "${INTERSHEET_REFS}"
-			(at 50.9429 74.93 0)
+		(at 46.99 59.69 0)
+		(fields_autoplaced yes)
+		(effects
+			(font
+				(size 1.27 1.27)
+			)
+			(justify left)
+		)
+		(property "Intersheetrefs" "${INTERSHEET_REFS}"
+			(at 57.2929 59.69 0)
 			(effects
 				(font
@@
 		(dnp no)
 		(fields_autoplaced yes)
-		(property "Reference" "#PWR?"
+		(property "Reference" "#PWR03"
 			(at 102.87 38.1 0)
 			(effects
@@
 		)
 		(instances
-			(project "TS schematics"
+			(project ""
 				(path "/55cbadab-af07-45b3-b9ce-9748abc6dcd0/0d00eec6-8293-4237-af5c-7114093f30fd"
-					(reference "#PWR?")
+					(reference "#PWR03")
 					(unit 1)
 				)
@@
 		(dnp no)
 		(fields_autoplaced yes)
-		(property "Reference" "#PWR?"
+		(property "Reference" "#PWR02"
 			(at 92.71 40.64 0)
 			(effects
@@
 		)
 		(instances
-			(project "TS schematics"
+			(project ""
 				(path "/55cbadab-af07-45b3-b9ce-9748abc6dcd0/0d00eec6-8293-4237-af5c-7114093f30fd"
-					(reference "#PWR?")
+					(reference "#PWR02")
 					(unit 1)
 				)
@@
 	(symbol
 		(lib_id "power:GND")
-		(at 53.34 77.47 0)
+		(at 64.77 62.23 0)
 		(unit 1)
 		(exclude_from_sim no)
@@
 		(dnp no)
 		(fields_autoplaced yes)
-		(property "Reference" "#PWR?"
-			(at 53.34 83.82 0)
+		(property "Reference" "#PWR01"
+			(at 64.77 68.58 0)
 			(effects
 				(font
@@
 		)
 		(property "Value" "GND"
-			(at 53.34 82.55 0)
+			(at 64.77 67.31 0)
 			(effects
 				(font
@@
 		)
 		(property "Footprint" ""
-			(at 53.34 77.47 0)
+			(at 64.77 62.23 0)
 			(effects
 				(font
@@
 		)
 		(property "Datasheet" ""
-			(at 53.34 77.47 0)
+			(at 64.77 62.23 0)
 			(effects
 				(font
@@
 		)
 		(property "Description" "Power symbol creates a global label with name \"GND\" , ground"
-			(at 53.34 77.47 0)
+			(at 64.77 62.23 0)
 			(effects
 				(font
@@
 		)
 		(instances
-			(project "TS schematics"
+			(project ""
 				(path "/55cbadab-af07-45b3-b9ce-9748abc6dcd0/0d00eec6-8293-4237-af5c-7114093f30fd"
-					(reference "#PWR?")
+					(reference "#PWR01")
 					(unit 1)
 				)
@@
 		(dnp no)
 		(fields_autoplaced yes)
-		(property "Reference" "#PWR?"
+		(property "Reference" "#PWR05"
 			(at 92.71 78.74 0)
 			(effects
@@
 		)
 		(instances
-			(project "TS schematics"
+			(project ""
 				(path "/55cbadab-af07-45b3-b9ce-9748abc6dcd0/0d00eec6-8293-4237-af5c-7114093f30fd"
-					(reference "#PWR?")
+					(reference "#PWR05")
 					(unit 1)
 				)
@@
 		(dnp no)
 		(fields_autoplaced yes)
-		(property "Reference" "#PWR?"
+		(property "Reference" "#PWR04"
 			(at 102.87 55.88 0)
 			(effects
@@
 		)
 		(instances
-			(project "TS schematics"
+			(project ""
 				(path "/55cbadab-af07-45b3-b9ce-9748abc6dcd0/0d00eec6-8293-4237-af5c-7114093f30fd"
-					(reference "#PWR?")
+					(reference "#PWR04")
 					(unit 1)
 				)
@@
 	(symbol
 		(lib_id "Connector_Generic:Conn_01x05")
-		(at 35.56 77.47 0)
+		(at 41.91 62.23 0)
 		(mirror y)
 		(unit 1)
@@
 		(dnp no)
 		(fields_autoplaced yes)
-		(property "Reference" "J?"
-			(at 35.56 66.04 0)
+		(property "Reference" "J2"
+			(at 41.91 50.8 0)
 			(effects
 				(font
@@
 		)
 		(property "Value" "CAN-BUS"
-			(at 35.56 68.58 0)
+			(at 41.91 53.34 0)
 			(effects
 				(font
@@
 		)
 		(property "Footprint" ""
-			(at 35.56 77.47 0)
+			(at 41.91 62.23 0)
 			(effects
 				(font
@@
 		)
 		(property "Datasheet" "~"
-			(at 35.56 77.47 0)
+			(at 41.91 62.23 0)
 			(effects
 				(font
@@
 		)
 		(property "Description" "Generic connector, single row, 01x05, script generated (kicad-library-utils/schlib/autogen/connector/)"
-			(at 35.56 77.47 0)
+			(at 41.91 62.23 0)
 			(effects
 				(font
@@
 		)
 		(instances
-			(project "TS schematics"
+			(project ""
 				(path "/55cbadab-af07-45b3-b9ce-9748abc6dcd0/0d00eec6-8293-4237-af5c-7114093f30fd"
-					(reference "J?")
+					(reference "J2")
 					(unit 1)
 				)
@@
 		(dnp no)
 		(fields_autoplaced yes)
-		(property "Reference" "J?"
+		(property "Reference" "J1"
 			(at 91.44 26.67 0)
 			(effects
@@
 		)
 		(instances
-			(project "TS schematics"
+			(project ""
 				(path "/55cbadab-af07-45b3-b9ce-9748abc6dcd0/0d00eec6-8293-4237-af5c-7114093f30fd"
-					(reference "J?")
+					(reference "J1")
 					(unit 1)
 				)
@@
 		)
 	)
-	(sheet_instances
-		(path "/"
-			(page "1")
-		)
-	)
-	(embedded_fonts no)
 )
