File: kicad/VCU_V2_kicad9/VCU_V2_kicad9.kicad_sch (KiCad schematic)
At the start: 81 parts, among them J1 AVR-ISP-6, J10 Conn_01x04, J11 USB_C_Receptacle_USB2.0_14P, J12 Conn_01x09, J13 Conn_01x03, J14 Conn_01x03, J15 Conn_01x03, J16 Conn_01x03, J17 Conn_01x03, J2 Conn_01x02, J3 Conn_01x03, J4 Conn_01x03, J5 Conn_01x03, J6 Conn_01x02, J7 Conn_01x02, J8 Conn_01x02, J9 Conn_01x04, Q2 MMBT3904, Q3 TO-252 PMOS, SW1 SW_Push, U1 ATmega328P-A, U2 MCP2515-xSO, U3 TJA1051T, U4 LM2576S-5, U5 AMS1117-3.3, U6 CH340C, Y1 16MHz, Y2 16MHz

Commit message: vcu v2
Parts:
- added J18, J19: Conn_01x03, Connector_JST:JST_XH_B3B-XH-A_1x03_P2.50mm_Vertical, symbol Connector_Generic:Conn_01x03
- J11: footprint Connector_USB:USB_C_Receptacle_G-Switch_GT-USB-7010ASV -> RMC_Connnector:USB_C_Receptacle_G-Switch_GT-USB-7010ASV_Handsolder
- Q2: footprint Package_TO_SOT_SMD:SOT-23 -> RMC_SOT:SOT-23
- U3: footprint Package_SO:SOIC-8_3.9x4.9mm_P1.27mm -> RMC_SO:SOIC-8_3.9x4.9mm_P1.27mm_RMC_Handsolder
- U4: footprint Package_TO_SOT_SMD:TO-252-5_TabPin3 -> RMC_TO:TO-263-5_TabPin3_Handsolder
- U5: footprint Package_TO_SOT_SMD:SOT-223-3_TabPin2 -> RMC_SOT:SOT-223-3_TabPin2_Handsolder
- U6: footprint Package_SO:SOIC-16_3.9x9.9mm_P1.27mm -> RMC_SO:SOIC-16_3.9x9.9mm_P1.27mm_Handsolder
- Y1, Y2: footprint RMC_Crystal:Crystal_HC49-U_Vertical_W_SMD_Handolder -> RMC_Crystal:Crystal_HC49-U_Vertical_W_SMD
Connections:
- net +3.3V is gone; now on net +3V3: R39.1
- net CS is gone; now on net CS_CAN: U2.16 (~{CS})
- net +5V: now also J18.3 (Pin_3), J19.3 (Pin_3)
- net DC/RS: no longer U1.1 (PD3)
- net GND: now also J18.1 (Pin_1), J19.1 (Pin_1)
- net RESET_SCREEN: no longer U1.32 (PD2)
- new net PD2: J18.2 (Pin_2), U1.32 (PD2)
- new net PD3: J19.2 (Pin_2), U1.1 (PD3)

Commit message: VCU v3.1 changes
Changed lines of the file:
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@@
 	)
 	(junction
-		(at 33.02 43.18)
-		(diameter 0)
-		(color 0 0 0 0)
-	)
-	(junction
 		(at 261.62 80.01)
 		(diameter 0)
@@
 	)
 	(junction
+		(at 33.02 43.18)
+		(diameter 0)
+		(color 0 0 0 0)
+	)
+	(junction
 		(at 257.81 106.68)
 		(diameter 0)
@@
 	(wire
 		(pts
-			(xy 30.48 43.18) (xy 33.02 43.18)
-		)
-		(stroke
-			(width 0)
-			(type default)
-		)
-	)
-	(wire
-		(pts
 			(xy 274.32 67.31) (xy 274.32 71.12)
 		)
@@
 	(symbol
 		(lib_id "power:+5V")
-		(at 30.48 43.18 90)
+		(at 33.02 43.18 90)
 		(unit 1)
 		(exclude_from_sim no)
@@
 		(fields_autoplaced yes)
 		(property "Reference" "#PWR01"
-			(at 34.29 43.18 0)
+			(at 36.83 43.18 0)
 			(effects
 				(font
@@
 		)
 		(property "Value" "+5V"
-			(at 26.67 43.1799 90)
+			(at 29.21 43.1799 90)
 			(effects
 				(font
@@
 		)
 		(property "Footprint" ""
-			(at 30.48 43.18 0)
+			(at 33.02 43.18 0)
 			(effects
 				(font
@@
 		)
 		(property "Datasheet" ""
-			(at 30.48 43.18 0)
+			(at 33.02 43.18 0)
 			(effects
 				(font
@@
 		)
 		(property "Description" "Power symbol creates a global label with name \"+5V\""
-			(at 30.48 43.18 0)
+			(at 33.02 43.18 0)
 			(effects
 				(font
