File: kicad/VCU_V2_kicad9/VCU_V2_kicad9.kicad_pcb (KiCad board)
At the start: 2 copper layers, 100 x 100 mm, 81 parts, among them J1 AVR-ISP-6, J10 Conn_01x04, J11 USB_C_Receptacle_USB2.0_14P, J12 Conn_01x09, J13 Conn_01x03, J14 Conn_01x03, J15 Conn_01x03, J16 Conn_01x03, J17 Conn_01x03, J2 Conn_01x02, J3 Conn_01x03, J4 Conn_01x03, J5 Conn_01x03, J6 Conn_01x02, J7 Conn_01x02, J8 Conn_01x02, J9 Conn_01x04, Q2 MMBT3904, Q3 TO-252 PMOS, SW1 SW_Push, U1 ATmega328P-A, U2 MCP2515-xSO, U3 TJA1051T, U4 LM2576S-5, U5 AMS1117-3.3, U6 CH340C, Y1 16MHz, Y2 16MHz

Commit message: vcu v2
Parts:
- added J18: Conn_01x03, Connector_JST:JST_XH_B3B-XH-A_1x03_P2.50mm_Vertical, F.Cu at (121.5, 129.8)
- added J19: Conn_01x03, Connector_JST:JST_XH_B3B-XH-A_1x03_P2.50mm_Vertical, F.Cu at (121.5, 137.4)
- J11: footprint Connector_USB:USB_C_Receptacle_G-Switch_GT-USB-7010ASV -> RMC_Connnector:USB_C_Receptacle_G-Switch_GT-USB-7010ASV_Handsolder
- Q2: footprint Package_TO_SOT_SMD:SOT-23 -> RMC_SOT:SOT-23
- U3: footprint Package_SO:SOIC-8_3.9x4.9mm_P1.27mm -> RMC_SO:SOIC-8_3.9x4.9mm_P1.27mm_RMC_Handsolder
- U4: footprint Package_TO_SOT_SMD:TO-252-5_TabPin3 -> RMC_TO:TO-263-5_TabPin3_Handsolder
- U5: footprint Package_TO_SOT_SMD:SOT-223-3_TabPin2 -> RMC_SOT:SOT-223-3_TabPin2_Handsolder
- U6: footprint Package_SO:SOIC-16_3.9x9.9mm_P1.27mm -> RMC_SO:SOIC-16_3.9x9.9mm_P1.27mm_Handsolder
- Y1, Y2: footprint RMC_Crystal:Crystal_HC49-U_Vertical_W_SMD_Handolder -> RMC_Crystal:Crystal_HC49-U_Vertical_W_SMD
- moved J13 100.8 mm to (121.7, 145.1), turned to 180 degrees
- moved R38 5.12 mm to (110.6, 90.1), turned to -90 degrees
- moved U4 4.96 mm to (119.7, 87.8)
- moved D3 3.09 mm to (110.6, 94.8), turned to 90 degrees
- moved C8 2.95 mm to (148.6, 133.8)
- moved C9 2.95 mm to (157.6, 133.8)
- moved R8 2.95 mm to (153.1, 133.8)
- moved Y2 2.95 mm to (150.6, 130.1)
- moved R44 0.67 mm to (147.0, 90.7)
- moved C15 0.66 mm to (133.9, 120.3)
- moved D4 0.21 mm to (119.8, 114.8)
- moved R39 0.21 mm to (114.9, 114.8)
- turned R7 to 90 degrees
Connections:
- C12 pad 1: +12V -> +5V
- C14 pad 1: +12V -> +5V
- R39 pad 1: +3.3V -> +3V3
- U1 pad 1: DC/RS -> /PD3
- U1 pad 32: RESET_SCREEN -> /PD2
- U2 pad 16: CS -> CS_CAN
- U5 pad 3: +12V -> +5V
Routing:
- net +5V: track 0.00 -> 508.8 mm, vias 0 -> 15
- net +3V3: track 0.00 -> 176.6 mm
- net +12V: track 0.00 -> 110.4 mm, vias 0 -> 4
- net TXD: track 0.00 -> 79.6 mm, vias 0 -> 2
- net RXD: track 0.00 -> 79.2 mm, vias 0 -> 2
- net /PD4: track 0.00 -> 76.1 mm
- net SCK: track 0.00 -> 73.7 mm, vias 0 -> 2
- net MOSI: track 0.00 -> 71.4 mm, vias 0 -> 5
- net /ADC6: track 0.00 -> 70.9 mm
- net SCL: track 0.00 -> 69.0 mm, vias 0 -> 2
- net CS_SCREEN: track 0.00 -> 68.7 mm, vias 0 -> 2
- net /PD3: track 0.00 -> 68.7 mm
- net MISO: track 0.00 -> 67.4 mm, vias 0 -> 2
- net RESET_SCREEN: track 0.00 -> 67.0 mm, vias 0 -> 2
- net SDA: track 0.00 -> 66.5 mm
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
Commit message: L
Parts:
- added G***: LOGO, LOGO, B.Cu at (149.8, 99.5)
