File: kicad/VCU_V3.1/VCU_V3_1_PREFAB/VCU_V3_1_PREFAB.kicad_sch (KiCad schematic)
At the start: 140 parts, among them J1 AVR-ISP-6, J2 Conn_01x24, J3 Conn_01x24, J4 Conn_01x04_Pin, J5 USB_C_Receptacle_USB2.0_14P, Q1 MMBT3906, Q2 Q_NMOS_GDS, Q3 MMBT3906, Q4 Q_NMOS_GDS, Q5 MMBT3906, Q6 Q_NMOS_GDS, Q7 MMBT3906, Q8 Q_NMOS_GDS, SW1 SW_Push, U1 ATmega328P-A, U10 TJA1051T, U11 ADuM1201AR, U12 MCP2515-xST, U13 MCP2515-xST, U14 MCP2515-xST, U16 LTV-817S, U17 ADuM1201AR, U18 ADuM1201AR, U19 OP07, U2 LM2575-5.0BU, U20 OP07, U21 OP07, U22 OP07, U23 LTV-817S, U24 LTV-817S, U25 LTV-817S, U3 CH340N, U5 TJA1051T, U6 AMS1117-3.3, U9 TJA1051T, Y1 16MHz, Y2 20MHz, Y3 20MHz, Y4 20MHz

Commit message: VCU v3.1 changes
Parts:
- added JP1: Jumper_2_Open, Jumper:SolderJumper-2_P1.3mm_Open_Pad1.0x1.5mm, symbol Jumper:Jumper_2_Open
- Q2, Q4, Q6, Q8: footprint Better_Handsolder:TO-252-2 -> RMC_TO:TO-252-2
- R33: value 1k -> 500R
- U10, U11, U17, U18, U5, U9: footprint Package_SO:SOIC-8_3.9x4.9mm_P1.27mm -> RMC_SO:SOIC-8_3.9x4.9mm_P1.27mm_RMC_Handsolder
- U12, U13, U14: footprint Package_SO:TSSOP-20_4.4x6.5mm_P0.65mm -> RMC_SO:TSSOP-20_4.4x6.5mm_P0.65mm
- U19, U20, U21, U22: footprint Package_SO:SOIC-8-1EP_3.9x4.9mm_P1.27mm_EP2.29x3mm -> RMC_SO:SOIC-8_3.9x4.9mm_P1.27mm_RMC_Handsolder
- U3: footprint Package_SO:SOP-8_3.9x4.9mm_P1.27mm -> RMC_SO:SOIC-8_3.9x4.9mm_P1.27mm_RMC_Handsolder
- U6: footprint Package_TO_SOT_SMD:SOT-223-3_TabPin2 -> RMC_SOT:SOT-223-3_TabPin2_Handsolder
Connections:
- net +5V: now also JP1.1 (A)
- net at C2.1, U1.20 (AREF): now also JP1.2 (B)
Other:
- moved on the sheet: C2

Commit message: VCU V3.1 preview patch v2
DRC debug
Change to pmos
remove usb c and add xh
remap pinout
rewiring
Parts:
- removed D4, D5, D6, D9: IR204A, LED_SMD:LED_1206_3216Metric_Pad1.42x1.75mm_HandSolder, symbol LED:IR204A
- removed D7: D, Diode_SMD:D_SMA_Handsoldering, symbol Device:D
- removed J5: USB_C_Receptacle_USB2.0_14P, RMC_Connnector:USB_C_Receptacle_G-Switch_GT-USB-7010ASV_Handsolder, symbol Connector:USB_C_Receptacle_USB2.0_14P
- removed Q1, Q3, Q5, Q7: MMBT3906, Package_TO_SOT_SMD:SOT-23, symbol Transistor_BJT:MMBT3906
- removed Q2, Q4, Q6, Q8: Q_NMOS_GDS, RMC_TO:TO-252-2, symbol Transistor_FET:Q_NMOS_GDS
- removed R12, R14, R17, R21, R25, R27: 1k, RMC_Resistor:R_0805_2012Metric_Pad1.20x1.40mm_HandSolder_L, symbol Device:R
- removed R13, R20, R26: 100k, RMC_Resistor:R_0805_2012Metric_Pad1.20x1.40mm_HandSolder_L, symbol Device:R
- removed R34: 5K1, RMC_Resistor:R_0805_2012Metric_Pad1.20x1.40mm_HandSolder_L, symbol Device:R
- removed R35: 5k1, RMC_Resistor:R_0805_2012Metric_Pad1.20x1.40mm_HandSolder_L, symbol Device:R
- added D11: IR204A, LED_SMD:LED_1206_3216Metric_Pad1.42x1.75mm_HandSolder, symbol LED:IR204A
- added D13, D14, D15, D16, D17, D18, D19, D20: LED, RMC_LED:LED_0805_2012Metric_Pad1.45x1.40mm_HandSolder, symbol Device:LED
- added J6: Conn_01x04_Pin, Connector_JST:JST_XH_B4B-XH-A_1x04_P2.50mm_Vertical, symbol Connector:Conn_01x04_Pin
- added Q11, Q13, Q15, Q17: MMBT3904, RMC_SOT:SOT-23, symbol Transistor_BJT:MMBT3904
- added Q12, Q14, Q16, Q18: BSC030P03NS3, RMC_SO:Infineon_PG-TDSON-8_6.15x5.15mm, symbol RMC:PMOS_tdson-8
- added R36, R52, R53, R54, R55, R57, R58, R59, R60, R62, R63, R64, R65, R67: 1k, RMC_Resistor:R_0805_2012Metric_Pad1.20x1.40mm_HandSolder_L, symbol Device:R
- added R56, R61, R66: 100k, RMC_Resistor:R_0805_2012Metric_Pad1.20x1.40mm_HandSolder_L, symbol Device:R
- added R68: 500R, RMC_Resistor:R_0805_2012Metric_Pad1.20x1.40mm_HandSolder_L, symbol Device:R
- R49: value 100k -> 1k
- R50: value 1k -> 100k
Connections:
- net +12V: now also R49.1, D13.2 (A), D15.2 (A), D17.2 (A), D19.2 (A), Q12.1 (S), Q12.2 (S), Q12.3 (S), Q14.1 (S), Q14.2 (S), Q14.3 (S), Q16.1 (S), Q16.2 (S), Q16.3 (S), Q18.1 (S), Q18.2 (S), Q18.3 (S), R55.1, R60.1, R65.1; no longer R49.2
- net +5V: now also J6.1 (Pin_1)
- net BRAKE OUT: now also D18.2 (A), Q16.5 (D), Q16.6 (D), Q16.7 (D), Q16.8 (D), R62.2
- net BUZZER_OUT: now also J3.4 (Pin_4), D16.2 (A), Q14.5 (D), Q14.6 (D), Q14.7 (D), Q14.8 (D), R57.2; no longer J3.6 (Pin_6)
- net CAN3+: now also J3.15 (Pin_15), J3.7 (Pin_7); no longer J3.12 (Pin_12), J3.4 (Pin_4)
- net CAN3-: now also J3.16 (Pin_16), J3.8 (Pin_8); no longer J3.13 (Pin_13), J3.5 (Pin_5)
- net D+: now also J6.3 (Pin_3)
- net D-: now also J6.2 (Pin_2)
- net GND: now also J3.12 (Pin_12), J3.13 (Pin_13), J3.14 (Pin_14), R50.2, J6.4 (Pin_4), Q11.2 (E), Q13.2 (E), Q15.2 (E), Q17.2 (E), R56.2, R61.2, R66.2, R68.2; no longer J3.7 (Pin_7), R48.1, R50.1
- net LED_OUTPUT: now also J3.6 (Pin_6), D20.2 (A), Q18.5 (D), Q18.6 (D), Q18.7 (D), Q18.8 (D), R67.2; no longer J3.8 (Pin_8)
- net PD4: now also D11.2 (A); no longer J3.14 (Pin_14)
- net VehicleStatus OUT: now also D14.2 (A), Q12.5 (D), Q12.6 (D), Q12.7 (D), Q12.8 (D), R52.2
- net at U23.3: now also R58.1
- net at U16.3: now also R63.1
- net at R48.2: now also R49.2, R50.1, Q11.3 (C), Q12.4 (G)
- net at U25.3: now also R36.1
- net at U24.3: now also R53.1
- new net: Q13.3 (C), Q14.4 (G), R54.2, R55.2, R56.1
- new net: D18.1 (K), R62.1
- new net: Q17.1 (B), R63.2
- new net: D20.1 (K), R67.1
- new net: D19.1 (K), R64.1
- new net: Q15.3 (C), Q16.4 (G), R59.2, R60.2, R61.1
- new net: Q13.1 (B), R53.2
- new net: Q17.3 (C), Q18.4 (G), R64.2, R65.2, R66.1
- new net: D16.1 (K), R57.1
- new net: Q11.1 (B), R36.2
- new net: D17.1 (K), R59.1
- new net: D11.1 (K), R68.1
- new net: D15.1 (K), R54.1
- new net: D14.1 (K), R52.1
- new net: Q15.1 (B), R58.2
- new net: D13.1 (K), R48.1
- no-connect marks 23 -> 24
Other:
- note removed: "tighten the trace change inductor and 817 footprint add ch340n so change pin"
- moved on the sheet: R10, R16, R24, R32, R37, R38, R39, R47, U16, U23, U24, U25
