File: kicad/VCU V3.2/PDU_P.kicad_sch (KiCad schematic)
At the start: 7 parts, among them Q1 BSC030P03NS3, Q3 MMBT3904

Commit message: VCU V3.2
Parts:
- renumbered Q3 to Q2, Q1 to Q5, R3 to R10, R6 to R13, R5 to R18, R4 to R5
