File: kicad/VCU V3.2/AIN.kicad_sch (KiCad schematic)
At the start: 4 parts, among them U6 OP07

Commit message: VCU V3.2
Parts:
- removed C19: 100nF, symbol Device:C
- removed R21, R22: R, symbol Device:R
- removed U6: OP07, symbol Amplifier_Operational:OP07
- added C26: 100nF, symbol Device:C
- added U12: LM358, symbol Amplifier_Operational:LM358
Connections:
- net GND: now also C26.2, U12.4 (V-)
- new net +5V: C26.1, U12.8 (V+)
- new net AIN1: U12.3 (+)
- new net AIN2: U12.5 (+)
- new net AOUT_1: U12.1, U12.2 (-)
- new net AOUT_2: U12.6 (-), U12.7
- no-connect marks 2 -> 0

Commit message: VCU V3.2
Parts:
- added C30, C31: 100nF, RMC_Capacitor:C_0805_2012Metric_Pad1.18x1.45mm_HandSolder_L, symbol Device:C
- C32: renamed from C26; footprint (none) -> RMC_Capacitor:C_0805_2012Metric_Pad1.18x1.45mm_HandSolder_L
- U13: renamed from U12; footprint (none) -> RMC_SO:SOIC-8_3.9x4.9mm_P1.27mm_RMC_Handsolder
Connections:
- net AIN1: now also C30.1
- net AIN2: now also C31.1
- net GND: now also C30.2, C31.2
