File: kicad/VCU V3.2/AIN.kicad_sch (KiCad schematic)
At the start: 4 parts, among them U13 LM358

Commit message: VCU V3.2 FINISH LAYOUT
Parts:
- added C37, C38: 100nF, RMC_Capacitor:C_0805_2012Metric_Pad1.18x1.45mm_HandSolder_L, symbol Device:C
- U13: value LM358 -> SGM722
Connections:
- net AOUT_1: now also C38.2
- net AOUT_2: now also C37.2
- net GND: now also C37.1, C38.1
