File: kicad/VCU V3.2/APPS_gain.kicad_sch (KiCad schematic)
At the start: 6 parts, among them U7 OP07

Commit message: VCU V3.2
Parts:
- renumbered R26 to R25, R30 to R26

Commit message: VCU V3.2
Parts:
- added C23, C25: 100nF, RMC_Capacitor:C_0805_2012Metric_Pad1.18x1.45mm_HandSolder_L, symbol Device:C
- C24: renamed from C20; footprint (none) -> RMC_Capacitor:C_0805_2012Metric_Pad1.18x1.45mm_HandSolder_L
- R26: renamed from R23; footprint (none) -> RMC_Resistor:R_0805_2012Metric_Pad1.20x1.40mm_HandSolder_L
- R27: renamed from R24; footprint (none) -> RMC_Resistor:R_0805_2012Metric_Pad1.20x1.40mm_HandSolder_L
- R28: renamed from R25; footprint (none) -> RMC_Resistor:R_0805_2012Metric_Pad1.20x1.40mm_HandSolder_L
- R29: renamed from R26; footprint (none) -> RMC_Resistor:R_0805_2012Metric_Pad1.20x1.40mm_HandSolder_L
- U7: footprint (none) -> RMC_SO:SOIC-8_3.9x4.9mm_P1.27mm_RMC_Handsolder
Connections:
- net APPS: now also C25.1
- net GND: now also C23.2, C25.2
- net VCC: no longer C24.1, U7.7 (V+)
- net VOUT: now also C23.1
- new net AVCC: C24.1, U7.7 (V+)
Other:
- moved on the sheet: C24, R26, R27
