File: kicad/VCU V3.2/LM2575 AMS1117.kicad_sch (KiCad schematic)
At the start: 12 parts, among them U2 LM2575-5.0BU, U3 AMS1117-3.3

Commit message: VCU V3.2
Parts:
- renumbered C12 to C10, C13 to C11, C14 to C12, C2 to C13, C4 to C14, C1 to C7, C11 to C8, C3 to C9
Changed lines of the file:
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@@
 		(dnp no)
 		(fields_autoplaced yes)
-		(property "Reference" "#PWR02"
+		(property "Reference" "#PWR015"
 			(at 118.11 69.85 0)
 			(effects
@@
 			(project "VCU V3.2"
 				(path "/763833dc-bbcb-46fa-abab-1e60581348ee/4de3fa49-f848-498f-8af8-097b30b6f2cd"
-					(reference "#PWR02")
+					(reference "#PWR015")
 					(unit 1)
 				)
@@
 		(dnp no)
 		(fields_autoplaced yes)
-		(property "Reference" "C12"
+		(property "Reference" "C10"
 			(at 106.68 104.1399 0)
 			(effects
@@
 			(project "VCU V3.2"
 				(path "/763833dc-bbcb-46fa-abab-1e60581348ee/4de3fa49-f848-498f-8af8-097b30b6f2cd"
-					(reference "C12")
+					(reference "C10")
 					(unit 1)
 				)
@@
 		(dnp no)
 		(fields_autoplaced yes)
-		(property "Reference" "C1"
+		(property "Reference" "C7"
 			(at 86.36 54.9909 0)
 			(effects
@@
 			(project "VCU V3.2"
 				(path "/763833dc-bbcb-46fa-abab-1e60581348ee/4de3fa49-f848-498f-8af8-097b30b6f2cd"
-					(reference "C1")
+					(reference "C7")
 					(unit 1)
 				)
@@
 		(dnp no)
 		(fields_autoplaced yes)
-		(property "Reference" "C4"
+		(property "Reference" "C14"
 			(at 167.64 58.4199 0)
 			(effects
@@
 			(project "VCU V3.2"
 				(path "/763833dc-bbcb-46fa-abab-1e60581348ee/4de3fa49-f848-498f-8af8-097b30b6f2cd"
-					(reference "C4")
+					(reference "C14")
 					(unit 1)
 				)
@@
 		(dnp no)
 		(fields_autoplaced yes)
-		(property "Reference" "C13"
+		(property "Reference" "C11"
 			(at 133.35 103.2509 0)
 			(effects
@@
 			(project "VCU V3.2"
 				(path "/763833dc-bbcb-46fa-abab-1e60581348ee/4de3fa49-f848-498f-8af8-097b30b6f2cd"
-					(reference "C13")
+					(reference "C11")
 					(unit 1)
 				)
@@
 		(dnp no)
 		(fields_autoplaced yes)
-		(property "Reference" "C11"
+		(property "Reference" "C8"
 			(at 93.98 103.2509 0)
 			(effects
@@
 			(project "VCU V3.2"
 				(path "/763833dc-bbcb-46fa-abab-1e60581348ee/4de3fa49-f848-498f-8af8-097b30b6f2cd"
-					(reference "C11")
+					(reference "C8")
 					(unit 1)
 				)
@@
 		(dnp no)
 		(fields_autoplaced yes)
-		(property "Reference" "#PWR03"
+		(property "Reference" "#PWR013"
 			(at 82.55 54.61 0)
 			(effects
@@
 			(project "VCU V3.2"
 				(path "/763833dc-bbcb-46fa-abab-1e60581348ee/4de3fa49-f848-498f-8af8-097b30b6f2cd"
-					(reference "#PWR03")
+					(reference "#PWR013")
 					(unit 1)
 				)
@@
 		(dnp no)
 		(fields_autoplaced yes)
-		(property "Reference" "#PWR015"
+		(property "Reference" "#PWR014"
 			(at 90.17 105.41 0)
 			(effects
@@
 			(project "VCU V3.2"
 				(path "/763833dc-bbcb-46fa-abab-1e60581348ee/4de3fa49-f848-498f-8af8-097b30b6f2cd"
-					(reference "#PWR015")
+					(reference "#PWR014")
 					(unit 1)
 				)
@@
 		(dnp no)
 		(fields_autoplaced yes)
-		(property "Reference" "C14"
+		(property "Reference" "C12"
 			(at 146.05 104.1399 0)
 			(effects
@@
 			(project "VCU V3.2"
 				(path "/763833dc-bbcb-46fa-abab-1e60581348ee/4de3fa49-f848-498f-8af8-097b30b6f2cd"
-					(reference "C14")
+					(reference "C12")
 					(unit 1)
 				)
@@
 		(dnp no)
 		(fields_autoplaced yes)
-		(property "Reference" "C2"
+		(property "Reference" "C13"
 			(at 154.94 57.5309 0)
 			(effects
@@
 			(project "VCU V3.2"
 				(path "/763833dc-bbcb-46fa-abab-1e60581348ee/4de3fa49-f848-498f-8af8-097b30b6f2cd"
-					(reference "C2")
+					(reference "C13")
 					(unit 1)
 				)
@@
 		(dnp no)
 		(fields_autoplaced yes)
-		(property "Reference" "#PWR04"
+		(property "Reference" "#PWR018"
 			(at 163.83 54.61 0)
 			(effects
@@
 			(project "VCU V3.2"
 				(path "/763833dc-bbcb-46fa-abab-1e60581348ee/4de3fa49-f848-498f-8af8-097b30b6f2cd"
-					(reference "#PWR04")
+					(reference "#PWR018")
 					(unit 1)
 				)
@@
 		(dnp no)
 		(fields_autoplaced yes)
-		(property "Reference" "C3"
+		(property "Reference" "C9"
 			(at 99.06 55.8799 0)
 			(effects
@@
 			(project "VCU V3.2"
 				(path "/763833dc-bbcb-46fa-abab-1e60581348ee/4de3fa49-f848-498f-8af8-097b30b6f2cd"
-					(reference "C3")
-					(unit 1)
-				)
+					(reference "C9")
+					(unit 1)
+				)

Commit message: VCU V3.2
Parts:
- added D10, D9: LED, RMC_LED:LED_0805_2012Metric_Pad1.45x1.40mm_HandSolder, symbol Device:LED
- added F1: 12V 3A, Fuse:Fuse_1210_3225Metric_Pad1.42x2.65mm_HandSolder, symbol Device:Fuse
- added F2: 5V 1A, Fuse:Fuse_1210_3225Metric_Pad1.42x2.65mm_HandSolder, symbol Device:Fuse
- added R69, R70: 1k, RMC_Resistor:R_0805_2012Metric_Pad1.20x1.40mm_HandSolder_L, symbol Device:R
- C10: renamed from C9; footprint (none) -> RMC_Capacitor:C_0805_2012Metric_Pad1.18x1.45mm_HandSolder_L
- C11: renamed from C10; footprint (none) -> RMC_Capacitor:C_0805_2012Metric_Pad1.18x1.45mm_HandSolder_L
- C12: renamed from C11; footprint (none) -> RMC_Capacitor:C_0805_2012Metric_Pad1.18x1.45mm_HandSolder_L
- C13: renamed from C12; footprint (none) -> RMC_Capacitor:C_0805_2012Metric_Pad1.18x1.45mm_HandSolder_L
- C14: renamed from C13; footprint (none) -> RMC_Capacitor:CP_Radial_D6.3mm_P2.50mm_handsolder
- C15: renamed from C14; footprint (none) -> RMC_Capacitor:C_0805_2012Metric_Pad1.18x1.45mm_HandSolder_L
- C8: renamed from C7; footprint (none) -> RMC_Capacitor:CP_Radial_D6.3mm_P2.50mm_handsolder
- C9: renamed from C8; footprint (none) -> RMC_Capacitor:C_0805_2012Metric_Pad1.18x1.45mm_HandSolder_L
- D1: value D_Schottky -> SS32; footprint (none) -> Diode_SMD:D_SMA_Handsoldering
- L1: footprint (none) -> RMC_Inductor:L_TDK_SLF12575
- U2: footprint Package_TO_SOT_SMD:TO-263-5_TabPin3 -> RMC_TO:TO-263-5_TabPin3_Long
- U3: footprint Package_TO_SOT_SMD:SOT-223-3_TabPin2 -> RMC_SOT:SOT-223-3_TabPin2_Handsolder
Connections:
- net +3V3: now also D10.2 (A), F2.1; no longer C12.1, C13.1, U3.2 (VO)
- net +5V: now also D9.2 (A), F1.1; no longer C14.1, C15.1, L1.2, U2.4 (FB)
- net GND: now also R69.2, R70.2
- new net: C12.1, C13.1, F2.2, U3.2 (VO)
- new net: D10.1 (K), R70.1
- new net: C14.1, C15.1, F1.2, L1.2, U2.4 (FB)
- new net: D9.1 (K), R69.1
