File: kicad/VCU V3.2/LM2575 AMS1117.kicad_sch (KiCad schematic)
At the start: 18 parts, among them U2 LM2575-5.0BU, U3 AMS1117-3.3

Commit message: VCU V3.2 FINISH LAYOUT
Parts:
- removed C11, C13: 100nF, RMC_Capacitor:C_0805_2012Metric_Pad1.18x1.45mm_HandSolder_L, symbol Device:C
- removed C12: 22uF, RMC_Capacitor:C_0805_2012Metric_Pad1.18x1.45mm_HandSolder_L, symbol Device:C_Polarized
- removed C9: 10uF, RMC_Capacitor:C_0805_2012Metric_Pad1.18x1.45mm_HandSolder_L, symbol Device:C_Polarized
- removed D10: LED, RMC_LED:LED_0805_2012Metric_Pad1.45x1.40mm_HandSolder, symbol Device:LED
- removed F2: 5V 1A, Fuse:Fuse_1210_3225Metric_Pad1.42x2.65mm_HandSolder, symbol Device:Fuse
- removed R70: 1k, RMC_Resistor:R_0805_2012Metric_Pad1.20x1.40mm_HandSolder_L, symbol Device:R
- removed U3: AMS1117-3.3, RMC_SOT:SOT-223-3_TabPin2_Handsolder, symbol Regulator_Linear:AMS1117-3.3
