File: kicad/VCU V3.2/PDU_P_sot23.kicad_sch (KiCad schematic)
At the start: 7 parts, among them Q1 MMBT3904, Q2 BSC030P03NS3

Commit message: VCU V3.2
Parts:
- removed D2: LED, RMC_LED:LED_0805_2012Metric_Pad1.45x1.40mm_HandSolder, symbol Device:LED
- removed Q1: MMBT3904, RMC_SOT:SOT-23, symbol Transistor_BJT:MMBT3904
- removed Q2: BSC030P03NS3, RMC_SO:Infineon_PG-TDSON-8_6.15x5.15mm, symbol RMC:PMOS_tdson-8
- removed R5, R6, R7: 1k, RMC_Resistor:R_0805_2012Metric_Pad1.20x1.40mm_HandSolder_L, symbol Device:R
- removed R8: 100k, RMC_Resistor:R_0805_2012Metric_Pad1.20x1.40mm_HandSolder_L, symbol Device:R
- added D6: LED, RMC_LED:LED_0805_2012Metric_Pad1.45x1.40mm_HandSolder, symbol Device:LED
- added JP1: Jumper_3_Open, Jumper:SolderJumper-3_P1.3mm_Open_Pad1.0x1.5mm, symbol Jumper:Jumper_3_Open
- added Q10: AO3401A, Package_TO_SOT_SMD:SOT-23, symbol Transistor_FET:AO3401A
- added Q9: MMBT3904, RMC_SOT:SOT-23, symbol Transistor_BJT:MMBT3904
- added R57, R58, R59: 1k, RMC_Resistor:R_0805_2012Metric_Pad1.20x1.40mm_HandSolder_L, symbol Device:R
- added R60: 100k, RMC_Resistor:R_0805_2012Metric_Pad1.20x1.40mm_HandSolder_L, symbol Device:R
Connections:
- net GND: now also Q9.2 (E), R60.2
- net OUT: now also Q10.3 (D)
- net SIGNAL: now also R57.1
- new net: Q10.1 (G), Q9.3 (C), R58.2, R59.2, R60.1
- new net: D6.2 (A), JP1.2 (C), Q10.2 (S), R59.1
- new net: Q9.1 (B), R57.2
- new net: D6.1 (K), R58.1
- new net VIN_H: JP1.1 (A)
- new net VIN_L: JP1.3 (B)
