File: kicad/VCU V3.2/PDU_P_sot23.kicad_sch (KiCad schematic)
At the start: 8 parts, among them Q10 AO3401A, Q9 MMBT3904

Commit message: AHHHHH vcu v3.2
Parts:
- Q10: footprint Package_TO_SOT_SMD:SOT-23 -> RMC_SOT:SOT-23
Changed lines of the file:
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@@
 			)
 		)
-		(property "Footprint" "Package_TO_SOT_SMD:SOT-23"
+		(property "Footprint" "RMC_SOT:SOT-23"
 			(at 154.94 79.375 0)
 			(effects
