File: kicad/VCU V3.2/PDU_P4.kicad_sch (KiCad schematic)
At the start: 9 parts, among them U12 LTV-847S

Commit message: AHHHHH vcu v3.2
Connections:
- net PDU_1/SIGNAL: now also U12.9; no longer U12.15
- net PDU_1/VIN: now also U12.10; no longer U12.16
- net PDU_2/SIGNAL: now also U12.11; no longer U12.13
- net PDU_2/VIN: now also U12.12; no longer U12.14
- net PDU_3/SIGNAL: now also U12.13; no longer U12.11
- net PDU_3/VIN: now also U12.14; no longer U12.12
- net PDU_4/SIGNAL: now also U12.15; no longer U12.9
- net PDU_4/VIN: now also U12.16; no longer U12.10
- net at U12.3: now also R55.2; no longer R54.2
- net at U12.5: now also R54.2; no longer R55.2
- net at R56.2: now also U12.1; no longer U12.7
- net at R53.2: now also U12.7; no longer U12.1
Other:
- moved on the sheet: U12A, U12B, U12C, U12D
Changed lines of the file:
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@@
 	(symbol
 		(lib_id "Isolator:LTV-847S")
-		(at 113.03 87.63 0)
+		(at 113.03 109.22 0)
 		(unit 2)
 		(exclude_from_sim no)
@@
 		(fields_autoplaced yes)
 		(property "Reference" "U12"
-			(at 113.03 78.74 0)
+			(at 113.03 100.33 0)
 			(effects
 				(font
@@
 		)
 		(property "Value" "LTV-847S"
-			(at 113.03 81.28 0)
+			(at 113.03 102.87 0)
 			(effects
 				(font
@@
 		)
 		(property "Footprint" "Package_DIP:SMDIP-16_W9.53mm"
-			(at 113.03 95.25 0)
+			(at 113.03 116.84 0)
 			(effects
 				(font
@@
 		)
 		(property "Datasheet" "http://www.us.liteon.com/downloads/LTV-817-827-847.PDF"
-			(at 97.79 76.2 0)
+			(at 97.79 97.79 0)
 			(effects
 				(font
@@
 		)
 		(property "Description" "DC Optocoupler, Vce 35V, CTR 50%, SMDIP-16"
-			(at 113.03 87.63 0)
+			(at 113.03 109.22 0)
 			(effects
 				(font
@@
 	(symbol
 		(lib_id "Isolator:LTV-847S")
-		(at 113.03 109.22 0)
+		(at 113.03 87.63 0)
 		(unit 3)
 		(exclude_from_sim no)
@@
 		(dnp no)
 		(property "Reference" "U12"
-			(at 113.03 100.33 0)
+			(at 113.03 78.74 0)
 			(effects
 				(font
@@
 		)
 		(property "Value" "LTV-847S"
-			(at 113.03 102.87 0)
+			(at 113.03 81.28 0)
 			(effects
 				(font
@@
 		)
 		(property "Footprint" "Package_DIP:SMDIP-16_W9.53mm"
-			(at 113.03 116.84 0)
+			(at 113.03 95.25 0)
 			(effects
 				(font
@@
 		)
 		(property "Datasheet" "http://www.us.liteon.com/downloads/LTV-817-827-847.PDF"
-			(at 97.79 97.79 0)
+			(at 97.79 76.2 0)
 			(effects
 				(font
@@
 		)
 		(property "Description" "DC Optocoupler, Vce 35V, CTR 50%, SMDIP-16"
-			(at 113.03 109.22 0)
+			(at 113.03 87.63 0)
 			(effects
 				(font
@@
 	(symbol
 		(lib_id "Isolator:LTV-847S")
+		(at 113.03 64.77 0)
+		(unit 4)
+		(exclude_from_sim no)
+		(in_bom yes)
+		(on_board yes)
+		(dnp no)
+		(fields_autoplaced yes)
+		(property "Reference" "U12"
+			(at 113.03 55.88 0)
+			(effects
+				(font
+					(size 1.27 1.27)
+				)
+			)
+		)
+		(property "Value" "LTV-847S"
+			(at 113.03 58.42 0)
+			(effects
+				(font
+					(size 1.27 1.27)
+				)
+			)
+		)
+		(property "Footprint" "Package_DIP:SMDIP-16_W9.53mm"
+			(at 113.03 72.39 0)
+			(effects
+				(font
+					(size 1.27 1.27)
+				)
+				(hide yes)
+			)
+		)
+		(property "Datasheet" "http://www.us.liteon.com/downloads/LTV-817-827-847.PDF"
+			(at 97.79 53.34 0)
+			(effects
+				(font
+					(size 1.27 1.27)
+				)
+				(hide yes)
+			)
+		)
+		(property "Description" "DC Optocoupler, Vce 35V, CTR 50%, SMDIP-16"
+			(at 113.03 64.77 0)
+			(effects
+				(font
+					(size 1.27 1.27)
+				)
+				(hide yes)
+			)
+		)
+		(pin "16"
+		)
+		(pin "3"
+		)
+		(pin "14"
+		)
+		(pin "1"
+		)
+		(pin "2"
+		)
+		(pin "15"
+		)
+		(pin "4"
+		)
+		(pin "5"
+		)
+		(pin "12"
+		)
+		(pin "11"
+		)
+		(pin "7"
+		)
+		(pin "8"
+		)
+		(pin "10"
+		)
+		(pin "13"
+		)
+		(pin "6"
+		)
+		(pin "9"
+		)
+		(instances
+			(project "VCU V3.2"
+				(path "/763833dc-bbcb-46fa-abab-1e60581348ee/4f3c75e6-583d-4c3b-bd1a-9a6f89986770"
+					(reference "U12")
+					(unit 4)
+				)
+			)
+		)
+	)
+	(symbol
+		(lib_id "Isolator:LTV-847S")
 		(at 113.03 135.89 0)
-		(unit 4)
+		(unit 1)
 		(exclude_from_sim no)
 		(in_bom yes)
@@
 			(effects
 				(font
-					(size 1.27 1.27)
-				)
-				(hide yes)
-			)
-		)
-		(pin "16"
-		)
-		(pin "3"
-		)
-		(pin "14"
-		)
-		(pin "1"
-		)
-		(pin "2"
-		)
-		(pin "15"
-		)
-		(pin "4"
-		)
-		(pin "5"
-		)
-		(pin "12"
-		)
-		(pin "11"
-		)
-		(pin "7"
-		)
-		(pin "8"
-		)
-		(pin "10"
-		)
-		(pin "13"
-		)
-		(pin "6"
-		)
-		(pin "9"
-		)
-		(instances
-			(project "VCU V3.2"
-				(path "/763833dc-bbcb-46fa-abab-1e60581348ee/4f3c75e6-583d-4c3b-bd1a-9a6f89986770"
-					(reference "U12")
-					(unit 4)
-				)
-			)
-		)
-	)
-	(symbol
-		(lib_id "Isolator:LTV-847S")
-		(at 113.03 64.77 0)
-		(unit 1)
-		(exclude_from_sim no)
-		(in_bom yes)
-		(on_board yes)
-		(dnp no)
-		(fields_autoplaced yes)
-		(property "Reference" "U12"
-			(at 113.03 55.88 0)
-			(effects
-				(font
-					(size 1.27 1.27)
-				)
-			)
-		)
-		(property "Value" "LTV-847S"
-			(at 113.03 58.42 0)
-			(effects
-				(font
-					(size 1.27 1.27)
-				)
-			)
-		)
-		(property "Footprint" "Package_DIP:SMDIP-16_W9.53mm"
-			(at 113.03 72.39 0)
-			(effects
-				(font
-					(size 1.27 1.27)
-				)
-				(hide yes)
-			)
-		)
-		(property "Datasheet" "http://www.us.liteon.com/downloads/LTV-817-827-847.PDF"
-			(at 97.79 53.34 0)
-			(effects
-				(font
-					(size 1.27 1.27)
-				)
-				(hide yes)
-			)
-		)
-		(property "Description" "DC Optocoupler, Vce 35V, CTR 50%, SMDIP-16"
-			(at 113.03 64.77 0)
-			(effects
-				(font
