File: kicad/VCU V3.2/PDU_P4.kicad_sch (KiCad schematic)
At the start: 9 parts, among them U12 LTV-847S

Commit message: VCU V3.2 DONE HAHA
Do you remember? the 21st night of September.
Parts:
- U12: footprint Package_DIP:SMDIP-16_W9.53mm -> to be sorted:SMDIP-16_W9.53mm
Changed lines of the file:
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@@
 			)
 		)
-		(property "Footprint" "Package_DIP:SMDIP-16_W9.53mm"
+		(property "Footprint" "to be sorted:SMDIP-16_W9.53mm"
 			(at 113.03 116.84 0)
 			(effects
@@
 			)
 		)
-		(property "Footprint" "Package_DIP:SMDIP-16_W9.53mm"
+		(property "Footprint" "to be sorted:SMDIP-16_W9.53mm"
 			(at 113.03 95.25 0)
 			(effects
@@
 			)
 		)
-		(property "Footprint" "Package_DIP:SMDIP-16_W9.53mm"
+		(property "Footprint" "to be sorted:SMDIP-16_W9.53mm"
 			(at 113.03 72.39 0)
 			(effects
@@
 			)
 		)
-		(property "Footprint" "Package_DIP:SMDIP-16_W9.53mm"
+		(property "Footprint" "to be sorted:SMDIP-16_W9.53mm"
 			(at 113.03 143.51 0)
 			(effects
