File: kicad/VCU V3.2/VCU V3.2.kicad_sch (KiCad schematic)
At the start: 12 parts, among them J1 AVR-ISP-6, SW1 SW_Push, U1 ATmega328P-A, Y1 16MHz

Commit message: VCU V3.2
Parts:
- added J2: ~, Better_Handsolder:HD241_24pin, symbol HD241:HD241
- added J3: ~, Better_Handsolder:HD241_GF30, symbol HD241:HD241
- renumbered C5 to C1, C6 to C2, C7 to C3, C8 to C4, C9 to C5, C10 to C6
Connections:
- net +5V: now also J2.14, J3.3, J3.4
- net APPS_3VGND: now also J3.18
- net APPS_3VIN: now also J3.2
- net APPS_3VOUT: now also J3.10
- net APPS_5VGND: now also J3.17
- net APPS_5VIN: now also J3.1
- net APPS_5VOUT: now also J3.9
- net GND: now also J2.15, J2.16, J2.23, J2.24, J2.7, J2.8, J3.19, J3.20, J3.24
- net MISO: now also J2.19
- net MOSI: now also J2.20
- net PDU_1: now also J2.3; no longer U1.30 (PD0)
- net PDU_2: now also J2.4; no longer U1.31 (PD1)
- net PDU_3: now also J2.5; no longer U1.32 (PD2)
- net PDU_4: now also J2.6; no longer U1.1 (PD3)
- net RESET: now also J2.22
- net SCK: now also J2.21
- net OUT_2: now reaches U1.10 (PD6)
- net OUT_3: now reaches U1.11 (PD7)
- net OUT_4: now reaches U1.12 (PB0)
- net CS_1: now reaches U1.13 (PB1)
- net CS_2: now reaches U1.14 (PB2)
- net CURRENT_MCU: now reaches U1.2 (PD4)
- net OUT_1: now reaches U1.9 (PD5)
- new net +12V: J2.1, J2.10, J2.17, J2.18, J2.2, J2.9
- new net BRAKE_AIN: J3.11
- new net BRAKE_AIN_MCU: U1.1 (PD3)
- new net CANH_1: J3.13, J3.5
- new net CANH_2: J3.15, J3.7
- new net CANL_1: J3.14, J3.6
- new net CANL_2: J3.16, J3.8
- new net CURRENT_AIN: J3.12
- new net IGN_12V: J2.11
- new net IGN_5V: U1.32 (PD2)
- new net RXD: J2.12, U1.30 (PD0)
- new net TXD: J2.13, U1.31 (PD1)
Other:
- removed sheet PDU_1
- removed sheet PDU_2
- removed sheet PDU_3
- removed sheet PDU_4
- added sheet Analog Input (AIN.kicad_sch)
- added sheet PDU_P8 (PDU_P8.kicad_sch)
- sheet Digital Input ports: added IN, OUT; removed none

Commit message: vcuv3.2 haha where
Parts:
- added D6, D7, D8: D, symbol Device:D
- added R3, R4: 4k7, symbol Device:R
- C4, C5: value 22pF -> 20pF
Connections:
- net +5V: now also D6.1 (K); no longer J1.2 (VCC)
- net BRAKE_AIN_MCU: now also U1.23 (PC0); no longer U1.1 (PD3)
- net CS_1: now also D7.1 (K)
- net CS_2: now also D8.1 (K)
- net CURRENT_MCU: now also U1.24 (PC1); no longer U1.2 (PD4)
- net GND: no longer J3.24
- net IGN_12V: now also J3.24; no longer J2.11
- net IGN_5V: now also U1.28 (PC5); no longer U1.32 (PD2)
- net DIN_1: now reaches J3.21
- net DIN_2: now reaches J3.22
- net DIN_3: now reaches J3.23
- new net: D8.2 (A), R3.2
- new net: D7.2 (A), R4.2
- new net +5VD: D6.2 (A), J1.2 (VCC), R3.1, R4.1
- new net DIN5V_1: U1.32 (PD2)
- new net DIN5V_2: U1.1 (PD3)
- new net DIN5V_3: U1.2 (PD4)
Other:
- sheet Digital Input ports: added INPUT_1, INPUT_2, INPUT_3, INPUT_4, OUT_1, OUT_2, OUT_3, OUT_4; removed IN, OUT

Commit message: VCU V3.2
Parts:
- removed D6, D7, D8: D, symbol Device:D
- added C4: 100nF, RMC_Capacitor:C_0805_2012Metric_Pad1.18x1.45mm_HandSolder_L, symbol Device:C
- added H1, H2, H3, H4: MountingHole_Pad, RMC_MountingHole:MountingHole_3.2mmx5mm_M3_ISO7380, symbol Mechanical:MountingHole_Pad
- added J4: Conn_01x03, Connector_JST:JST_XH_B3B-XH-A_1x03_P2.50mm_Vertical, symbol Connector_Generic:Conn_01x03
- added J5: Conn_01x04, Connector_JST:JST_XH_B4B-XH-A_1x04_P2.50mm_Vertical, symbol Connector_Generic:Conn_01x04
- C1, C2, C3: footprint (none) -> RMC_Capacitor:C_0805_2012Metric_Pad1.18x1.45mm_HandSolder_L
- C5: renamed from C4; footprint (none) -> RMC_Capacitor:C_0805_2012Metric_Pad1.18x1.45mm_HandSolder_L
- C6: renamed from C5; footprint (none) -> RMC_Capacitor:C_0805_2012Metric_Pad1.18x1.45mm_HandSolder_L
- C7: renamed from C6; footprint (none) -> RMC_Capacitor:C_0805_2012Metric_Pad1.18x1.45mm_HandSolder_L
- J1: renamed from J2; footprint Better_Handsolder:HD241_24pin -> RMC_Connnector:HD241_24pin
- J2: renamed from J3; footprint Better_Handsolder:HD241_GF30 -> RMC_Connnector:HD241_GF30
- J3: renamed from J1; footprint (none) -> RMC_Connnector:PinHeader_2x03_P2.54mm_Vertical_handsolder
- R1: renamed from R4; value 4k7 -> 47k; footprint (none) -> RMC_Resistor:R_0805_2012Metric_Pad1.20x1.40mm_HandSolder_L
- R2: renamed from R3; value 4k7 -> 47k; footprint (none) -> RMC_Resistor:R_0805_2012Metric_Pad1.20x1.40mm_HandSolder_L
- R3: renamed from R1; footprint (none) -> RMC_Resistor:R_0805_2012Metric_Pad1.20x1.40mm_HandSolder_L
- R4: renamed from R2; footprint (none) -> RMC_Resistor:R_0805_2012Metric_Pad1.20x1.40mm_HandSolder_L
- SW1: footprint (none) -> Button_Switch_THT:SW_PUSH_6mm
- U1: footprint Package_QFP:TQFP-32_7x7mm_P0.8mm -> RMC_QFP:TQFP-32_7x7mm_P0.8mm_L
- Y1: footprint (none) -> RMC_Crystal:Crystal_HC49-U_Vertical_W_SMD_Handolder
Connections:
- net +5VD is gone; now on net +5V: J3.2 (VCC), R1.1, R2.1
- net +5V: now also J1.19, C4.1; no longer J1.14
- net CS_1: now also R1.2
- net CS_2: now also R2.2
- net GND: now also C4.2, J4.3 (Pin_3), J5.4 (Pin_4)
- net MISO: now also J5.1 (Pin_1); no longer J1.19
- net MOSI: now also J5.2 (Pin_2); no longer J1.20
- net PDU_1: now also J1.11
- net PDU_2: now also J1.12
- net PDU_3: now also J1.13
- net PDU_4: now also J1.14
- net RESET: no longer J1.22
- net RXD: now also J4.1 (Pin_1); no longer J1.12
- net SCK: now also J5.3 (Pin_3); no longer J1.21
- net TXD: now also J4.2 (Pin_2); no longer J1.13
- net OUT_5: now reaches U1.25 (PC2)
- net OUT_6: now reaches U1.26 (PC3)
- net OUT_7: now reaches U1.27 (PC4)
- new net GNDA: H1.1, H2.1, H3.1, H4.1
- new net PDU_5: J1.20
- new net PDU_6: J1.21
- new net PDU_7: J1.22
Other:
- sheet PDU_P8 renamed PDU_P4_1
- added sheet PDU_5 (PDU_P_sot23.kicad_sch)
- added sheet PDU_6 (PDU_P_sot23.kicad_sch)
- added sheet PDU_7 (PDU_P_sot23.kicad_sch)
- sheet APPS_3V3 ports: added AVCC; removed none
- sheet PDU_P4_1: file PDU_P8.kicad_sch -> PDU_P4.kicad_sch
- moved on the sheet: C2, C3, J3, R1, R2

Commit message: AHHHHH vcu v3.2
Connections:
- net CANH_1 renamed CAN1-
- net CANH_2 renamed CAN2-
- net CANL_1 renamed CAN1+
- net CANL_2 renamed CAN2+
Other:
- added sheet CAN BUS_3 (MCP2515+ TJA1051.kicad_sch)

Commit message: haha VCU V3.2 AND NEW SCHEMATICS HAHAHA
Parts:
- removed J1: ~, RMC_Connnector:HD241_24pin, symbol HD241:HD241
- removed J2: ~, RMC_Connnector:HD241_GF30, symbol HD241:HD241
Other:
- added sheet Connectors (VCU_connector.kicad_sch)
