File: kicad/VCU V3.2/VCU V3.2.kicad_sch (KiCad schematic)
At the start: 21 parts, among them J3 AVR-ISP-6, J4 Conn_01x03, J5 Conn_01x04, SW1 SW_Push, U1 ATmega328P-A, Y1 16MHz

Commit message: VCU V3.2 FINISH LAYOUT
Parts:
- added JP5: Jumper_3_Open, Jumper:SolderJumper-3_P1.3mm_Open_Pad1.0x1.5mm, symbol Jumper:Jumper_3_Open
- added R74: 47k, RMC_Resistor:R_0805_2012Metric_Pad1.20x1.40mm_HandSolder_L, symbol Device:R
Connections:
- net +5V: now also R74.1
- net TXD: now also JP5.1 (A); no longer U1.31 (PD1)
- new net: JP5.2 (C), U1.31 (PD1)
- new net CS_3: JP5.3 (B), R74.2
Other:
- moved on the sheet: J3
