File: kicad/VCU V3.2/MCP2515+ TJA1051.kicad_sch (KiCad schematic)
At the start: 9 parts, among them U6 MCP2515-xST, U8 TJA1051T, Y2 20MHz

Commit message: VCU V3.2
Parts:
- added R32: 120R, symbol Device:R
- renumbered C18 to C15, C17 to C16, C15 to C17, C16 to C18, R20 to R19, R25 to R20, U6 to U4, U8 to U5
Connections:
- net CANH: now also R32.2
- net CANL: now also R32.1

Commit message: vcuv3.2 haha where
Parts:
- C15, C16: value 22pF -> 16pF
Changed lines of the file:
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@@
 			)
 		)
-		(property "Value" "22pF"
+		(property "Value" "16pF"
 			(at 47.625 76.8349 90)
 			(effects
@@
 			)
 		)
-		(property "Value" "22pF"
+		(property "Value" "16pF"
 			(at 47.625 95.8851 90)
 			(effects

Commit message: VCU V3.2
Parts:
- C16: renamed from C15; footprint (none) -> RMC_Capacitor:C_0805_2012Metric_Pad1.18x1.45mm_HandSolder_L
- C17: renamed from C16; footprint (none) -> RMC_Capacitor:C_0805_2012Metric_Pad1.18x1.45mm_HandSolder_L
- C18: renamed from C17; footprint (none) -> RMC_Capacitor:C_0805_2012Metric_Pad1.18x1.45mm_HandSolder_L
- C19: renamed from C18; footprint (none) -> RMC_Capacitor:C_0805_2012Metric_Pad1.18x1.45mm_HandSolder_L
- R21: renamed from R19; footprint (none) -> RMC_Resistor:R_0805_2012Metric_Pad1.20x1.40mm_HandSolder_L
- R22: renamed from R20; footprint (none) -> RMC_Resistor:R_0805_2012Metric_Pad1.20x1.40mm_HandSolder_L
- R23: renamed from R32; footprint (none) -> RMC_Resistor:R_0805_2012Metric_Pad1.20x1.40mm_HandSolder_L
- U4: footprint Package_SO:TSSOP-20_4.4x6.5mm_P0.65mm -> RMC_SO:TSSOP-20_4.4x6.5mm_P0.65mm
- U5: footprint Package_SO:SOIC-8_3.9x4.9mm_P1.27mm -> RMC_SO:SOIC-8_3.9x4.9mm_P1.27mm_RMC_Handsolder
- Y2: footprint (none) -> RMC_Crystal:Crystal_HC49-U_Vertical_W_SMD_Handolder

Commit message: VCU V3.2 FINISH LAYOUT
Changed lines of the file:
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@@
-		)
-	)
-	(global_label "XTAL2"
-		(shape input)
-		(at 91.44 83.82 180)
-		(fields_autoplaced yes)
-		(effects
-			(font
-				(size 1.27 1.27)
-			)
-			(justify right)
-		)
-		(property "Intersheetrefs" "${INTERSHEET_REFS}"
-			(at 82.9515 83.82 0)
-			(effects
-				(font
-					(size 1.27 1.27)
-				)
-				(justify right)
-				(hide yes)
-			)
-		)
-	)
-	(global_label "XTAL1"
-		(shape input)
-		(at 64.77 90.17 0)
-		(fields_autoplaced yes)
-		(effects
-			(font
-				(size 1.27 1.27)
-			)
-			(justify left)
-		)
-		(property "Intersheetrefs" "${INTERSHEET_REFS}"
-			(at 73.2585 90.17 0)
-			(effects
-				(font
-					(size 1.27 1.27)
-				)
-				(justify left)
-				(hide yes)
-			)
 		)
 	)
@@
 		(property "Intersheetrefs" "${INTERSHEET_REFS}"
 			(at 83.8586 63.5 0)
-			(effects
-				(font
-					(size 1.27 1.27)
-				)
-				(justify right)
-				(hide yes)
-			)
-		)
-	)
-	(global_label "XTAL2"
-		(shape input)
-		(at 64.77 82.55 0)
-		(fields_autoplaced yes)
-		(effects
-			(font
-				(size 1.27 1.27)
-			)
-			(justify left)
-		)
-		(property "Intersheetrefs" "${INTERSHEET_REFS}"
-			(at 73.2585 82.55 0)
-			(effects
-				(font
-					(size 1.27 1.27)
-				)
-				(justify left)
-				(hide yes)
-			)
-		)
-	)
-	(global_label "XTAL1"
-		(shape input)
-		(at 91.44 86.36 180)
-		(fields_autoplaced yes)
-		(effects
-			(font
-				(size 1.27 1.27)
-			)
-			(justify right)
-		)
-		(property "Intersheetrefs" "${INTERSHEET_REFS}"
-			(at 82.9515 86.36 0)
 			(effects
 				(font
@@
 		)
 	)
+	(hierarchical_label "XTAL1"
+		(shape input)
+		(at 91.44 86.36 180)
+		(effects
+			(font
+				(size 1.27 1.27)
+			)
+			(justify right)
+		)
+	)
 	(hierarchical_label "CANL"
 		(shape input)
@@
 			)
 			(justify left)
+		)
+	)
+	(hierarchical_label "XTAL2"
+		(shape input)
+		(at 91.44 83.82 180)
+		(effects
+			(font
+				(size 1.27 1.27)
+			)
+			(justify right)
 		)
 	)
@@
 		)
 	)
+	(hierarchical_label "XTAL1"
+		(shape input)
+		(at 64.77 90.17 0)
+		(effects
+			(font
+				(size 1.27 1.27)
+			)
+			(justify left)
+		)
+	)
+	(hierarchical_label "XTAL2"
+		(shape input)
+		(at 64.77 82.55 0)
+		(effects
+			(font
+				(size 1.27 1.27)
+			)
+			(justify left)
+		)
+	)
