File: kicad/VCU V3.2/SRU.kicad_sch (KiCad schematic)
At the start: 5 parts, among them U9 LTV-817S

Commit message: VCU V3.2
Parts:
- removed R27: 10k, symbol Device:R
- added R44: 10k, symbol Device:R
- renumbered C24 to C25, R28 to R29, R29 to R31, U9 to U10
Connections:
- net GND: now also R44.1
- net IN: now also C25.1, R44.2
- net at R29.2, U10.1: no longer C25.1
Other:
- moved on the sheet: C25, R29, R31, U10

Commit message: vcuv3.2 haha where
Parts:
- removed C25: 100nF, symbol Device:C
- removed R29: 1k, symbol Device:R
- removed R31: 4k7, symbol Device:R
- removed R44: 10k, symbol Device:R
- removed U10: LTV-817S, Package_DIP:SMDIP-4_W9.53mm, symbol Isolator:LTV-817S
- added CA2, CA3, CA4, CA6: 100nF, RMC_Capacitor:C_0805_2012Metric_Pad1.18x1.45mm_HandSolder_L, symbol Device:C
- added R54, R55, R56, R69: 10k, RMC_Resistor:R_0805_2012Metric_Pad1.20x1.40mm_HandSolder_L, symbol Device:R
- added R57, R58, R59, R60, R62, R63, R64, R77: 1k, RMC_Resistor:R_0805_2012Metric_Pad1.20x1.40mm_HandSolder_L, symbol Device:R
- added R65, R66, R67, R68: 4.7k, RMC_Resistor:R_0805_2012Metric_Pad1.20x1.40mm_HandSolder_L, symbol Device:R
- added U13: 40106, CD40106BMT:SOIC127P600X175-14N, symbol 4xxx:40106
- added U14: LTV-847S, Package_DIP:SMDIP-16_W9.53mm, symbol Isolator:LTV-847S
Connections:
- net GND: now also CA2.2, CA3.2, CA4.2, CA6.1, R54.2, R55.2, R56.2, R69.1, U14.11, U14.13, U14.15, U14.2, U14.4, U14.6, U14.8, U14.9
- new net: CA6.2, R57.2, R69.2, U13.1
- new net: CA3.1, R55.1, R59.2, U13.5
- new net: CA2.1, R54.1, R58.2, U13.3
- new net: R63.1, U13.6
- new net: R63.2, U14.5
- new net: R64.1, U13.8
- new net: R64.2, U14.7
- new net: R62.1, U13.4
- new net: R60.2, U13.9
- new net: R62.2, U14.3
- new net: R77.2, U14.1
- new net: R77.1, U13.2
- new net +5VD: R65.2, R66.2, R67.2, R68.2
- new net INPUT_1: R57.1
- new net INPUT_2: R58.1
- new net INPUT_3: R59.1
- new net INPUT_4: CA4.1, R56.1, R60.1
- new net OUT_1: R65.1, U14.16
- new net OUT_2: R66.1, U14.14
- new net OUT_3: R67.1, U14.12
- new net OUT_4: R68.1, U14.10

Commit message: VCU V3.2
Parts:
- added CA5: 100nF, RMC_Capacitor:C_0805_2012Metric_Pad1.18x1.45mm_HandSolder_L, symbol Device:C
- U10: renamed from U13; footprint CD40106BMT:SOIC127P600X175-14N -> RMC_SO:SOIC127P600X175-14N
- renumbered CA6 to CA1, R57 to R33, R58 to R34, R59 to R35, R56 to R36, R69 to R37, R55 to R38, R54 to R39, R60 to R40, R77 to R41, R62 to R42, R63 to R43, R64 to R44, R65 to R45, R66 to R46, R67 to R47, R68 to R48, U14 to U11
Connections:
- net GND: now also U10.7 (VSS), CA5.2
- net +5VD renamed +5V
- net +5V: now also U10.14 (VDD), CA5.1
- no-connect marks 0 -> 4

Commit message: AHHHHH vcu v3.2
Parts:
- added unit 7 of U10
- added unit 5 of U10
- added unit 6 of U10
Connections:
- net +5V: now also U10.14 (VDD); no longer U10.14 (VDD)
- net GND: now also U10.7 (VSS); no longer U10.7 (VSS)

Commit message: haha VCU V3.2 AND NEW SCHEMATICS HAHAHA
Connections:
- net OUT_1: now also U11.10; no longer U11.16
- net OUT_2: now also U11.12; no longer U11.14
- net OUT_3: now also U11.14; no longer U11.12
- net OUT_4: now also U11.16; no longer U11.10
- net at R43.2: now also U11.3; no longer U11.5
- net at R44.2: now also U11.1; no longer U11.7
- net at R42.2: now also U11.5; no longer U11.3
- net at R41.2: now also U11.7; no longer U11.1
Other:
- moved on the sheet: U11A, U11B, U11C, U11D

Commit message: VCU V3.2 FINISH LAYOUT
Connections:
- net INPUT_4: no longer CA4.1, R36.1
- net at R40.2, U10.9: now also CA4.1, R36.1
Other:
- moved on the sheet: R40
Changed lines of the file:
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@@
 	(wire
 		(pts
-			(xy 120.65 135.89) (xy 129.54 135.89)
+			(xy 120.65 135.89) (xy 137.16 135.89)
 		)
 		(stroke
@@
 		(pts
 			(xy 106.68 107.95) (xy 119.38 107.95)
-		)
-		(stroke
-			(width 0)
-			(type default)
-		)
-	)
-	(wire
-		(pts
-			(xy 96.647 135.89) (xy 104.14 135.89)
 		)
 		(stroke
@@
 	(hierarchical_label "INPUT_4"
 		(shape input)
-		(at 96.647 135.89 180)
+		(at 96.52 135.89 180)
 		(effects
 			(font
@@
 	(symbol
 		(lib_id "Device:R")
-		(at 133.35 135.89 90)
+		(at 100.33 135.89 90)
 		(unit 1)
 		(exclude_from_sim no)
@@
 		(dnp no)
 		(property "Reference" "R40"
-			(at 133.35 133.35 90)
+			(at 100.33 133.35 90)
 			(effects
 				(font
@@
 		)
 		(property "Value" "1k"
-			(at 133.35 135.89 90)
+			(at 100.33 135.89 90)
 			(effects
 				(font
@@
 		)
 		(property "Footprint" "RMC_Resistor:R_0805_2012Metric_Pad1.20x1.40mm_HandSolder_L"
-			(at 133.35 137.668 90)
+			(at 100.33 137.668 90)
 			(effects
 				(font
@@
 		)
 		(property "Datasheet" "~"
-			(at 133.35 135.89 0)
+			(at 100.33 135.89 0)
 			(effects
 				(font
@@
 		)
 		(property "Description" ""
-			(at 133.35 135.89 0)
-			(effects
-				(font
+			(at 100.33 135.89 0)
+			(effects
+				(font

Commit message: VCU V3.2 DONE HAHA
Do you remember? the 21st night of September.
Parts:
- U11: footprint Package_DIP:SMDIP-16_W9.53mm -> to be sorted:SMDIP-16_W9.53mm
Changed lines of the file:
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@@
 			)
 		)
-		(property "Footprint" "Package_DIP:SMDIP-16_W9.53mm"
+		(property "Footprint" "to be sorted:SMDIP-16_W9.53mm"
 			(at 157.48 90.17 0)
 			(effects
@@
 			)
 		)
-		(property "Footprint" "Package_DIP:SMDIP-16_W9.53mm"
+		(property "Footprint" "to be sorted:SMDIP-16_W9.53mm"
 			(at 167.64 146.05 0)
 			(effects
@@
 			)
 		)
-		(property "Footprint" "Package_DIP:SMDIP-16_W9.53mm"
+		(property "Footprint" "to be sorted:SMDIP-16_W9.53mm"
 			(at 157.48 63.5 0)
 			(effects
@@
 			)
 		)
-		(property "Footprint" "Package_DIP:SMDIP-16_W9.53mm"
+		(property "Footprint" "to be sorted:SMDIP-16_W9.53mm"
 			(at 157.48 118.11 0)
 			(effects
