File: kicad/SSRU_v3.2/SSRU_v3.2.kicad_pcb (KiCad board)
At the start: 2 copper layers, 95 x 78 mm, 82 parts, among them J1 Conn_01x03, J2 Conn_01x24, J3 Conn_02x03_Odd_Even, J31 Conn_01x04, J4 AVR-ISP-6, J5 Conn_01x03, SW1 SW_Push, U1 MCP2515-xST, U10 TJA1051T, U12 TJA1051T, U2 ATmega328P-A, U3 LM2904, U4 LM2576S-5, U5 AMS1117-3.3, U6 MCP2515-xST, U8 74LVC1G17, Y1 16MHz, Y3 20MHz, Y4 20MHz

Commit message: stuffs
Parts:
- moved U6 182.7 mm to (164.2, 92.0), turned to -90 degrees
- moved U1 16.0 mm to (164.2, 108.0)
Routing:
- net Net-(U1-TXCAN): track 26.4 -> 13.2 mm
- net Net-(U10-TXD): track 0.00 -> 13.3 mm
- net Net-(U6-OSC2): track 0.00 -> 12.1 mm
- net Net-(U1-OSC1): track 21.7 -> 10.4 mm
- net Net-(U1-OSC2): track 21.8 -> 10.6 mm
- net Net-(U6-OSC1): track 0.00 -> 11.0 mm
- net Net-(U1-RXCAN): track 19.3 -> 9.67 mm
- net Net-(U10-RXD): track 0.00 -> 9.67 mm
- net MOSI: track 61.0 -> 58.7 mm
- net SCK: track 46.6 -> 44.5 mm
- net MISO: track 51.9 -> 50.0 mm
- net CS_CAN2: track 35.8 -> 34.2 mm
- net Net-(U1-~{RESET}): track 4.41 -> 5.73 mm

Commit message: Done SSRUV3.2 VCU V3.2
Parts:
- removed C10, C8: 100nF, RMC_Capacitor:C_0805_2012Metric_Pad1.18x1.45mm_HandSolder_L
- removed C20: 22uF, Capacitor_Tantalum_SMD:CP_EIA-7343-30_AVX-N_HandSolder
- removed C9: 10uF, RMC_Capacitor:C_0805_2012Metric_Pad1.18x1.45mm_HandSolder_L
- removed D4: LED, RMC_LED:LED_0805_2012Metric_Pad1.45x1.40mm_HandSolder
- removed D6: SMA Diode, Diode_SMD:D_SMA_Handsoldering
- removed F1, F3: Fuse, to be sorted:Fuse_1210_3225Metric_Pad1.42x2.65mm_HandSolder
- removed J1: Conn_01x03, Connector_PinHeader_2.54mm:PinHeader_1x03_P2.54mm_Vertical
- removed J3: Conn_02x03_Odd_Even, Connector_PinHeader_2.54mm:PinHeader_2x03_P2.54mm_Vertical
- removed R37: 50k, RMC_Resistor:R_0805_2012Metric_Pad1.20x1.40mm_HandSolder_L
- removed R39: 120R, RMC_Resistor:R_0805_2012Metric_Pad1.20x1.40mm_HandSolder_L
- removed R7, R8: 1M, RMC_Resistor:R_0805_2012Metric_Pad1.20x1.40mm_HandSolder_L
- removed U5: AMS1117-3.3, RMC_SOT:SOT-223-3_TabPin2_Handsolder
- added C32: 100nF, RMC_Capacitor:C_0805_2012Metric_Pad1.18x1.45mm_HandSolder_L, F.Cu at (126.0, 101.8)
- added C37: 100nF, RMC_Capacitor:C_0805_2012Metric_Pad1.18x1.45mm_HandSolder_L, F.Cu at (141.5, 103.0)
- C26, C27, C41, C42: value 22pF -> 16pF
- C31, C36, R1, R2, R6, U3: moved to F.Cu
- moved G*** 130.4 mm to (125.0, 129.5)
- moved R6 31.3 mm to (181.5, 108.5), turned to 180 degrees
- moved R40 19.6 mm to (122.5, 112.0)
- moved R2 14.5 mm to (142.5, 99.5)
- moved C36 14.3 mm to (140.3, 99.5)
- moved SW1 8.01 mm to (180.2, 123.1), turned to -90 degrees
- moved J31 7.50 mm to (193.8, 124.0), turned to 180 degrees
- moved U3 6.26 mm to (133.7, 101.2), turned to 180 degrees
- moved C23 4.63 mm to (136.5, 97.0), turned to 0 degrees
- moved C19 3.99 mm to (144.3, 122.0)
- moved C30 3.99 mm to (145.6, 118.7)
- moved J5 3.99 mm to (139.6, 123.2)
- moved R3 3.99 mm to (140.6, 125.7)
- moved U8 3.99 mm to (140.1, 119.7)
- moved C24 3.29 mm to (184.5, 135.2)
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Connections:
- J2 pad 12: POT2_IN -> POT1_IN
- J2 pad 13: j1 -> POT2_IN
- J2 pad 14: j2 -> ENCODER+
- J2 pad 15: j3 -> I2C+
- J2 pad 18: CAN1- -> FLOW_IN
- J2 pad 19: CAN1+ -> PUMP_NTC_50k
- J2 pad 21: DS18B20 -> +5V
- J2 pad 22: unconnected-(J2-Pin_22-Pad22) -> +5V
- J2 pad 23: unconnected-(J2-Pin_23-Pad23) -> +5V
- J2 pad 24: unconnected-(J2-Pin_24-Pad24) -> GND
- J2 pad 4: POT1_IN -> GND
- J2 pad 5: +3.3V -> GND
- J2 pad 6: I2C+ -> ENCODER-
- J2 pad 8: GND -> DS18B20
- J2 pad 9: +12V -> +5V
- J31 pad 2: UD+ -> 328-
- J31 pad 3: UD- -> 328+
- J31 pad 4: Net-(J31-Pin_4) -> +5V
- U2 pad 1: ENCODER- -> unconnected-(U2-PD3-Pad1)
- U2 pad 19: POT2_OUT -> unconnected-(U2-ADC6-Pad19)
- U2 pad 22: POT1_OUT -> POT2_OUT
- U2 pad 23: BRAKE_TEMP_OUT1 -> POT1_OUT
- U2 pad 24: BRAKE_TEMP_OUT2 -> PUMP_NTC_50k
- U2 pad 25: unconnected-(U2-PC2-Pad25) -> ENCODER-
- U2 pad 26: PUMP_NTC_50k -> ENCODER+
- U2 pad 32: ENCODER+ -> unconnected-(U2-PD2-Pad32)
- U3 pad 1: POT1_OUT -> POT2_OUT
- U3 pad 2: POT1_OUT -> POT2_OUT
- U3 pad 3: POT1_IN -> POT2_IN
- U3 pad 5: POT2_IN -> POT1_IN
- U3 pad 6: POT2_OUT -> POT1_OUT
- U3 pad 7: POT2_OUT -> POT1_OUT
Routing:
- net +12V: track 94.0 -> 0.00 mm
- net PUMP_PWM: track 77.6 -> 0.00 mm, vias 1 -> 0
- net unconnected-(J2-Pin_23-Pad23): track 75.0 -> 0.00 mm
- net unconnected-(J2-Pin_24-Pad24): track 73.7 -> 0.00 mm
- net BRAKE_TEMP_OUT2: track 59.3 -> 0.00 mm, vias 2 -> 0
- net BRAKE_TEMP_OUT1: track 57.6 -> 0.00 mm, vias 2 -> 0
- net +3.3V: track 50.8 -> 0.00 mm, vias 2 -> 0
- net FLOW_IN: track 14.1 -> 63.3 mm, vias 0 -> 1
- net FLOW_OUT: track 71.5 -> 107.0 mm
- net unconnected-(J2-Pin_22-Pad22): track 32.8 -> 0.00 mm, vias 1 -> 0
- net (no net): track 30.8 -> 0.00 mm, vias 1 -> 0
- net POT1_OUT: track 53.3 -> 82.4 mm, vias 1 -> 0
- net PUMP_NTC_50k: track 71.9 -> 98.4 mm, vias 2 -> 0
- net j3: track 24.2 -> 0.00 mm
- net j2: track 24.0 -> 0.00 mm
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- removed copper zone on F.Cu, net (none)
- removed copper zone on F.Cu, net +5V
- removed copper zone on F.Cu, net Net-(C10-Pad2)
- removed copper zone on F.Cu, net unconnected-(J2-Pin_22-Pad22)
Other:
- board text added: "+12V CAN2L CAN2H GND GND ENCB SDA DS18"
- board text added: "+5V CAN1L CAN1H POT1 POT2 ENCA SCL GND"
- board text added: "+5V FLOW NTC +5V +5V +5V +5V GND"
- board text added: "+5V MOSI GND"
- board text added: "+5V RX TX GND"
- board text added: "MISO SCK RST"
- board text added: "RBR_SSRU_V3.2 23/09/2025 PCB by Nicholas Chan Code by Jasmine Lee"
- board text added: "RST"

Commit message: gerbers
Connections:
- U2 pad 27: I2C+ -> I2C-
- U2 pad 28: I2C- -> I2C+
Routing:
- net I2C+: track 98.4 -> 98.0 mm, vias 2 -> 0
Changed lines of the file:
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@@
 			(psa4output no)
 			(plot_black_and_white yes)
-			(plotinvisibletext no)
 			(sketchpadsonfab no)
 			(plotpadnumbers no)
@@
 			(drillshape 0)
 			(scaleselection 1)
-			(outputdirectory "./")
+			(outputdirectory "./SSRU_GERBER")
 		)
 	)
@@
 			(size 2 0.55)
 			(layers "F.Cu" "F.Mask" "F.Paste")
-			(net 44 "I2C+")
+			(net 55 "I2C-")
 			(pinfunction "PC4")
 			(pintype "bidirectional")
@@
 			(size 2 0.55)
 			(layers "F.Cu" "F.Mask" "F.Paste")
-			(net 55 "I2C-")
+			(net 44 "I2C+")
 			(pinfunction "PC5")
 			(pintype "bidirectional")
@@
 	)
 	(segment
-		(start 188.5 115.103554)
-		(end 184.353554 119.25)
+		(start 157.75 115.5)
+		(end 161.5 119.25)
 		(width 0.25)
 		(layer "F.Cu")
@@
 	)
 	(segment
-		(start 139.25 115.5)
-		(end 134.75 111)
+		(start 184.353554 119.25)
+		(end 188.5 115.103554)
 		(width 0.25)
 		(layer "F.Cu")
@@
 	)
 	(segment
-		(start 134.75 111)
-		(end 116.355 111)
+		(start 139.25 115.5)
+		(end 157.75 115.5)
 		(width 0.25)
 		(layer "F.Cu")
@@
 	(segment
 		(start 116.355 111)
-		(end 114.175 108.82)
-		(width 0.25)
-		(layer "F.Cu")
-		(net 44)
-	)
-	(segment
-		(start 184.353554 119.25)
-		(end 161.5 119.25)
+		(end 134.75 111)
 		(width 0.25)
 		(layer "F.Cu")
@@
 	)
 	(segment
-		(start 188.5 104.396446)
-		(end 188.5 115.103554)
+		(start 134.75 111)
+		(end 139.25 115.5)
 		(width 0.25)
 		(layer "F.Cu")
@@
 	)
 	(segment
-		(start 186.75 102.646446)
-		(end 188.5 104.396446)
+		(start 188.5 115.103554)
+		(end 188.5 104.065686)
 		(width 0.25)
 		(layer "F.Cu")
@@
 	)
 	(segment
-		(start 157.75 115.5)
-		(end 139.25 115.5)
+		(start 114.175 108.82)
+		(end 116.355 111)
 		(width 0.25)
 		(layer "F.Cu")
@@
 	(segment
 		(start 161.5 119.25)
-		(end 157.75 115.5)
-		(width 0.25)
-		(layer "F.Cu")
-		(net 44)
-	)
-	(segment
-		(start 184.75 101.447056)
-		(end 183.298097 99.995153)
+		(end 184.353554 119.25)
 		(width 0.25)
 		(layer "F.Cu")
@@
 	)
 	(segment
-		(start 186.75 102.25)
-		(end 186.75 102.646446)
+		(start 188.5 104.065686)
+		(end 183.863782 99.429468)
 		(width 0.25)
 		(layer "F.Cu")
 		(net 44)
 	)
-	(via
-		(at 184.75 101.447056)
-		(size 0.6)
-		(drill 0.3)
-		(layers "F.Cu" "B.Cu")
-		(net 44)
-	)
-	(via
-		(at 186.75 102.25)
-		(size 0.6)
-		(drill 0.3)
-		(layers "F.Cu" "B.Cu")
-		(net 44)
-	)
-	(segment
-		(start 184.75 101.5)
-		(end 185 101.75)
-		(width 0.25)
-		(layer "B.Cu")
-		(net 44)
-	)
-	(segment
-		(start 184.75 101.447056)
-		(end 184.75 101.5)
-		(width 0.25)
-		(layer "B.Cu")
-		(net 44)
-	)
-	(segment
-		(start 185 101.75)
-		(end 186.25 101.75)
-		(width 0.25)
-		(layer "B.Cu")
-		(net 44)
-	)
-	(segment
-		(start 186.25 101.75)
-		(end 186.75 102.25)
-		(width 0.25)
-		(layer "B.Cu")
-		(net 44)
-	)
 	(segment
 		(start 140.89 121.51)
@@
 	)
 	(segment
-		(start 188 114.896446)
-		(end 184.146446 118.75)
-		(width 0.25)
-		(layer "F.Cu")
-		(net 55)
-	)
-	(segment
-		(start 120.055 110.5)
-		(end 118.375 108.82)
+		(start 118.375 108.82)
+		(end 120.055 110.5)
 		(width 0.25)
 		(layer "F.Cu")
@@
 	(segment
 		(start 158 115)
-		(end 139.5 115)
+		(end 161.75 118.75)
 		(width 0.25)
 		(layer "F.Cu")
@@
 	)
 	(segment
-		(start 185.75 102.353554)
-		(end 188 104.603554)
+		(start 188 114.896446)
+		(end 188 104.697056)
 		(width 0.25)
 		(layer "F.Cu")
@@
 	)
 	(segment
-		(start 161.75 118.75)
+		(start 139.5 115)
 		(end 158 115)
 		(width 0.25)
@@
 	)
 	(segment
-		(start 188 104.603554)
+		(start 184.146446 118.75)
 		(end 188 114.896446)
 		(width 0.25)
@@
 	)
 	(segment
-		(start 139.5 115)
-		(end 135 110.5)
-		(width 0.25)
-		(layer "F.Cu")
-		(net 55)
-	)
-	(segment
-		(start 184.146446 118.75)
-		(end 161.75 118.75)
+		(start 135 110.5)
+		(end 139.5 115)
 		(width 0.25)
 		(layer "F.Cu")
@@
 	)
 	(segment
-		(start 135 110.5)
-		(end 120.055 110.5)
+		(start 120.055 110.5)
+		(end 135 110.5)
 		(width 0.25)
 		(layer "F.Cu")
@@
 	)
 	(segment
-		(start 183.863782 99.429468)
-		(end 185.75 101.315686)
+		(start 188 104.697056)
+		(end 183.298097 99.995153)
 		(width 0.25)
 		(layer "F.Cu")
@@
 	)
 	(segment
-		(start 185.75 101.315686)
-		(end 185.75 102.353554)
+		(start 161.75 118.75)
+		(end 184.146446 118.75)
 		(width 0.25)
 		(layer "F.Cu")
