File: kicad/SSRU_v3.2/SSRU_v3.2.kicad_sch (KiCad schematic)
At the start: 81 parts, among them J1 Conn_01x03, J2 Conn_01x24, J3 Conn_02x03_Odd_Even, J31 Conn_01x04, J4 AVR-ISP-6, J5 Conn_01x03, SW1 SW_Push, U1 MCP2515-xST, U10 TJA1051T, U12 TJA1051T, U2 ATmega328P-A, U3 LM2904, U4 LM2576S-5, U5 AMS1117-3.3, U6 MCP2515-xST, U8 74LVC1G17, Y1 16MHz, Y3 20MHz, Y4 20MHz

Commit message: Done SSRUV3.2 VCU V3.2
Parts:
- removed C10, C8: 100nF, RMC_Capacitor:C_0805_2012Metric_Pad1.18x1.45mm_HandSolder_L, symbol Device:C
- removed C20: 22uF, Capacitor_Tantalum_SMD:CP_EIA-7343-30_AVX-N_HandSolder, symbol Device:C_Polarized
- removed C9: 10uF, RMC_Capacitor:C_0805_2012Metric_Pad1.18x1.45mm_HandSolder_L, symbol Device:C
- removed D4: LED, RMC_LED:LED_0805_2012Metric_Pad1.45x1.40mm_HandSolder, symbol Device:LED
- removed D6: SMA Diode, Diode_SMD:D_SMA_Handsoldering, symbol Device:D_Zener
- removed F1, F3: Fuse, to be sorted:Fuse_1210_3225Metric_Pad1.42x2.65mm_HandSolder, symbol Device:Fuse
- removed J1: Conn_01x03, Connector_PinHeader_2.54mm:PinHeader_1x03_P2.54mm_Vertical, symbol Connector_Generic:Conn_01x03
- removed J3: Conn_02x03_Odd_Even, Connector_PinHeader_2.54mm:PinHeader_2x03_P2.54mm_Vertical, symbol Connector_Generic:Conn_02x03_Odd_Even
- removed R37: 50k, RMC_Resistor:R_0805_2012Metric_Pad1.20x1.40mm_HandSolder_L, symbol Device:R
- removed R39: 120R, RMC_Resistor:R_0805_2012Metric_Pad1.20x1.40mm_HandSolder_L, symbol Device:R
- removed R7, R8: 1M, RMC_Resistor:R_0805_2012Metric_Pad1.20x1.40mm_HandSolder_L, symbol Device:R
- removed U5: AMS1117-3.3, RMC_SOT:SOT-223-3_TabPin2_Handsolder, symbol Regulator_Linear:AMS1117-3.3
- added C32, C37: 100nF, RMC_Capacitor:C_0805_2012Metric_Pad1.18x1.45mm_HandSolder_L, symbol Device:C
- C26, C27, C41, C42: value 22pF -> 16pF
Connections:
- net +3.3V is gone; now on net GND: J2.5 (Pin_5)
- net BRAKE_TEMP_OUT1 is gone; now on net POT1_OUT: U2.23 (PC0)
- net BRAKE_TEMP_OUT2 is gone; now on net PUMP_NTC_50k: U2.24 (PC1)
- net UD+ is gone; now on net 328-: J31.2 (Pin_2)
- net UD- is gone; now on net 328+: J31.3 (Pin_3)
- net j1 is gone; now on net POT2_IN: J2.13 (Pin_13)
- net j2 is gone; now on net ENCODER+: J2.14 (Pin_14)
- net j3 is gone; now on net I2C+: J2.15 (Pin_15)
- net +12V: no longer J2.9 (Pin_9)
- net +5V: now also J2.21 (Pin_21), J2.22 (Pin_22), J2.23 (Pin_23), J2.9 (Pin_9), J31.4 (Pin_4)
- net CAN1+: no longer J2.19 (Pin_19)
- net CAN1-: no longer J2.18 (Pin_18)
- net DS18B20: now also J2.8 (Pin_8); no longer J2.21 (Pin_21)
- net ENCODER+: now also U2.26 (PC3); no longer U2.32 (PD2)
- net ENCODER-: now also J2.6 (Pin_6), U2.25 (PC2); no longer U2.1 (PD3)
- net FLOW_IN: now also J2.18 (Pin_18)
- net GND: now also J2.24 (Pin_24), J2.4 (Pin_4), C32.1, C37.1; no longer J2.8 (Pin_8)
- net I2C+: no longer J2.6 (Pin_6)
- net POT1_IN: now also J2.12 (Pin_12), U3.5 (+); no longer J2.4 (Pin_4), U3.3 (+)
- net POT1_OUT: now also U3.6 (-), U3.7, C32.2; no longer U2.22 (ADC7), U3.1, U3.2 (-)
- net POT2_IN: now also U3.3 (+); no longer J2.12 (Pin_12), U3.5 (+)
- net POT2_OUT: now also U2.22 (ADC7), U3.1, U3.2 (-), C37.2; no longer U2.19 (ADC6), U3.6 (-), U3.7
- net PUMP_NTC_50k: now also J2.19 (Pin_19); no longer U2.26 (PC3)
Other:
- moved on the sheet: C19, C28, C30, C41, C42, J31, J5, R18, R3, U3A, U3B, U8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

Commit message: gerbers
Connections:
- net I2C+: now also U2.28 (PC5); no longer U2.27 (PC4)
- net I2C-: now also U2.27 (PC4); no longer U2.28 (PC5)
Changed lines of the file:
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@@
 	(global_label "SCL"
 		(shape input)
-		(at 92.71 67.31 0)
-		(fields_autoplaced yes)
-		(effects
-			(font
-				(size 1.27 1.27)
-			)
-			(justify left)
-		)
-		(property "Intersheetrefs" "${INTERSHEET_REFS}"
-			(at 99.2028 67.31 0)
+		(at 92.71 69.85 0)
+		(fields_autoplaced yes)
+		(effects
+			(font
+				(size 1.27 1.27)
+			)
+			(justify left)
+		)
+		(property "Intersheetrefs" "${INTERSHEET_REFS}"
+			(at 99.2633 69.85 0)
 			(effects
 				(font
@@
 		)
 	)
+	(global_label "CS_CAN2"
+		(shape input)
+		(at 116.84 43.18 0)
+		(fields_autoplaced yes)
+		(effects
+			(font
+				(size 1.27 1.27)
+			)
+			(justify left)
+		)
+		(property "Intersheetrefs" "${INTERSHEET_REFS}"
+			(at 129.0175 43.18 0)
+			(effects
+				(font
+					(size 1.27 1.27)
+				)
+				(justify left)
+				(hide yes)
+			)
+		)
+	)
 	(global_label "POT1_IN"
 		(shape input)
@@
 				)
 				(justify right)
+				(hide yes)
+			)
+		)
+	)
+	(global_label "CS_CAN1"
+		(shape input)
+		(at 116.84 45.72 0)
+		(fields_autoplaced yes)
+		(effects
+			(font
+				(size 1.27 1.27)
+			)
+			(justify left)
+		)
+		(property "Intersheetrefs" "${INTERSHEET_REFS}"
+			(at 128.1709 45.72 0)
+			(effects
+				(font
+					(size 1.27 1.27)
+				)
+				(justify left)
 				(hide yes)
 			)
@@
 	(global_label "SDA"
 		(shape input)
-		(at 92.71 69.85 0)
-		(fields_autoplaced yes)
-		(effects
-			(font
-				(size 1.27 1.27)
-			)
-			(justify left)
-		)
-		(property "Intersheetrefs" "${INTERSHEET_REFS}"
-			(at 99.2633 69.85 0)
-			(effects
-				(font
+		(at 92.71 67.31 0)
+		(fields_autoplaced yes)
+		(effects
+			(font
+				(size 1.27 1.27)
+			)
+			(justify left)
+		)
+		(property "Intersheetrefs" "${INTERSHEET_REFS}"
+			(at 99.2028 67.31 0)
+			(effects
+				(font
