File: kicad/TSAL_G_V4_2/TSAL_G_V4_2.kicad_sch (KiCad schematic)
At the start: 110 parts, among them J1 Conn_01x02_Pin, J2 Conn_01x02_Pin, J3 Conn_01x02_Pin, J4 Conn_01x02_Pin, J5 Conn_01x02_Pin, J6 Conn_01x02_Pin, J7 Conn_01x02_Pin, J8 Conn_01x02_Pin, Q1 PMOS, Q2 MMBT3904, U1 TLV431, U10 74HC04, U11 74HC86, U12 LM393, U13 LM393, U14 LM393, U15 LM393, U16 LM393, U17 LM393, U2 LTV-817S, U3 B1212, U4 74HC00, U5 4023, U6 LTV-847S, U7 LTV-847S, U8 74HC02, U9 74HC02

Commit message: AHHHHH vcu v3.2
Parts:
- removed D2: D, Diode_SMD:D_SMA_Handsoldering, symbol Device:D
Connections:
- net VCC: now also F2.2
Changed lines of the file:
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@@
 	(wire
 		(pts
+			(xy 200.66 137.16) (xy 200.66 136.398)
+		)
+		(stroke
+			(width 0)
+			(type default)
+		)
+	)
+	(wire
+		(pts
 			(xy 445.262 232.41) (xy 445.262 233.172)
 		)
@@
 	(wire
 		(pts
+			(xy 208.28 136.398) (xy 209.296 136.398)
+		)
+		(stroke
+			(width 0)
+			(type default)
+		)
+	)
+	(wire
+		(pts
 			(xy 468.884 232.664) (xy 468.884 233.426)
 		)
@@
 	(wire
 		(pts
+			(xy 200.66 136.398) (xy 195.326 136.398)
+		)
+		(stroke
+			(width 0)
+			(type default)
+		)
+	)
+	(wire
+		(pts
 			(xy 519.938 123.952) (xy 518.16 123.952)
 		)
@@
 	(wire
 		(pts
+			(xy 208.28 137.16) (xy 208.28 136.398)
+		)
+		(stroke
+			(width 0)
+			(type default)
+		)
+	)
+	(wire
+		(pts
 			(xy 269.748 136.144) (xy 284.988 136.144)
 		)
@@
 		)
 	)
-	(polyline
+	(wire
 		(pts
-			(xy 239.776 150.368) (xy 135.636 150.368)
+			(xy 200.66 137.16) (xy 208.28 137.16)
 		)
 		(stroke
 			(width 0)
-			(type dash)
+			(type default)
 		)
 	)
-	(wire
+	(polyline
 		(pts
-			(xy 108.966 76.708) (xy 114.046 76.708)
+			(xy 239.776 150.368) (xy 135.636 150.368)
 		)
 		(stroke
 			(width 0)
-			(type default)
+			(type dash)
 		)
 	)
 	(wire
 		(pts
-			(xy 199.136 136.398) (xy 195.326 136.398)
+			(xy 108.966 76.708) (xy 114.046 76.708)
 		)
 		(stroke
@@
 	(wire
 		(pts
-			(xy 209.296 136.398) (xy 206.756 136.398)
-		)
-		(stroke
-			(width 0)
-			(type default)
-		)
-	)
-	(wire
-		(pts
 			(xy 59.436 37.338) (xy 67.056 37.338)
 		)
@@
 					(unit 1)
 				)
-			)
-		)
-	)
-	(symbol
-		(lib_id "Device:D")
-		(at 202.946 136.398 0)
-		(mirror x)
-		(unit 1)
-		(exclude_from_sim no)
-		(in_bom yes)
-		(on_board yes)
-		(dnp no)
-		(property "Reference" "D2"
-			(at 201.7776 138.4046 90)
-			(effects
-				(font
-					(size 1.27 1.27)
-				)
-				(justify left)
-			)
-		)
-		(property "Value" "D"
-			(at 204.089 138.4046 90)
-			(effects
-				(font
-					(size 1.27 1.27)
-				)
-				(justify left)
-			)
-		)
-		(property "Footprint" "Diode_SMD:D_SMA_Handsoldering"
-			(at 202.946 136.398 0)
-			(effects
-				(font
-					(size 1.27 1.27)
-				)
-				(hide yes)
-			)
-		)
-		(property "Datasheet" "~"
-			(at 202.946 136.398 0)
-			(effects
-				(font
-					(size 1.27 1.27)
-				)
-				(hide yes)
-			)
-		)
-		(property "Description" ""
-			(at 202.946 136.398 0)
-			(effects
-				(font
-					(size 1.27 1.27)
-				)
-				(hide yes)
-			)
-		)
-		(pin "2"
-		)
-		(pin "1"
-		)
-		(instances
-			(project "TSAL_G_V4_2"
-				(path "/85dd7182-b71e-445a-95f4-dedd1af3b46e"
-					(reference "D2")
-					(unit 1)
-				)

Commit message: Updated TSAL G V4.2
this board already got fabbed
test is needed
Parts:
- removed C22, C23, C24: 0.1uF, RMC_Capacitor:C_0805_2012Metric_Pad1.18x1.45mm_HandSolder_L, symbol Device:C
- removed J3, J4, J5: Conn_01x02_Pin, Connector_Molex:Molex_Micro-Fit_3.0_43650-0215_1x02_P3.00mm_Vertical, symbol Connector:Conn_01x02_Pin
- removed R17, R23, R27: 1k, RMC_Resistor:R_0805_2012Metric_Pad1.20x1.40mm_HandSolder_L, symbol Device:R
- removed unit 6 of U10
- removed U12, U13, U17: LM393, RMC_SO:SOIC-8_3.9x4.9mm_P1.27mm_RMC_Handsolder, symbol Comparator:LM393
- removed U6: LTV-847S, Package_DIP:SMDIP-16_W9.53mm, symbol Isolator:LTV-847S
- added C2, C3, C4: 1u-10u, RMC_Capacitor:C_0805_2012Metric_Pad1.18x1.45mm_HandSolder_L, symbol Device:C
- added D2: D, Diode_SMD:D_SMA_Handsoldering, symbol Device:D
- added J3, J6, J7: Conn_01x03_Pin, Connector_Molex:Molex_Micro-Fit_3.0_43650-0315_1x03_P3.00mm_Vertical, symbol Connector:Conn_01x03_Pin
- added R10, R11, R12: 1M, RMC_Resistor:R_0805_2012Metric_Pad1.20x1.40mm_HandSolder_L, symbol Device:R
- added R13, R14, R47, R48, R49, R50: 4.7k, RMC_Resistor:R_0805_2012Metric_Pad1.20x1.40mm_HandSolder_L, symbol Device:R
- added R19, R34, R51, R52, R53: 1k, RMC_Resistor:R_0805_2012Metric_Pad1.20x1.40mm_HandSolder_L, symbol Device:R
- added unit 6 of U11
- added U2, U3: LM393, RMC_SO:SOIC-8_3.9x4.9mm_P1.27mm_RMC_Handsolder, symbol Comparator:LM393
- C11: renamed from C8; footprint RMC_Capacitor:C_0805_2012Metric_Pad1.18x1.45mm_HandSolder_L -> Capacitor_THT:CP_Radial_D5.0mm_P2.50mm
- renumbered C7 to C10, C15 to C12, C16 to C13, C17 to C14, C18 to C15, C19 to C16, C13 to C17, C21 to C18, C14 to C19, C2 to C5, C3 to C6, C4 to C7, C5 to C8, C6 to C9, D9 to D10, D14 to D11, D10 to D13, D11 to D14, D6 to D3, D3 to D4, D4 to D5, D7 to D6, D5 to D7, D13 to D9, J6 to J4, J7 to J5, Q2 to Q1, Q1 to Q2, R10 to R15, R11 to R16, R12 to R17, R13 to R18, R16 to R21, R18 to R22, R14 to R23, R15 to R24, R21 to R25, R19 to R26, R25 to R27, R22 to R28, R24 to R29, R34 to R30, R26 to R31, R28 to R32, R31 to R33, R36 to R35, R29 to R36, R33 to R37, R30 to R38, R32 to R39, R42 to R40, R43 to R41, R35 to R42, R37 to R43, R38 to R44, R39 to R45, R40 to R46, U9 to U10, U10 to U11, U11 to U12, U14 to U13, U15 to U14, U16 to U15, U2 to U4, U3 to U5, U4 to U6, U5 to U7, U7 to U8, U8 to U9
Connections:
- net +5V: now also R13.2, R47.2, R48.2, R49.2, R50.2, U2.8 (V+), U3.8 (V+)
- net AIR_H: now also U12.5, U8.11; no longer U12.10, U8.13
- net AIR_H_AUX: now also R27.1, U12.4, R51.2; no longer R20.1, U12.9
- net AIR_L: now also U12.10, U6.4, U8.13; no longer U12.13, U6.12, U8.15
- net AIR_L_AUX: now also R20.1, U12.9, U6.5, R52.2; no longer R27.1, U12.12, U6.13
- net GLV-: now also C2.2, C3.2, C4.2, R14.1, R19.1, U2.4 (V-), U3.4 (V-)
- net Light_out: now also U10.13, R34.1; no longer Q1.1 (B)
- net PRECHARGE: now also U6.12, U8.9; no longer U6.4, U8.11
- net PRECHARGE_AUX: now also U6.13, R53.2; no longer U6.5
- net RAW MCU_V: now also R19.2
- net RAW_AIR_H: now also U8.6, J6.2 (Pin_2); no longer U8.4
- net RAW_AIR_L: now also U8.4, J3.2 (Pin_2); no longer U8.2
- net RAW_PRECHARGE: now also U8.8, J7.2 (Pin_2); no longer U8.6
- net RAW_SCS: now also R50.1
- net VCC: now also D2.1 (K); no longer F2.2
- net VDD: now also U8.10, U8.12, U8.14, J3.1 (Pin_1), J6.1 (Pin_1), J7.1 (Pin_1); no longer U8.12, U8.14, U8.16
- net at U7.8: now also U6.11; no longer U6.6
- net at R29.2: now also U8.3; no longer U8.1
- net at U7.2: now also U6.6; no longer U6.11
- net AIR_L_F: now reaches U10.6
- net AIR_L_F: now also R48.1, U3.1; no longer U12.11
- net at R22.2: now also U8.5; no longer U8.3
- net at R33.2: now also U8.7; no longer U8.5
- net PRECHARGE_F: now reaches U10.3
- net PRECHARGE_F: now also R49.1, U2.1; no longer U12.3
- net AIR_H_F: now reaches U10.5
- net AIR_H_F: now also R47.1, U3.7; no longer U12.8
- net AUX_error renamed RELAY STATUS
- new net: D2.2 (A), F2.2
- new net: J3.3 (Pin_3), R52.1
- new net: J6.3 (Pin_3), R51.1
- new net: J7.3 (Pin_3), R53.1
- new net: Q1.1 (B), R34.2
- new net AIR_H_unmatch: C3.1, R11.2, U3.5 (+)
- new net AIR_H_unmatch_trig: R11.1, U12.6
- new net AIR_L_unmatch: C4.1, R12.2, U3.3 (+)
- new net AIR_L_unmatch_trig: R12.1, U12.8
- new net PRECHARGE_unmatch: C2.1, R10.2, U2.3 (+)
- new net PRECHARGE_unmatch_trig: R10.1, U12.3
- new net V_REF_DELAY: R13.1, R14.2, U2.2 (-), U3.2 (-), U3.6 (-)
- no-connect marks 14 -> 15
Other:
- moved on the sheet: C12, C13, C14, C15, C16, C20, D10, D11, D3, D6, D8, D9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
