File: kicad/BSPD/BSPD.kicad_sch (KiCad schematic)
At the start: 59 parts, among them J1 Conn_01x02, J2 Conn_01x02, J3 Conn_01x02, K1 SANYOU_SRD_Form_C, Q1 AO3400A, Q2 AO3401A, Q3 AO3400A, U1 LM393, U2 LM393, U3 74AHC1G00, U4 74AHC1G00, U5 LM78M05_TO252, U6 LM393, U7 LM393

Commit message: minor fix
Parts:
- added F1: Fuse, Fuse:Fuse_0805_2012Metric_Pad1.15x1.40mm_HandSolder, symbol Device:Fuse
- added R26, R27: 10k, Resistor_SMD:R_0805_2012Metric_Pad1.20x1.40mm_HandSolder, symbol Device:R
- added R28, R29: 100k, Resistor_SMD:R_0805_2012Metric_Pad1.20x1.40mm_HandSolder, symbol Device:R
Connections:
- net +12V: now also F1.1; no longer J3.1 (Pin_1)
- net GND: now also R28.2, R29.1
- net SIGN1: now also R26.2, R29.2; no longer J1.2 (Pin_2)
- net SIGN2: now also R27.2, R28.1; no longer J1.1 (Pin_1)
- new net: J1.1 (Pin_1), R27.1
- new net: F1.2, J3.1 (Pin_1)
- new net: J1.2 (Pin_2), R26.1
Other:
- note added: "Brake Pressure Sensor Hall Current Sensor"
- moved on the sheet: J1, J2, J3
